Commit message: Use reflect param

File: tiago_v2_prototype_description/robots/tiago_v2_prototype.urdf.xacro (robot description, xacro)
@@ -26,6 +26,6 @@
 <xacro:tiago_dual_torso name="torso" parent="base_link" has_screen="false"/>
 <!-- Arms -->
-<xacro:tiago_sea_arm name="arm_left" parent="torso_lift_link" reflect="1" arm_1_offset="0" arm_2_offset="0" arm_3_offset="0" arm_4_offset="0" arm_5_offset="0" arm_6_offset="0" arm_7_offset="0">
-  <origin xyz="0.13445 0.09 -0.156" rpy="1.0668 0 2.9933"/>
+<xacro:tiago_sea_arm name="arm_left" parent="torso_lift_link" reflect="-1" arm_1_offset="0" arm_2_offset="0" arm_3_offset="0" arm_4_offset="0" arm_5_offset="0" arm_6_offset="0" arm_7_offset="0">
+  <origin xyz="0.13445 0.09 -0.156" rpy="-1.0668 0 -0.14829"/>
 </xacro:tiago_sea_arm>
 <xacro:tiago_sea_arm name="arm_right" parent="torso_lift_link" reflect="1" arm_1_offset="0" arm_2_offset="0" arm_3_offset="0" arm_4_offset="0" arm_5_offset="0" arm_6_offset="0" arm_7_offset="0">

Commit message: Mounting pose of the arms in an external file

File: tiago_v2_prototype_description/robots/tiago_v2_prototype.urdf.xacro (robot description, xacro)
@@ -21,4 +21,9 @@
 <xacro:include filename="$(find tiago_dual_description)/urdf/torso/torso_dual.urdf.xacro" />
 <xacro:include filename="$(find tiago_sea_arm_description)/urdf/arm.urdf.xacro" />
+<xacro:include filename="$(find tiago_v2_prototype_description)/urdf/arm.mounting.xacro" />
+<xacro:property name="arm_left_xyz" value="${mounting_x + mounting_offset_x} ${mounting_y + mounting_offset_y} ${mounting_z + mounting_offset_z}" />
+<xacro:property name="arm_right_xyz" value="${mounting_x + mounting_offset_x} ${-(mounting_y + mounting_offset_y)} ${mounting_z + mounting_offset_z}" />
+<xacro:property name="arm_left_rpy" value="${-(mounting_roll + mounting_offset_roll)} ${-(mounting_pitch + mounting_offset_pitch)} ${-3.1415 + (mounting_yaw + mounting_offset_yaw)}" />
+<xacro:property name="arm_right_rpy" value="${-(mounting_roll + mounting_offset_roll)} ${-(mounting_pitch + mounting_offset_pitch)} ${-(mounting_yaw + mounting_offset_yaw)}" />
 <!-- Base -->
 <xacro:base_sensors name="base" front_laser_model="$(arg laser_model)" rear_laser_model="$(arg laser_model)"/>
@@ -27,8 +32,8 @@
 <!-- Arms -->
 <xacro:tiago_sea_arm name="arm_left" parent="torso_lift_link" reflect="-1" arm_1_offset="0" arm_2_offset="0" arm_3_offset="0" arm_4_offset="0" arm_5_offset="0" arm_6_offset="0" arm_7_offset="0">
-  <origin xyz="0.13445 0.09 -0.156" rpy="-1.0668 0 -0.14829"/>
+  <origin xyz="${arm_left_xyz}" rpy="${arm_left_rpy}"/>
 </xacro:tiago_sea_arm>
 <xacro:tiago_sea_arm name="arm_right" parent="torso_lift_link" reflect="1" arm_1_offset="0" arm_2_offset="0" arm_3_offset="0" arm_4_offset="0" arm_5_offset="0" arm_6_offset="0" arm_7_offset="0">
-  <origin xyz="0.13445 -0.09 -0.156" rpy="-1.0668 0 -2.9933"/>
+  <origin xyz="${arm_right_xyz}" rpy="${arm_right_rpy}"/>
 </xacro:tiago_sea_arm>
 </robot>

Commit message: Added params for arm placement and params in launch files

File: tiago_v2_prototype_description/robots/tiago_v2_prototype.urdf.xacro (robot description, xacro)
@@ -30,10 +30,18 @@
 <!-- Torso. TODO: change for custom torso -->
 <xacro:tiago_dual_torso name="torso" parent="base_link" has_screen="false"/>
+<xacro:arg name="arm_x" default="0.13445" />
+<xacro:arg name="arm_y" default="0.09" />
+<xacro:arg name="arm_z" default="-0.156" />
+<xacro:arg name="arm_roll" default="-1.0668" />
+<xacro:arg name="arm_pitch" default="0.0" />
+<xacro:arg name="arm_yaw" default="-0.14829" />
 <!-- Arms -->
 <xacro:tiago_sea_arm name="arm_left" parent="torso_lift_link" reflect="-1" arm_1_offset="0" arm_2_offset="0" arm_3_offset="0" arm_4_offset="0" arm_5_offset="0" arm_6_offset="0" arm_7_offset="0">
-  <origin xyz="${arm_left_xyz}" rpy="${arm_left_rpy}"/>
+  <origin xyz="$(arg arm_x) $(arg arm_y) $(arg arm_z)"
+          rpy="$(arg arm_roll) $(arg arm_pitch) $(arg arm_yaw)"/>
 </xacro:tiago_sea_arm>
 <xacro:tiago_sea_arm name="arm_right" parent="torso_lift_link" reflect="1" arm_1_offset="0" arm_2_offset="0" arm_3_offset="0" arm_4_offset="0" arm_5_offset="0" arm_6_offset="0" arm_7_offset="0">
-  <origin xyz="${arm_right_xyz}" rpy="${arm_right_rpy}"/>
+  <origin xyz="$(arg arm_x) ${-1.0*$(arg arm_y)} $(arg arm_z)"
+          rpy="$(arg arm_roll) $(arg arm_pitch) ${-3.1415-$(arg arm_yaw)}"/>
 </xacro:tiago_sea_arm>
 </robot>

Commit message: update for new arms placement

File: tiago_v2_prototype_description/robots/tiago_v2_prototype.urdf.xacro (robot description, xacro)
@@ -31,13 +31,14 @@
 <xacro:tiago_dual_torso name="torso" parent="base_link" has_screen="false"/>
 <!--
- xyz="0.13672 0.089185 -0.14357"
-      rpy="0.84402 0 2.812" />
+<origin
+      xyz="0.10529 0.15915 -0.11927"
+      rpy="-2.0679 0 -1.2217" />
 -->
-<xacro:arg name="arm_x" default="0.11049" />
-<xacro:arg name="arm_y" default="0.16261" />
-<xacro:arg name="arm_z" default="-0.12217" />
-<xacro:arg name="arm_roll" default="-2.0487" />
-<xacro:arg name="arm_pitch" default="0.019356" />
-<xacro:arg name="arm_yaw" default="-1.11659" />
+<xacro:arg name="arm_x" default="0.10529" />
+<xacro:arg name="arm_y" default="0.15915" />
+<xacro:arg name="arm_z" default="-0.11927" />
+<xacro:arg name="arm_roll" default="-2.0679" />
+<xacro:arg name="arm_pitch" default="0.0" />
+<xacro:arg name="arm_yaw" default="-1.2217" />
 <!-- Arms -->
 <xacro:tiago_sea_arm name="arm_left" parent="torso_lift_link" reflect="-1" arm_1_offset="0" arm_2_offset="0" arm_3_offset="0" arm_4_offset="0" arm_5_offset="0" arm_6_offset="0" arm_7_offset="0">

Commit message: First v2 proto alsmost working version

File: tiago_v2_prototype_description/robots/tiago_v2_prototype.urdf.xacro (robot description, xacro)
@@ -18,21 +18,17 @@
 <!-- Includes -->
 <xacro:include filename="$(find tiago_v2_prototype_description)/gazebo/gazebo.urdf.xacro" />
+<xacro:include filename="$(find tiago_v2_prototype_description)/urdf/torso/torso_dual.urdf.xacro" />
+<xacro:include filename="$(find tiago_v2_prototype_description)/urdf/head/head.urdf.xacro" />
 <xacro:include filename="$(find omni_base_description)/urdf/base/base_sensors.urdf.xacro" />
-<xacro:include filename="$(find tiago_dual_description)/urdf/torso/torso_dual.urdf.xacro" />
-<xacro:include filename="$(find tiago_sea_arm_description)/urdf/arm.urdf.xacro" />
-<xacro:include filename="$(find tiago_v2_prototype_description)/urdf/arm.mounting.xacro" />
-<xacro:property name="arm_left_xyz" value="${mounting_x + mounting_offset_x} ${mounting_y + mounting_offset_y} ${mounting_z + mounting_offset_z}" />
-<xacro:property name="arm_right_xyz" value="${mounting_x + mounting_offset_x} ${-(mounting_y + mounting_offset_y)} ${mounting_z + mounting_offset_z}" />
-<xacro:property name="arm_left_rpy" value="${-(mounting_roll + mounting_offset_roll)} ${-(mounting_pitch + mounting_offset_pitch)} ${-3.1415 + (mounting_yaw + mounting_offset_yaw)}" />
-<xacro:property name="arm_right_rpy" value="${-(mounting_roll + mounting_offset_roll)} ${-(mounting_pitch + mounting_offset_pitch)} ${-(mounting_yaw + mounting_offset_yaw)}" />
+<xacro:include filename="$(find tiago_v2_prototype_description)/urdf/arm/arm.urdf.xacro" />
 <!-- Base -->
 <xacro:base_sensors name="base" front_laser_model="$(arg laser_model)" rear_laser_model="$(arg laser_model)"/>
 <!-- Torso. TODO: change for custom torso -->
-<xacro:tiago_dual_torso name="torso" parent="base_link" has_screen="false"/>
+<xacro:tiago_v2_torso name="torso" parent="base_link"/>
+<xacro:tiago_v2_head name="head" parent="torso_lift_link"/>
 <!--
 <origin
       xyz="0.10529 0.15915 -0.11927"
       rpy="-2.0679 0 -1.2217" />
--->
 <xacro:arg name="arm_x" default="0.10529" />
 <xacro:arg name="arm_y" default="0.15915" />
@@ -41,12 +37,19 @@
 <xacro:arg name="arm_pitch" default="0.0" />
 <xacro:arg name="arm_yaw" default="-1.2217" />
+-->
+<xacro:arg name="arm_x" default="0.08976" />
+<xacro:arg name="arm_y" default="0.15918" />
+<xacro:arg name="arm_z" default="-0.092008" />
+<xacro:arg name="arm_roll" default="-2.0679" />
+<xacro:arg name="arm_pitch" default="0.0" />
+<xacro:arg name="arm_yaw" default="-1.2217" />
 <!-- Arms -->
-<xacro:tiago_sea_arm name="arm_left" parent="torso_lift_link" reflect="-1" arm_1_offset="0" arm_2_offset="0" arm_3_offset="0" arm_4_offset="0" arm_5_offset="0" arm_6_offset="0" arm_7_offset="0">
+<xacro:tiago_v2_arm name="arm_left" parent="torso_lift_link" reflect="-1" arm_1_offset="0" arm_2_offset="0" arm_3_offset="0" arm_4_offset="0" arm_5_offset="0" arm_6_offset="0" arm_7_offset="0">
   <origin xyz="$(arg arm_x) $(arg arm_y) $(arg arm_z)"
           rpy="$(arg arm_roll) $(arg arm_pitch) $(arg arm_yaw)"/>
-</xacro:tiago_sea_arm>
-<xacro:tiago_sea_arm name="arm_right" parent="torso_lift_link" reflect="1" arm_1_offset="0" arm_2_offset="0" arm_3_offset="0" arm_4_offset="0" arm_5_offset="0" arm_6_offset="0" arm_7_offset="0">
+</xacro:tiago_v2_arm>
+<xacro:tiago_v2_arm name="arm_right" parent="torso_lift_link" reflect="1" arm_1_offset="0" arm_2_offset="0" arm_3_offset="0" arm_4_offset="0" arm_5_offset="0" arm_6_offset="0" arm_7_offset="0">
   <origin xyz="$(arg arm_x) ${-1.0*$(arg arm_y)} $(arg arm_z)"
 	  rpy="$(arg arm_roll) ${-1.0*$(arg arm_pitch)} ${-3.14159 -$(arg arm_yaw)}"/>
-</xacro:tiago_sea_arm>
+</xacro:tiago_v2_arm>
 </robot>

Commit message: both arms fixed and tool link added

File: tiago_v2_prototype_description/robots/tiago_v2_prototype.urdf.xacro (robot description, xacro)
@@ -14,5 +14,5 @@
 <robot  xmlns:xacro="http://ros.org/wiki/xacro" name="tiago_v2_prototype">
 <!-- Parameters -->
-<xacro:arg name="laser_model" default="sick-571"/> <!-- false, hokuyo, sick-551, sick-561, sick-571-->
+<xacro:arg name="laser_model" default="hokuyo"/> <!-- false, hokuyo, sick-551, sick-561, sick-571-->
 <xacro:property name="laser_model" value="$(arg laser_model)" />
 <!-- Includes -->

File: tiago_v2_prototype_description/urdf/arm/arm.urdf.xacro (robot description, xacro)
@@ -140,5 +140,5 @@
         </geometry>
         <material name="">
-          <color rgba="0.89412 0.91373 0.92941 1" />
+           <color rgba="0.29804 0.29804 0.29804 1" />
         </material>
       </visual>
@@ -184,5 +184,5 @@
         </geometry>
         <material name="">
-          <color rgba="0.89412 0.91373 0.92941 1" />
+           <color rgba="0.29804 0.29804 0.29804 1" />
         </material>
       </visual>
@@ -224,5 +224,5 @@
         </geometry>
         <material name="">
-          <color rgba="0.75294 0.75294 0.75294 1" />
+           <color rgba="0.29804 0.29804 0.29804 1" />
         </material>
       </visual>
@@ -269,5 +269,5 @@
         </geometry>
         <material name="">
-          <color rgba="0.75294 0.75294 0.75294 1" />
+           <color rgba="0.29804 0.29804 0.29804 1" />
         </material>
       </visual>
@@ -291,17 +291,19 @@
     </joint>
     <!-- ARM 7 LINK -->
-<!--
     <link name="${name}_7_link">
-      <inertial>
-        <origin xyz="-4.9961E-13 1.8172E-12 -0.030946" rpy="0 0 0" />
-        <mass value="0.20434" />
-        <inertia
-          ixx="0.00011401"
-          ixy="-2.6547E-15"
-          ixz="-1.9524E-16"
-          iyy="0.00011401"
-          iyz="7.1031E-16"
-          izz="0.00010539" />
-      </inertial>
+       <inertial>
+      <origin
+        xyz="-6.764E-18 -1.4549E-16 0.018549"
+        rpy="0 0 0" />
+      <mass
+        value="0.10189" />
+      <inertia
+        ixx="5.1076E-05"
+        ixy="-1.0899E-21"
+        ixz="-5.93E-21"
+        iyy="5.0882E-05"
+        iyz="-8.5344E-21"
+        izz="9.705E-05" />
+    </inertial>
       <visual>
         <origin xyz="0 0 0" rpy="0 0 0" />
@@ -310,5 +312,5 @@
         </geometry>
         <material name="">
-          <color rgba="0.75294 0.75294 0.75294 1" />
+           <color rgba="0.29804 0.29804 0.29804 1" />
         </material>
       </visual>
@@ -320,9 +322,9 @@
       </collision>
     </link>
-  -->
     <!-- ARM 7 JOINT -->
-<!--
     <joint name="${name}_7_joint" type="revolute">
-      <origin xyz="0 0.135 -0.0431" rpy="1.5708 1.5708 0" />
+      <origin
+      xyz="-0.1166 0 0"
+      rpy="0 -1.5708 0" />
       <parent link="${name}_6_link" />
       <child link="${name}_7_link" />
@@ -330,14 +332,22 @@
       <limit lower="${arm_7_joint_lb}" upper="${arm_7_joint_ub}" effort="${arm_7_max_effort}" velocity="${arm_7_max_velocity}" />
     </joint>
--->
  <!--***********************-->
     <!--        TOOL           -->
     <!--***********************-->
-<!--
     <link name="${name}_tool_link">
-      <inertial>
-        <mass value="0.1" />
-        <inertia ixx="8.33E-07" ixy="0.0" ixz="0.0" iyy="8.33E-07" iyz="0.0" izz="1.25E-06" />
-      </inertial>
+     <inertial>
+      <origin
+        xyz="5.0493E-18 -4.4892E-17 -0.0068514"
+        rpy="0 0 0" />
+      <mass
+        value="0.10189" />
+      <inertia
+        ixx="5.1076E-05"
+        ixy="-1.0374E-21"
+        ixz="-5.9164E-21"
+        iyy="5.0882E-05"
+        iyz="-8.5211E-21"
+        izz="9.705E-05" />
+    </inertial>
       <visual>
         <origin xyz="0.001 0 0" rpy="0 1.5708 0" />
@@ -345,5 +355,7 @@
           <cylinder radius="0.005" length="0.005"/>
         </geometry>
-        <material name="LightGrey" />
+        <material name="">
+          <color rgba="0.29804 0.29804 0.29804 1" />
+        </material>
       </visual>
       <collision>
@@ -357,7 +369,6 @@
       <parent link="${name}_7_link" />
       <child link="${name}_tool_link" />
-        <origin xyz="0 0 -0.07" rpy="3.1415 0 0" />
-    </joint>
-  -->
+        <origin xyz="0 0 0.0254" rpy="3.1415 0 0" />
+    </joint>
     <!-- TRANSMISSIONS -->
     <xacro:arm_simple_transmission name="${name}" number="1" reduction="1.0" offset_value="${arm_1_offset}"/>

File: tiago_v2_prototype_description/urdf/head/head.urdf.xacro (robot description, xacro)
@@ -42,12 +42,14 @@
         <origin xyz="0 0 0" rpy="0 0 0"/>
         <geometry>
-          <mesh filename="package://tiago_v2_prototype_description/meshes/head/head_1_link.stl" scale="1 1 1"/>
+          <mesh filename="package://tiago_v2_prototype_description/meshes/head/head_1_link.STL" scale="1 1 1"/>
         </geometry>
-        <material name="White" />
+        <material name="">
+          <color rgba="0.29804 0.29804 0.29804 1" />
+        </material>
       </visual>
       <collision>
         <origin xyz="0.0 0 0" rpy="0 0 0.0" />
         <geometry>
-          <mesh filename="package://tiago_v2_prototype_description/meshes/head/head_1_link.stl" scale="1 1 1"/>
+          <mesh filename="package://tiago_v2_prototype_description/meshes/head/head_1_link.STL" scale="1 1 1"/>
         </geometry>
         <material name="White" />
@@ -86,12 +88,14 @@
         <origin xyz="0 0 0" rpy="0 0 0" />
         <geometry>
-          <mesh filename="package://tiago_v2_prototype_description/meshes/head/head_2_link.stl" scale="1 1 1"/>
+          <mesh filename="package://tiago_v2_prototype_description/meshes/head/head_2_link.STL" scale="1 1 1"/>
         </geometry>
-        <material name="White" />
+        <material name="">
+          <color rgba="0.29804 0.29804 0.29804 1" />
+        </material>
       </visual>
       <collision>
         <origin xyz="0 0 0" rpy="0 0 0" />
         <geometry>
-          <mesh filename="package://tiago_v2_prototype_description/meshes/head/head_2_link.stl" scale="1 1 1"/>
+          <mesh filename="package://tiago_v2_prototype_description/meshes/head/head_2_link.STL" scale="1 1 1"/>
         </geometry>
       </collision>

File: tiago_v2_prototype_description/urdf/torso/torso_dual.urdf.xacro (robot description, xacro)
@@ -19,15 +19,15 @@
      <inertial>
       <origin
-        xyz="0.0012723 -0.007076 0.14739"
+        xyz="0.0014857 -0.0077054 0.14693"
         rpy="0 0 0" />
       <mass
-        value="15.476" />
+        value="15.527" />
       <inertia
-        ixx="0.179"
-        ixy="0.00019166"
-        ixz="-0.004948"
-        iyy="0.20071"
-        iyz="0.00016524"
-        izz="0.084001" />
+        ixx="0.17904"
+        ixy="0.00019412"
+        ixz="-0.0049479"
+        iyy="0.20082"
+        iyz="0.00015981"
+        izz="0.084141" />
     </inertial>
     <visual>
@@ -39,8 +39,6 @@
           filename="package://tiago_v2_prototype_description/meshes/torso/torso_fixed_link.STL" />
       </geometry>
-      <material
-        name="">
-        <color
-          rgba="0.752941176470588 0.752941176470588 0.752941176470588 1" />
+      <material name="">
+        <color rgba="0.29804 0.29804 0.29804 1" />
       </material>
     </visual>
