Commit message: fixed inertia and joints naming

File: tiago_v2_prototype_description/robots/tiago_v2_prototype.urdf.xacro (robot description, xacro)
@@ -27,15 +27,4 @@
 <xacro:tiago_v2_torso name="torso" parent="base_link"/>
 <xacro:tiago_v2_head name="head" parent="torso_lift_link"/>
-<!--
-<origin
-      xyz="0.10529 0.15915 -0.11927"
-      rpy="-2.0679 0 -1.2217" />
-<xacro:arg name="arm_x" default="0.10529" />
-<xacro:arg name="arm_y" default="0.15915" />
-<xacro:arg name="arm_z" default="-0.11927" />
-<xacro:arg name="arm_roll" default="-2.0679" />
-<xacro:arg name="arm_pitch" default="0.0" />
-<xacro:arg name="arm_yaw" default="-1.2217" />
--->
 <xacro:arg name="arm_x" default="0.08976" />
 <xacro:arg name="arm_y" default="0.15918" />

File: tiago_v2_prototype_description/urdf/arm/arm.urdf.xacro (robot description, xacro)
@@ -39,17 +39,10 @@
     <link name="${name}_1_link">
       <inertial>
-      <origin
-        xyz="0.0023924 0.015901 0.1545"
-        rpy="0 0 0" />
-      <mass
-        value="1.0815" />
-      <inertia
-        ixx="0.0024428"
-        ixy="2.3301E-05"
-        ixz="5.9516E-05"
-        iyy="0.0023092"
-        iyz="-0.00020371"
-        izz="0.00092851" />
-    </inertial>
+        <origin xyz="0.0023924 0.015901 0.1545" rpy="0 0 0" />
+        <mass value="1.0815" />
+        <inertia ixx="0.0024428" ixy="2.3301E-05" ixz="5.9516E-05"
+                 iyy="0.0023092" iyz="-0.00020371"
+                 izz="0.00092851" />
+      </inertial>
       <visual>
         <origin xyz="0 0 0" rpy="0 0 0" />
@@ -78,18 +71,11 @@
     <!-- ARM 2 LINK -->
     <link name="${name}_2_link">
-       <inertial>
-      <origin
-        xyz="-0.11649 -0.017864 0.0053781"
-        rpy="0 0 0" />
-      <mass
-        value="0.99205" />
-      <inertia
-        ixx="0.00077291"
-        ixy="-0.00011001"
-        ixz="-0.00016133"
-        iyy="0.0014605"
-        iyz="-1.3237E-05"
-        izz="0.0015605" />
-    </inertial>
+      <inertial>
+        <origin xyz="-0.11649 -0.017864 0.0053781" rpy="0 0 0" />
+        <mass value="0.99205" />
+        <inertia ixx="0.00077291" ixy="-0.00011001" ixz="-0.00016133"
+                 iyy="0.0014605" iyz="-1.3237E-05"
+                 izz="0.0015605" />
+      </inertial>
       <visual>
         <origin xyz="0 0 0" rpy="0 0 0" />
@@ -110,10 +96,8 @@
     <!-- ARM 2 JOINT -->
     <joint name="${name}_2_joint" type="revolute">
-      <origin
-      xyz="0.0 0.02 0.18"
-      rpy="0 1.5708 0" />
+      <origin xyz="0.0 0.02 0.18" rpy="0 1.5708 0" />
       <parent link="${name}_1_link" />
       <child link="${name}_2_link" />
-      <axis xyz="0 0 -1" />
+      <axis xyz="0 0 1" />
       <limit lower="${arm_2_joint_lb}" upper="${arm_2_joint_ub}" effort="${arm_2_max_effort}" velocity="${arm_2_max_velocity}" />
     </joint>
@@ -121,17 +105,10 @@
     <link name="${name}_3_link">
       <inertial>
-      <origin
-        xyz="0.0023924 0.015901 0.1545"
-        rpy="0 0 0" />
-      <mass
-        value="1.0815" />
-      <inertia
-        ixx="0.0024428"
-        ixy="2.3301E-05"
-        ixz="5.9516E-05"
-        iyy="0.0023092"
-        iyz="-0.00020371"
-        izz="0.00092851" />
-    </inertial>
+        <origin xyz="0.0023924 0.015901 0.1545" rpy="0 0 0" />
+        <mass value="1.0816" />
+        <inertia ixx="0.0024426" ixy="2.3307E-05" ixz="5.9333E-05"
+                 iyy="0.0023089" iyz="-0.00020369"
+                 izz="0.00092843" />
+      </inertial>
       <visual>
         <origin xyz="0 0 0" rpy="0 0 0" />
@@ -152,6 +129,4 @@
     <!-- ARM 3 JOINT -->
     <joint name="${name}_3_joint" type="revolute">
-      <!-- <origin xyz="-0.02 0.16991 -0.04491"
-           rpy="${reflect * 1.5707} 1.5707 ${(reflect + 1) * 0.5 * 3.1415}" /> -->
       <origin
       xyz="-0.15 -0.02 0"
@@ -165,17 +140,17 @@
     <link name="${name}_4_link">
       <inertial>
-      <origin
-        xyz="-0.11649 -0.017864 0.0053781"
-        rpy="0 0 0" />
-      <mass
-        value="0.99205" />
-      <inertia
-        ixx="0.00077291"
-        ixy="-0.00011001"
-        ixz="-0.00016133"
-        iyy="0.0014605"
-        iyz="-1.3237E-05"
-        izz="0.0015605" />
-    </inertial>
+        <origin
+          xyz="-0.11649 -0.017864 0.0053781"
+          rpy="0 0 0" />
+        <mass
+          value="0.99204" />
+        <inertia
+          ixx="0.00077294"
+          ixy="-0.00011001"
+          ixz="-0.00016136"
+          iyy="0.0014605"
+          iyz="-1.3224E-05"
+          izz="0.0015605" />
+      </inertial>
       <visual>
         <origin xyz="0 0 0" rpy="0 0 0" />
@@ -196,8 +171,5 @@
     <!-- ARM 4 JOINT -->
     <joint name="${name}_4_joint" type="revolute">
-      <!--<origin xyz="-0.04491 -0.02 0.16009" rpy="1.5708 0 -1.5708" />-->
-     <origin
-      xyz="0 0.02 0.18"
-      rpy="0 1.5708 0" />
+      <origin xyz="0 0.02 0.18" rpy="0 1.5708 0" />
       <parent link="${name}_3_link" />
       <child link="${name}_4_link" />
@@ -208,13 +180,9 @@
     <link name="${name}_5_link">
       <inertial>
-        <origin xyz="-0.0034877 0.0007088 0.10161" rpy="0 0 0" />
-        <mass value="0.65" /> <!--1.3606-->
-        <inertia
-          ixx="0.0042327"
-          ixy="-1.4778E-06"
-          ixz="-0.00015838"
-          iyy="0.0039855"
-          iyz="-6.3812E-05"
-          izz="0.00090574" />
+        <origin xyz="0.0004859 0.00014289 0.129" rpy="0 0 0" />
+        <mass value="0.52538" />
+        <inertia ixx="0.0019111" ixy="-1.4245E-08" ixz="3.8663E-05"
+                 iyy="0.0018565" iyz="1.1356E-06"
+                 izz="0.00046496" />
       </inertial>
       <visual>
@@ -236,10 +204,5 @@
     <!-- ARM 5 JOINT -->
     <joint name="${name}_5_joint" type="revolute">
-    <!--
-      <origin xyz="-0.02 0.16991 -0.04491" rpy="-1.5708 1.5707 0" />
-    -->
-      <origin
-      xyz="-0.15 -0.02 0"
-      rpy="0 -1.5708 0" />
+      <origin xyz="-0.15 -0.02 0" rpy="0 -1.5708 0" />
       <parent link="${name}_4_link" />
       <child link="${name}_5_link" />
@@ -251,15 +214,15 @@
       <inertial>
         <origin
-        xyz="-0.0868246191017208 -7.20863653169701E-06 0.00452526175178974"
+        xyz="-0.086822 -7.7905E-06 0.0045258"
         rpy="0 0 0" />
-      <mass
-        value="0.667219281811054" />
-      <inertia
-        ixx="0.000356949168188171"
-        ixy="1.64330351077636E-07"
-        ixz="-9.5157761444025E-05"
-        iyy="0.000738465753656827"
-        iyz="1.21140041540438E-10"
-        izz="0.000753196424392043" />
+        <mass
+          value="0.66725" />
+        <inertia
+          ixx="0.00035696"
+          ixy="1.6019E-07"
+          ixz="-9.5191E-05"
+          iyy="0.00073846"
+          iyz="2.118E-08"
+          izz="0.00075321" />
       </inertial>
       <visual>
@@ -281,8 +244,5 @@
     <!-- ARM 6 JOINT -->
     <joint name="${name}_6_joint" type="revolute">
-      <!-- <origin xyz="-0.0431 0 0.16509" rpy="1.5708 0 -1.5708" /> -->
-      <origin
-      xyz="0 0 0.185"
-      rpy="1.4161 1.5708 1.4127" />
+      <origin xyz="0 0 0.185" rpy="0 1.5708 0" />
       <parent link="${name}_5_link" />
       <child link="${name}_6_link" />
@@ -378,6 +338,5 @@
     <xacro:arm_simple_transmission name="${name}" number="5" reduction="1.0" offset_value="${arm_5_offset}"/>
     <xacro:arm_simple_transmission name="${name}" number="6" reduction="1.0" offset_value="${arm_6_offset}"/>
-<!--<xacro:arm_simple_transmission name="${name}" number="7" reduction="1.0" offset_value="${arm_7_offset}"/>
--->
+    <xacro:arm_simple_transmission name="${name}" number="7" reduction="1.0" offset_value="${arm_7_offset}"/>
   </xacro:macro>
 </robot>

File: tiago_v2_prototype_description/urdf/head/head.urdf.xacro (robot description, xacro)
@@ -33,9 +33,13 @@
     <link name="${name}_1_link">
       <inertial>
-        <origin xyz="-0.00508 0.00237 0.07229" rpy="0.00000 0.00000 0.00000"/>
-        <mass value="0.62220"/>
-        <inertia ixx="0.00119200000" ixy="-0.00000700000" ixz="0.00009600000"
-                 iyy="0.00140200000" iyz="0.00000400000"
-                 izz="0.00088900000"/>
+        <origin xyz="0.013723 0.0015288 0.091095" rpy="0 0 0" />
+        <mass value="0.50253" />
+        <inertia
+          ixx="0.00073252"
+          ixy="-1.0801E-06"
+          ixz="-6.3715E-05"
+          iyy="0.0005861"
+          iyz="4.157E-10"
+          izz="0.00060232" />
       </inertial>
       <visual>
@@ -79,9 +83,9 @@
     <link name="${name}_2_link">
       <inertial>
-        <origin xyz="0.04700 0.05542 0.00022" rpy="0.00000 0.00000 0.00000"/>
-        <mass value="0.66123"/>
-        <inertia ixx="0.00462000000" ixy="0.00068900000" ixz="0.00000600000"
-                 iyy="0.00486100000" iyz="0.00000600000"
-                 izz="0.00313200000"/>
+        <origin xyz="0.0025967 0.11474 0.00021233" rpy="0 0 0" />
+        <mass value="1.2093"/>
+        <inertia ixx="0.0063697" ixy="0.00052067" ixz="-8.4666E-06"
+                 iyy="0.0045958" iyz="9.6501E-06"
+                 izz="0.0031995" />
       </inertial>
       <visual>

File: tiago_v2_prototype_description/urdf/torso/torso_dual.urdf.xacro (robot description, xacro)
@@ -17,17 +17,10 @@
   <!-- Bottom fixed part of column -->
   <link name="${name}_fixed_link">
-     <inertial>
-      <origin
-        xyz="0.0014857 -0.0077054 0.14693"
-        rpy="0 0 0" />
+    <inertial>
+      <origin  xyz="0.0014857 -0.0077054 0.14693" rpy="0 0 0" />
       <mass
         value="15.527" />
-      <inertia
-        ixx="0.17904"
-        ixy="0.00019412"
-        ixz="-0.0049479"
-        iyy="0.20082"
-        iyz="0.00015981"
-        izz="0.084141" />
+      <inertia ixx="0.17904" ixy="0.00019412" ixz="-0.0049479"
+               iyy="0.20082" iyz="0.00015981" izz="0.084141" />
     </inertial>
     <visual>
@@ -96,15 +89,15 @@
     <inertial>
       <origin
-        xyz="0.0072742 0.015983 -0.19528"
+        xyz="0.0014742 0.0065278 -0.20301"
         rpy="0 0 0" />
       <mass
-        value="10.027" />
+        value="9.547" />
       <inertia
-        ixx="0.042393"
-        ixy="5.0892E-05"
-        ixz="0.00016162"
-        iyy="0.031426"
-        iyz="-4.1547E-05"
-        izz="0.018869" />
+        ixx="0.042078"
+        ixy="5.6766E-05"
+        ixz="0.00014731"
+        iyy="0.031115"
+        iyz="-5.0165E-05"
+        izz="0.018659" />
     </inertial>
     <visual>

Commit message: grippers robotiq-2f-85 added for both arms

File: tiago_v2_prototype_description/robots/tiago_v2_prototype.urdf.xacro (robot description, xacro)
@@ -22,4 +22,11 @@
 <xacro:include filename="$(find omni_base_description)/urdf/base/base_sensors.urdf.xacro" />
 <xacro:include filename="$(find tiago_v2_prototype_description)/urdf/arm/arm.urdf.xacro" />
+<xacro:include filename="$(find tiago_v2_prototype_description)/urdf/end_effector/end_effector.urdf.xacro" />
+<!-- End effector -->
+<xacro:arg name="end_effector" default="robotiq-2f-85"/> <!-- for now only robotiq-2f-85 is available -->
+<xacro:property name="end_effector" value="$(arg end_effector)" />
+<xacro:property name="end_effector_name" value="gripper"/>
+<xacro:property name="end_effector_left_link" value="arm_left_tool_link"/>
+<xacro:property name="end_effector_right_link" value="arm_right_tool_link"/>
 <!-- Base -->
 <xacro:base_sensors name="base" front_laser_model="$(arg laser_model)" rear_laser_model="$(arg laser_model)"/>
@@ -42,3 +49,5 @@
 	  rpy="$(arg arm_roll) ${-1.0*$(arg arm_pitch)} ${-3.14159 -$(arg arm_yaw)}"/>
 </xacro:tiago_v2_arm>
+ <xacro:tiago_v2_prototype_end_effector name="${end_effector_name}_left" parent="${end_effector_left_link}" type="${end_effector}"/>
+ <xacro:tiago_v2_prototype_end_effector name="${end_effector_name}_right" parent="${end_effector_right_link}" type="${end_effector}"/>
 </robot>
