Commit message: Cleaning and simplification of collision meshes

File: tiago_v2_prototype_description/urdf/arm/arm.urdf.xacro (robot description, xacro)
@@ -49,5 +49,5 @@
         <geometry>
           <mesh
-            filename="package://tiago_v2_prototype_description/meshes/arm/arm_1_link.STL" />
+            filename="package://tiago_v2_prototype_description/meshes/arm/arm_1_link.stl" />
         </geometry>
         <material name="">
@@ -58,5 +58,5 @@
         <origin xyz="0 0 0" rpy="0 0 0" />
         <geometry>
-          <mesh filename="package://tiago_v2_prototype_description/meshes/arm/arm_1_link.STL" />
+          <mesh filename="package://tiago_v2_prototype_description/meshes/arm/arm_1_link_collision.stl" />
         </geometry>
       </collision>
@@ -81,5 +81,5 @@
         <origin xyz="0 0 0" rpy="0 0 0" />
         <geometry>
-          <mesh filename="package://tiago_v2_prototype_description/meshes/arm/arm_2_link.STL" />
+          <mesh filename="package://tiago_v2_prototype_description/meshes/arm/arm_2_link.stl" />
         </geometry>
         <material name="">
@@ -90,5 +90,5 @@
         <origin xyz="0 0 0" rpy="0 0 0" />
         <geometry>
-          <mesh filename="package://tiago_v2_prototype_description/meshes/arm/arm_2_link.STL" />
+          <mesh filename="package://tiago_v2_prototype_description/meshes/arm/arm_2_link_collision.stl" />
         </geometry>
       </collision>
@@ -114,14 +114,14 @@
         <origin xyz="0 0 0" rpy="0 0 0" />
         <geometry>
-          <mesh filename="package://tiago_v2_prototype_description/meshes/arm/arm_3_link.STL" />
-        </geometry>
-        <material name="">
-           <color rgba="0.29804 0.29804 0.29804 1" />
-        </material>
-      </visual>
-      <collision>
-        <origin xyz="0 0 0" rpy="0 0 0" />
-        <geometry>
-          <mesh filename="package://tiago_v2_prototype_description/meshes/arm/arm_3_link.STL" />
+          <mesh filename="package://tiago_v2_prototype_description/meshes/arm/arm_3_link.stl" />
+        </geometry>
+        <material name="">
+           <color rgba="0.29804 0.29804 0.29804 1" />
+        </material>
+      </visual>
+      <collision>
+        <origin xyz="0 0 0" rpy="0 0 0" />
+        <geometry>
+          <mesh filename="package://tiago_v2_prototype_description/meshes/arm/arm_3_link_collision.stl" />
         </geometry>
       </collision>
@@ -156,14 +156,14 @@
         <origin xyz="0 0 0" rpy="0 0 0" />
         <geometry>
-          <mesh filename="package://tiago_v2_prototype_description/meshes/arm/arm_4_link.STL" />
-        </geometry>
-        <material name="">
-           <color rgba="0.29804 0.29804 0.29804 1" />
-        </material>
-      </visual>
-      <collision>
-        <origin xyz="0 0 0" rpy="0 0 0" />
-        <geometry>
-          <mesh filename="package://tiago_v2_prototype_description/meshes/arm/arm_4_link.STL" />
+          <mesh filename="package://tiago_v2_prototype_description/meshes/arm/arm_4_link.stl" />
+        </geometry>
+        <material name="">
+           <color rgba="0.29804 0.29804 0.29804 1" />
+        </material>
+      </visual>
+      <collision>
+        <origin xyz="0 0 0" rpy="0 0 0" />
+        <geometry>
+          <mesh filename="package://tiago_v2_prototype_description/meshes/arm/arm_4_link_collision.stl" />
         </geometry>
       </collision>
@@ -189,14 +189,14 @@
         <origin xyz="0 0 0" rpy="0 0 0" />
         <geometry>
-          <mesh filename="package://tiago_v2_prototype_description/meshes/arm/arm_5_link.STL" />
-        </geometry>
-        <material name="">
-           <color rgba="0.29804 0.29804 0.29804 1" />
-        </material>
-      </visual>
-      <collision>
-        <origin xyz="0 0 0" rpy="0 0 0" />
-        <geometry>
-          <mesh filename="package://tiago_v2_prototype_description/meshes/arm/arm_5_link.STL" />
+          <mesh filename="package://tiago_v2_prototype_description/meshes/arm/arm_5_link.stl" />
+        </geometry>
+        <material name="">
+           <color rgba="0.29804 0.29804 0.29804 1" />
+        </material>
+      </visual>
+      <collision>
+        <origin xyz="0 0 0" rpy="0 0 0" />
+        <geometry>
+          <mesh filename="package://tiago_v2_prototype_description/meshes/arm/arm_5_link_collision.stl" />
         </geometry>
       </collision>
@@ -229,14 +229,14 @@
         <origin xyz="0 0 0" rpy="0 0 0" />
         <geometry>
-          <mesh filename="package://tiago_v2_prototype_description/meshes/arm/arm_6_link.STL" />
-        </geometry>
-        <material name="">
-           <color rgba="0.29804 0.29804 0.29804 1" />
-        </material>
-      </visual>
-      <collision>
-        <origin xyz="0 0 0" rpy="0 0 0" />
-        <geometry>
-          <mesh filename="package://tiago_v2_prototype_description/meshes/arm/arm_6_link.STL" />
+          <mesh filename="package://tiago_v2_prototype_description/meshes/arm/arm_6_link.stl" />
+        </geometry>
+        <material name="">
+           <color rgba="0.29804 0.29804 0.29804 1" />
+        </material>
+      </visual>
+      <collision>
+        <origin xyz="0 0 0" rpy="0 0 0" />
+        <geometry>
+          <mesh filename="package://tiago_v2_prototype_description/meshes/arm/arm_6_link_collision.stl" />
         </geometry>
       </collision>
@@ -269,14 +269,14 @@
         <origin xyz="0 0 0" rpy="0 0 0" />
         <geometry>
-          <mesh filename="package://tiago_v2_prototype_description/meshes/arm/arm_7_link.STL" />
-        </geometry>
-        <material name="">
-           <color rgba="0.29804 0.29804 0.29804 1" />
-        </material>
-      </visual>
-      <collision>
-        <origin xyz="0 0 0" rpy="0 0 0" />
-        <geometry>
-          <mesh filename="package://tiago_v2_prototype_description/meshes/arm/arm_7_link.STL" />
+          <mesh filename="package://tiago_v2_prototype_description/meshes/arm/arm_7_link.stl" />
+        </geometry>
+        <material name="">
+           <color rgba="0.29804 0.29804 0.29804 1" />
+        </material>
+      </visual>
+      <collision>
+        <origin xyz="0 0 0" rpy="0 0 0" />
+        <geometry>
+          <mesh filename="package://tiago_v2_prototype_description/meshes/arm/arm_7_link_collision.stl" />
         </geometry>
       </collision>

File: tiago_v2_prototype_description/urdf/head/head.urdf.xacro (robot description, xacro)
@@ -46,5 +46,5 @@
         <origin xyz="0 0 0" rpy="0 0 0"/>
         <geometry>
-          <mesh filename="package://tiago_v2_prototype_description/meshes/head/head_1_link.STL" scale="1 1 1"/>
+          <mesh filename="package://tiago_v2_prototype_description/meshes/head/head_1_link.stl" scale="1 1 1"/>
         </geometry>
         <material name="">
@@ -55,5 +55,5 @@
         <origin xyz="0.0 0 0" rpy="0 0 0.0" />
         <geometry>
-          <mesh filename="package://tiago_v2_prototype_description/meshes/head/head_1_link.STL" scale="1 1 1"/>
+          <mesh filename="package://tiago_v2_prototype_description/meshes/head/head_1_link_collision.stl" scale="1 1 1"/>
         </geometry>
         <material name="White" />
@@ -92,5 +92,5 @@
         <origin xyz="0 0 0" rpy="0 0 0" />
         <geometry>
-          <mesh filename="package://tiago_v2_prototype_description/meshes/head/head_2_link.STL" scale="1 1 1"/>
+          <mesh filename="package://tiago_v2_prototype_description/meshes/head/head_2_link.stl" scale="1 1 1"/>
         </geometry>
         <material name="">
@@ -101,5 +101,5 @@
         <origin xyz="0 0 0" rpy="0 0 0" />
         <geometry>
-          <mesh filename="package://tiago_v2_prototype_description/meshes/head/head_2_link.STL" scale="1 1 1"/>
+          <mesh filename="package://tiago_v2_prototype_description/meshes/head/head_2_link_collision.stl" scale="1 1 1"/>
         </geometry>
       </collision>

File: tiago_v2_prototype_description/urdf/torso/torso_dual.urdf.xacro (robot description, xacro)
@@ -30,5 +30,5 @@
       <geometry>
         <mesh
-          filename="package://tiago_v2_prototype_description/meshes/torso/torso_fixed_link.STL" />
+          filename="package://tiago_v2_prototype_description/meshes/torso/torso_fixed_link.stl" />
       </geometry>
       <material name="">
@@ -37,11 +37,31 @@
     </visual>
     <collision>
-      <origin
+   <!--   <origin
         xyz="0 0 0"
         rpy="0 0 0" />
       <geometry>
         <mesh
-          filename="package://tiago_v2_prototype_description/meshes/torso/torso_fixed_link.STL" />
+          filename="package://tiago_v2_prototype_description/meshes/torso/torso_fixed_link.stl" />
       </geometry>
+   -->
+      <origin rpy="0 0 0" xyz="0 0 0.1" />
+      <geometry>
+        <box size="0.23 0.253 0.2"/>
+      </geometry>
+      <material name="DarkGrey"/>
+    </collision>
+    <collision>
+      <origin rpy="0 0 0" xyz="0.18 0 0.03" />
+      <geometry>
+        <box size="0.15 0.253 0.06"/>
+      </geometry>
+      <material name="DarkGrey"/>
+    </collision>
+     <collision>
+      <origin rpy="0 0 0" xyz="-0.09 0 0.0" />
+      <geometry>
+        <box size="0.47 0.5 0.02"/>
+      </geometry>
+      <material name="DarkGrey"/>
     </collision>
   </link>
@@ -107,5 +127,5 @@
       <geometry>
         <mesh
-          filename="package://tiago_v2_prototype_description/meshes/torso/torso_lift_link.STL" />
+          filename="package://tiago_v2_prototype_description/meshes/torso/torso_lift_link.stl" />
       </geometry>
       <material
@@ -121,5 +141,5 @@
       <geometry>
         <mesh
-          filename="package://tiago_v2_prototype_description/meshes/torso/torso_lift_link.STL" />
+          filename="package://tiago_v2_prototype_description/meshes/torso/torso_lift_link_collision.stl" />
       </geometry>
     </collision>

Commit message: Added gazebo flags for joint and reformat dynamic parameters for ars, head and torso

File: tiago_v2_prototype_description/urdf/arm/arm.urdf.xacro (robot description, xacro)
@@ -39,9 +39,16 @@
     <link name="${name}_1_link">
       <inertial>
-        <origin xyz="0.0023924 0.015901 0.1545" rpy="0 0 0" />
-        <mass value="1.0815" />
-        <inertia ixx="0.0024428" ixy="2.3301E-05" ixz="5.9516E-05"
-                 iyy="0.0023092" iyz="-0.00020371"
-                 izz="0.00092851" />
+        <origin
+          xyz="0.0023908 0.015901 0.1545"
+          rpy="0 0 0" />
+        <mass
+          value="1.0816" />
+        <inertia
+          ixx="0.0024426"
+          ixy="2.3307E-05"
+          ixz="5.9333E-05"
+          iyy="0.0023089"
+          iyz="-0.00020369"
+          izz="0.00092843" />
       </inertial>
       <visual>
@@ -72,9 +79,16 @@
     <link name="${name}_2_link">
       <inertial>
-        <origin xyz="-0.11649 -0.017864 0.0053781" rpy="0 0 0" />
-        <mass value="0.99205" />
-        <inertia ixx="0.00077291" ixy="-0.00011001" ixz="-0.00016133"
-                 iyy="0.0014605" iyz="-1.3237E-05"
-                 izz="0.0015605" />
+        <origin
+          xyz="-0.11649 -0.017864 0.0053772"
+          rpy="0 0 0" />
+        <mass
+          value="0.99204" />
+        <inertia
+          ixx="0.00077294"
+          ixy="-0.00011001"
+          ixz="-0.00016136"
+          iyy="0.0014605"
+          iyz="-1.3224E-05"
+          izz="0.0015605" />
       </inertial>
       <visual>
@@ -105,9 +119,16 @@
     <link name="${name}_3_link">
       <inertial>
-        <origin xyz="0.0023924 0.015901 0.1545" rpy="0 0 0" />
-        <mass value="1.0816" />
-        <inertia ixx="0.0024426" ixy="2.3307E-05" ixz="5.9333E-05"
-                 iyy="0.0023089" iyz="-0.00020369"
-                 izz="0.00092843" />
+        <origin
+          xyz="0.0023908 0.015901 0.1545"
+          rpy="0 0 0" />
+        <mass
+          value="1.0816" />
+        <inertia
+          ixx="0.0024426"
+          ixy="2.3307E-05"
+          ixz="5.9333E-05"
+          iyy="0.0023089"
+          iyz="-0.00020369"
+          izz="0.00092843" />
       </inertial>
       <visual>
@@ -141,5 +162,5 @@
       <inertial>
         <origin
-          xyz="-0.11649 -0.017864 0.0053781"
+          xyz="-0.11649 -0.017864 0.0053772"
           rpy="0 0 0" />
         <mass
@@ -180,9 +201,16 @@
     <link name="${name}_5_link">
       <inertial>
-        <origin xyz="0.0004859 0.00014289 0.129" rpy="0 0 0" />
-        <mass value="0.52538" />
-        <inertia ixx="0.0019111" ixy="-1.4245E-08" ixz="3.8663E-05"
-                 iyy="0.0018565" iyz="1.1356E-06"
-                 izz="0.00046496" />
+        <origin
+          xyz="0.0004859 0.00014289 0.129"
+          rpy="0 0 0" />
+        <mass
+          value="0.52538" />
+        <inertia
+          ixx="0.0019111"
+          ixy="-1.4245E-08"
+          ixz="3.8663E-05"
+          iyy="0.0018565"
+          iyz="1.1356E-06"
+          izz="0.00046496" />
       </inertial>
       <visual>
@@ -214,6 +242,6 @@
       <inertial>
         <origin
-        xyz="-0.086822 -7.7905E-06 0.0045258"
-        rpy="0 0 0" />
+          xyz="-0.086822 -7.7905E-06 0.0045258"
+          rpy="0 0 0" />
         <mass
           value="0.66725" />
@@ -252,18 +280,18 @@
     <!-- ARM 7 LINK -->
     <link name="${name}_7_link">
-       <inertial>
-      <origin
-        xyz="-6.764E-18 -1.4549E-16 0.018549"
-        rpy="0 0 0" />
-      <mass
-        value="0.10189" />
-      <inertia
-        ixx="5.1076E-05"
-        ixy="-1.0899E-21"
-        ixz="-5.93E-21"
-        iyy="5.0882E-05"
-        iyz="-8.5344E-21"
-        izz="9.705E-05" />
-    </inertial>
+      <inertial>
+        <origin
+          xyz="-6.764E-18 -1.4549E-16 0.018549"
+          rpy="0 0 0" />
+        <mass
+          value="0.10189" />
+        <inertia
+          ixx="5.1076E-05"
+          ixy="-1.0899E-21"
+          ixz="-5.93E-21"
+          iyy="5.0882E-05"
+          iyz="-8.5344E-21"
+          izz="9.705E-05" />
+      </inertial>
       <visual>
         <origin xyz="0 0 0" rpy="0 0 0" />
@@ -292,4 +320,53 @@
       <limit lower="${arm_7_joint_lb}" upper="${arm_7_joint_ub}" effort="${arm_7_max_effort}" velocity="${arm_7_max_velocity}" />
     </joint>
+   <gazebo reference="${name}_1_link">
+     <mu1>0.9</mu1>
+     <mu2>0.9</mu2>
+   </gazebo>
+   <gazebo reference="${name}_2_link">
+     <mu1>0.9</mu1>
+     <mu2>0.9</mu2>
+   </gazebo>
+   <gazebo reference="${name}_3_link">
+     <mu1>0.9</mu1>
+     <mu2>0.9</mu2>
+   </gazebo>
+   <gazebo reference="${name}_4_link">
+     <mu1>0.9</mu1>
+     <mu2>0.9</mu2>
+   </gazebo>
+   <gazebo reference="${name}_5_link">
+     <mu1>0.9</mu1>
+     <mu2>0.9</mu2>
+   </gazebo>
+   <gazebo reference="${name}_6_link">
+     <mu1>0.9</mu1>
+     <mu2>0.9</mu2>
+   </gazebo>
+   <gazebo reference="${name}_7_link">
+     <mu1>0.9</mu1>
+     <mu2>0.9</mu2>
+   </gazebo>
+   <gazebo reference="${name}_1_joint">
+      <implicitSpringDamper>1</implicitSpringDamper>
+   </gazebo>
+   <gazebo reference="${name}_2_joint">
+      <implicitSpringDamper>1</implicitSpringDamper>
+   </gazebo>
+   <gazebo reference="${name}_3_joint">
+      <implicitSpringDamper>1</implicitSpringDamper>
+   </gazebo>
+   <gazebo reference="${name}_4_joint">
+      <implicitSpringDamper>1</implicitSpringDamper>
+   </gazebo>
+   <gazebo reference="${name}_5_joint">
+      <implicitSpringDamper>1</implicitSpringDamper>
+   </gazebo>
+   <gazebo reference="${name}_6_joint">
+      <implicitSpringDamper>1</implicitSpringDamper>
+   </gazebo>
+   <gazebo reference="${name}_7_joint">
+      <implicitSpringDamper>1</implicitSpringDamper>
+   </gazebo>
  <!--***********************-->
     <!--        TOOL           -->

File: tiago_v2_prototype_description/urdf/head/head.urdf.xacro (robot description, xacro)
@@ -34,14 +34,15 @@
       <inertial>
         <origin
-          xyz="0.0151529168350566 0.00114213181417127 0.0915264960362224"
+          xyz="0.013723 0.0015288 0.091095"
           rpy="0 0 0" />
-        <mass value="0.5232442430173" />
+        <mass
+          value="0.50253" />
         <inertia
-          ixx="0.000735269995053842"
-          ixy="-1.08043527376587E-06"
-          ixz="-6.37152476586251E-05"
-          iyy="0.000591525160132652"
-          iyz="-7.68106728600967E-12"
-          izz="0.000605065517138752" />
+          ixx="0.00073252"
+          ixy="-1.0801E-06"
+          ixz="-6.3715E-05"
+          iyy="0.0005861"
+          iyz="4.157E-10"
+          izz="0.00060232" />
       </inertial>
       <visual>
@@ -73,11 +74,4 @@
                          soft_upper_limit="${head_1_upper_limit * deg_to_rad - head_eps}" />
     </joint>
-    <gazebo reference="${name}_1_link">
-      <mu1>0.9</mu1>
-      <mu2>0.9</mu2>
-    </gazebo>
-    <gazebo reference="${name}_1_joint">
-       <implicitSpringDamper>1</implicitSpringDamper>
-    </gazebo>
     <!-- extensions -->
     <xacro:head_transmission name="${name}_1" reduction="1" offset_value="${head_1_joint_offset}"/>
@@ -85,15 +79,15 @@
       <inertial>
         <origin
-          xyz="0.00277337961585723 0.115101831131133 4.87500103012104E-05"
+          xyz="0.0025967 0.11474 0.00021233"
           rpy="0 0 0" />
         <mass
-          value="1.24570092574607" />
+          value="1.2093" />
         <inertia
-          ixx="0.00635908800181593"
-          ixy="0.000520891211224051"
-          ixz="-8.48824527287752E-06"
-          iyy="0.00458972596146156"
-          iyz="9.69834634769094E-06"
-          izz="0.00320064764172765" />
+          ixx="0.0063697"
+          ixy="0.00052067"
+          ixz="-8.4666E-06"
+          iyy="0.0045958"
+          iyz="9.6501E-06"
+          izz="0.0031995" />
       </inertial>
       <visual>
@@ -127,4 +121,18 @@
     </joint>
     <xacro:head_transmission name="${name}_2" reduction="1" offset_value="${head_2_joint_offset}"/>
+    <gazebo reference="${name}_1_link">
+      <mu1>0.9</mu1>
+      <mu2>0.9</mu2>
+    </gazebo>
+    <gazebo reference="${name}_2_link">
+      <mu1>0.9</mu1>
+      <mu2>0.9</mu2>
+    </gazebo>
+    <gazebo reference="${name}_1_joint">
+       <implicitSpringDamper>1</implicitSpringDamper>
+    </gazebo>
+    <gazebo reference="${name}_2_joint">
+       <implicitSpringDamper>1</implicitSpringDamper>
+    </gazebo>
   </xacro:macro>
 </robot>

File: tiago_v2_prototype_description/urdf/torso/torso_dual.urdf.xacro (robot description, xacro)
@@ -37,12 +37,4 @@
     </visual>
     <collision>
-   <!--   <origin
-        xyz="0 0 0"
-        rpy="0 0 0" />
-      <geometry>
-        <mesh
-          filename="package://tiago_v2_prototype_description/meshes/torso/torso_fixed_link.stl" />
-      </geometry>
-   -->
       <origin rpy="0 0 0" xyz="0 0 0.1" />
       <geometry>
@@ -58,5 +50,5 @@
       <material name="DarkGrey"/>
     </collision>
-     <collision>
+    <collision>
       <origin rpy="0 0 0" xyz="-0.09 0 0.0" />
       <geometry>
@@ -72,5 +64,5 @@
     <axis xyz="0 0 0" />
   </joint>
- <!-- Middle extending  -->
+  <!-- Middle extending  -->
   <link name="${name}_fixed_column_link">
     <inertial>
@@ -159,4 +151,7 @@
   </joint>
   <xacro:torso_simple_transmission name="torso_lift" reduction="1.0"/>
- </xacro:macro>
+  <gazebo reference="${name}_lift_joint">
+     <implicitSpringDamper>1</implicitSpringDamper>
+  </gazebo>
+  </xacro:macro>
 </robot>
