Commit message: update joint position limtis

File: tiago_v2_prototype_description/urdf/arm/arm.limits.xacro (robot description, xacro)
@@ -15,10 +15,10 @@
   <xacro:property name="arm_1_joint_ub" value="2.6" />
   <xacro:property name="arm_1_joint_lb" value="-2.6" />
-  <xacro:property name="arm_2_joint_ub" value="2.45" />
-  <xacro:property name="arm_2_joint_lb" value="-1.05" />
+  <xacro:property name="arm_2_joint_ub" value="2.44" />
+  <xacro:property name="arm_2_joint_lb" value="-1.10" />
   <xacro:property name="arm_3_joint_ub" value="2.6" />
   <xacro:property name="arm_3_joint_lb" value="-2.6" />
-  <xacro:property name="arm_4_joint_ub" value="2.45" />
-  <xacro:property name="arm_4_joint_lb" value="-1.05" />
+  <xacro:property name="arm_4_joint_ub" value="2.44" />
+  <xacro:property name="arm_4_joint_lb" value="-1.1" />
   <xacro:property name="arm_5_joint_ub" value="2.6" />
   <xacro:property name="arm_5_joint_lb" value="-2.6" />

Commit message: Flip joint_2 limits

File: tiago_v2_prototype_description/urdf/arm/arm.limits.xacro (robot description, xacro)
@@ -15,6 +15,6 @@
   <xacro:property name="arm_1_joint_ub" value="2.6" />
   <xacro:property name="arm_1_joint_lb" value="-2.6" />
-  <xacro:property name="arm_2_joint_ub" value="2.44" />
-  <xacro:property name="arm_2_joint_lb" value="-1.10" />
+  <xacro:property name="arm_2_joint_ub" value="1.10" />
+  <xacro:property name="arm_2_joint_lb" value="-2.44" />
   <xacro:property name="arm_3_joint_ub" value="2.6" />
   <xacro:property name="arm_3_joint_lb" value="-2.6" />

Commit message: 180 degrees flip of link 3 to improve motion ranges

File: tiago_v2_prototype_description/urdf/arm/arm.limits.xacro (robot description, xacro)
@@ -13,4 +13,8 @@
 -->
 <robot xmlns:xacro="http://ros.org/wiki/xacro">
+  <!--
+  <xacro:property name="arm_1_joint_ub" value="3.67" />
+  <xacro:property name="arm_1_joint_lb" value="-1.57" />
+  -->
   <xacro:property name="arm_1_joint_ub" value="2.6" />
   <xacro:property name="arm_1_joint_lb" value="-2.6" />

File: tiago_v2_prototype_description/urdf/arm/arm.urdf.xacro (robot description, xacro)
@@ -75,4 +75,7 @@
       <axis xyz="0 0 1" />
       <limit lower="${arm_1_joint_lb}" upper="${arm_1_joint_ub}" effort="${arm_1_max_effort}" velocity="${arm_1_max_velocity}" />
+      <!-- <limit lower="${-0.5*(reflect-1)*arm_1_joint_lb - 0.5*(reflect+1)*arm_1_joint_ub}"
+             upper="${-0.5*(reflect-1)*arm_1_joint_ub - 0.5*(reflect+1)*arm_1_joint_lb}" effort="${arm_1_max_effort}" velocity="${arm_1_max_velocity}" />
+      -->
     </joint>
     <!-- ARM 2 LINK -->
@@ -152,5 +155,5 @@
       <origin
       xyz="-0.15 -0.02 0"
-      rpy="0 -1.5707 0" />
+      rpy="3.1415 1.5707 0" />
       <parent link="${name}_2_link" />
       <child link="${name}_3_link" />
