Commit message: Reduce head joint limits and update dynamic parameters

File: tiago_v2_prototype_description/urdf/head/head.urdf.xacro (robot description, xacro)
@@ -20,8 +20,8 @@
   <xacro:property name="head_damping"  value="0.5" />
   <xacro:property name="head_max_vel"  value="3.0" />
-  <xacro:property name="head_1_lower_limit" value="-75"/>
-  <xacro:property name="head_1_upper_limit" value="75"/>
-  <xacro:property name="head_2_lower_limit" value="-60"/>
-  <xacro:property name="head_2_upper_limit" value="45"/>
+  <xacro:property name="head_1_lower_limit" value="-55"/>
+  <xacro:property name="head_1_upper_limit" value="55"/>
+  <xacro:property name="head_2_lower_limit" value="-55"/>
+  <xacro:property name="head_2_upper_limit" value="20"/>
   <xacro:property name="head_eps"      value="${0.07}" />
   <xacro:property name="head_1_joint_offset"      value="${0.0}" />
@@ -33,13 +33,15 @@
     <link name="${name}_1_link">
       <inertial>
-        <origin xyz="0.013723 0.0015288 0.091095" rpy="0 0 0" />
-        <mass value="0.50253" />
+        <origin
+          xyz="0.0151529168350566 0.00114213181417127 0.0915264960362224"
+          rpy="0 0 0" />
+        <mass value="0.5232442430173" />
         <inertia
-          ixx="0.00073252"
-          ixy="-1.0801E-06"
-          ixz="-6.3715E-05"
-          iyy="0.0005861"
-          iyz="4.157E-10"
-          izz="0.00060232" />
+          ixx="0.000735269995053842"
+          ixy="-1.08043527376587E-06"
+          ixz="-6.37152476586251E-05"
+          iyy="0.000591525160132652"
+          iyz="-7.68106728600967E-12"
+          izz="0.000605065517138752" />
       </inertial>
       <visual>
@@ -57,5 +59,4 @@
           <mesh filename="package://tiago_v2_prototype_description/meshes/head/head_1_link_collision.stl" scale="1 1 1"/>
         </geometry>
-        <material name="White" />
       </collision>
     </link>
@@ -83,9 +84,16 @@
     <link name="${name}_2_link">
       <inertial>
-        <origin xyz="0.0025967 0.11474 0.00021233" rpy="0 0 0" />
-        <mass value="1.2093"/>
-        <inertia ixx="0.0063697" ixy="0.00052067" ixz="-8.4666E-06"
-                 iyy="0.0045958" iyz="9.6501E-06"
-                 izz="0.0031995" />
+        <origin
+          xyz="0.00277337961585723 0.115101831131133 4.87500103012104E-05"
+          rpy="0 0 0" />
+        <mass
+          value="1.24570092574607" />
+        <inertia
+          ixx="0.00635908800181593"
+          ixy="0.000520891211224051"
+          ixz="-8.48824527287752E-06"
+          iyy="0.00458972596146156"
+          iyz="9.69834634769094E-06"
+          izz="0.00320064764172765" />
       </inertial>
       <visual>

Commit message: intel d435 added

File: tiago_v2_prototype_description/urdf/head/head.urdf.xacro (robot description, xacro)
@@ -16,4 +16,5 @@
   <xacro:include filename="$(find tiago_v2_prototype_description)/urdf/deg_to_rad.xacro" />
   <xacro:include filename="$(find tiago_v2_prototype_description)/urdf/head/head.transmission.xacro" />
+  <xacro:include filename="$(find realsense2_description)/urdf/_d435.urdf.xacro" />
   <!--Constant parameters-->
   <xacro:property name="head_friction" value="1.0" />
@@ -135,4 +136,9 @@
        <implicitSpringDamper>1</implicitSpringDamper>
     </gazebo>
+    <!-- Head camera: Intel D435 -->
+    <xacro:sensor_d435 parent="${name}_2_link" name="${name}_d435_camera" topics_ns="${name}_d435_camera" use_nominal_extrinsics="true">
+       <origin xyz="0.03815 0.14750 0.0"
+                rpy="${-90.0 * deg_to_rad} 0.0 0.0"/>
+    </xacro:sensor_d435>
   </xacro:macro>
 </robot>

Commit message: added head_screen_link to the URDF

File: tiago_v2_prototype_description/urdf/head/head.urdf.xacro (robot description, xacro)
@@ -122,4 +122,10 @@
     </joint>
     <xacro:head_transmission name="${name}_2" reduction="1" offset_value="${head_2_joint_offset}"/>
+    <link name="${name}_screen_link"/>
+    <joint name="${name}_screen_joint" type="fixed">
+      <parent link="${name}_2_link" />
+      <child link="${name}_screen_link" />
+        <origin xyz="0.0528 0.08 0.0" rpy="${-90.0 * deg_to_rad} 0 0" />
+    </joint>
     <gazebo reference="${name}_1_link">
       <mu1>0.9</mu1>

Commit message: Flipped the limits of the head

File: tiago_v2_prototype_description/urdf/head/head.urdf.xacro (robot description, xacro)
@@ -23,6 +23,6 @@
   <xacro:property name="head_1_lower_limit" value="-55"/>
   <xacro:property name="head_1_upper_limit" value="55"/>
-  <xacro:property name="head_2_lower_limit" value="-55"/>
-  <xacro:property name="head_2_upper_limit" value="20"/>
+  <xacro:property name="head_2_lower_limit" value="-20"/>
+  <xacro:property name="head_2_upper_limit" value="55"/>
   <xacro:property name="head_eps"      value="${0.07}" />
   <xacro:property name="head_1_joint_offset"      value="${0.0}" />
