Commit message: urdf support for is_public_sim

File: tiago_pro_description/gazebo/gazebo.urdf.xacro (robot description, xacro)
@@ -26,5 +26,10 @@
       <publish_rate>50</publish_rate>
       <publish_odom>true</publish_odom>
-      <publish_odom_tf>false</publish_odom_tf>
+      <xacro:if value="${is_public_sim}">
+        <publish_odom_tf>true</publish_odom_tf>
+      </xacro:if>
+      <xacro:unless value="${is_public_sim}">
+        <publish_odom_tf>false</publish_odom_tf>
+      </xacro:unless>
       <odometry_frame>odom</odometry_frame>
       <robot_base_frame>base_footprint</robot_base_frame>

File: tiago_pro_description/robots/tiago_pro.urdf.xacro (robot description, xacro)
@@ -29,4 +29,5 @@
   <xacro:arg name="ft_sensor_right" default="no-ft-sensor" />
   <xacro:arg name="use_sim" default="false"/>
+  <xacro:arg name="is_public_sim" default="false"/>
   <xacro:arg name="description_calibration_dir" default="$(find tiago_pro_description)/urdf"/>
   <xacro:arg name="extrinsic_calibration_dir" default="$(find tiago_pro_description)/urdf"/>
@@ -47,4 +48,5 @@
   <xacro:property name="arm_model" value="tiago-pro" />
   <xacro:property name="description_calibration_dir" value="${arg description_calibration_dir}"/>
+  <xacro:property name="is_public_sim" value="$(arg is_public_sim)" />
   <xacro:property name="has_arm_left" value="${arm_model_left not in ['no-arm']}"/>
   <xacro:property name="has_ft_sensor_left" value="${ft_sensor_left not in ['no-ft-sensor']}"/>
