Commit message: Added head

File: tiago_pro_description/urdf/head/head.urdf.xacro (robot description, xacro)
@@ -17,99 +17,75 @@
   <!--Constant parameters-->
   <xacro:property name="head_friction" value="1.0" />
-  <xacro:property name="head_damping"  value="0.5" />
-  <xacro:property name="head_max_vel"  value="3.0" />
-  <xacro:property name="head_1_lower_limit" value="-55"/>
-  <xacro:property name="head_1_upper_limit" value="55"/>
-  <xacro:property name="head_2_lower_limit" value="-20"/>
-  <xacro:property name="head_2_upper_limit" value="55"/>
-  <xacro:property name="head_eps"      value="${0.07}" />
-  <!-- <xacro:property name="head_1_joint_offset"      value="${0.0}" />
-  <xacro:property name="head_2_joint_offset"      value="${0.0}" /> -->
-  <!--************************-->
-  <!--     HEAD_1 (PAN)       -->
-  <!--************************-->
+  <xacro:property name="head_damping" value="0.5" />
+  <xacro:property name="head_max_vel" value="3.0" />
+  <xacro:property name="head_1_lower_limit" value="-1.309"/>
+  <xacro:property name="head_1_upper_limit" value="1.309"/>
+  <xacro:property name="head_2_lower_limit" value="-1.0472"/>
+  <xacro:property name="head_2_upper_limit" value="0.34907"/>
+  <xacro:property name="head_eps" value="${0.07}" />
   <xacro:macro name="tiago_pro_head" params="name parent">
+    <!-- Head Link 1-->
     <link name="${name}_1_link">
       <inertial>
-        <origin
-          xyz="0.013723 0.0015288 0.091095"
-          rpy="0 0 0" />
-        <mass
-          value="0.50253" />
-        <inertia
-          ixx="0.00073252"
-          ixy="-1.0801E-06"
-          ixz="-6.3715E-05"
-          iyy="0.0005861"
-          iyz="4.157E-10"
-          izz="0.00060232" />
+        <origin xyz="0.0016768 3.1033E-05 0.081737" rpy="0 0 0" />
+        <mass value="0.22677" />
+        <inertia ixx="0.00056619" ixy="3.0482E-07" ixz="6.7491E-05" iyy="0.00040222" iyz="-5.9322E-07" izz="0.00039176" />
       </inertial>
       <visual>
-        <origin xyz="0 0 0" rpy="0 0 0"/>
+        <origin xyz="0 0 0" rpy="0 0 0" />
         <geometry>
-          <mesh filename="package://tiago_pro_description/meshes/head/head_1_link.stl" scale="1 1 1"/>
+          <mesh filename="package://tiago_pro_description/meshes/head/head_1_link.stl" />
         </geometry>
-        <material name="pal/DarkGrey"/>
+        <material name="">
+          <color rgba="0.29804 0.29804 0.29804 1" />
+        </material>
       </visual>
       <collision>
-        <origin xyz="0.0 0 0" rpy="0 0 0.0" />
+        <origin xyz="0 0 0" rpy="0 0 0" />
         <geometry>
-          <mesh filename="package://tiago_pro_description/meshes/head/head_1_link_collision.stl" scale="1 1 1"/>
+          <mesh filename="package://tiago_pro_description/meshes/head/head_1_link_collision.stl" />
         </geometry>
       </collision>
     </link>
     <joint name="${name}_1_joint" type="revolute">
-      <parent link="${parent}"/>
-      <child link="${name}_1_link"/>
-      <origin xyz="0.0 0.0 0.04"  rpy="0 0 0" />
+      <origin xyz="0 0 0" rpy="0 0 3.14" />
+      <parent link="${parent}" />
+      <child link="head_1_link" />
       <axis xyz="0 0 1" />
-      <limit lower="${head_1_lower_limit * deg_to_rad}" upper="${head_1_upper_limit * deg_to_rad}" effort="5.197" velocity="${head_max_vel}" />
+      <limit lower="${head_1_lower_limit}" upper="${head_1_upper_limit}" effort="5.197" velocity="${head_max_vel}" />
       <dynamics damping="${head_damping}" friction="${head_friction}"/>
-      <safety_controller k_position="20"
-                         k_velocity="20"
-                         soft_lower_limit="${head_1_lower_limit * deg_to_rad + head_eps}"
-                         soft_upper_limit="${head_1_upper_limit * deg_to_rad - head_eps}" />
+      <safety_controller k_position="20" k_velocity="20" soft_lower_limit="${head_1_lower_limit + head_eps}" soft_upper_limit="${head_1_upper_limit - head_eps}" />
     </joint>
+    <!-- Head link 2-->
     <link name="${name}_2_link">
       <inertial>
-        <origin
-          xyz="0.0025967 0.11474 0.00021233"
-          rpy="0 0 0" />
-        <mass
-          value="1.2093" />
-        <inertia
-          ixx="0.0063697"
-          ixy="0.00052067"
-          ixz="-8.4666E-06"
-          iyy="0.0045958"
-          iyz="9.6501E-06"
-          izz="0.0031995" />
+        <origin xyz="-0.0087157 0.11401 -0.00024206" rpy="0 0 0" />
+        <mass value="0.84465" />
+        <inertia ixx="0.006226" ixy="-0.00055126" ixz="-7.2157E-06" iyy="0.0050209" iyz="-1.0342E-05" izz="0.002495" />
       </inertial>
       <visual>
         <origin xyz="0 0 0" rpy="0 0 0" />
         <geometry>
-          <mesh filename="package://tiago_pro_description/meshes/head/head_2_link.stl" scale="1 1 1"/>
+          <mesh filename="package://tiago_pro_description/meshes/head/head_2_link.stl" />
         </geometry>
-        <material name="White"/>
+        <material name="">
+          <color rgba="1 1 1 1" />
+        </material>
       </visual>
       <collision>
         <origin xyz="0 0 0" rpy="0 0 0" />
         <geometry>
-          <mesh filename="package://tiago_pro_description/meshes/head/head_2_link_collision.stl" scale="1 1 1"/>
+          <mesh filename="package://tiago_pro_description/meshes/head/head_2_link_collision.stl" />
         </geometry>
       </collision>
     </link>
-    <joint name="${name}_2_joint" type="revolute">
-      <parent link="${name}_1_link"/>
-      <child link="${name}_2_link"/>
-      <origin xyz="0.04597 0 0.10075"
-      rpy="1.5708 0 0" />
+    <joint name="head_2_joint" type="revolute">
+      <origin xyz="-0.0425 0 0.1011" rpy="1.5708 0 0" />
+      <parent link="${name}_1_link" />
+      <child link="${name}_2_link" />
       <axis xyz="0 0 -1" />
-      <limit lower="${head_2_lower_limit * deg_to_rad}" upper="${head_2_upper_limit * deg_to_rad}" effort="2.77" velocity="${head_max_vel}" />
+      <limit lower="${head_2_lower_limit}" upper="${head_2_upper_limit}" effort="2.77" velocity="${head_max_vel}" />
       <dynamics damping="${head_damping}" friction="${head_friction}"/>
-      <safety_controller k_position="20"
-                         k_velocity="20"
-                         soft_lower_limit="${head_2_lower_limit * deg_to_rad + head_eps}"
-                         soft_upper_limit="${head_2_upper_limit * deg_to_rad - head_eps}" />
+      <safety_controller k_position="20" k_velocity="20" soft_lower_limit="${head_2_lower_limit + head_eps}" soft_upper_limit="${head_2_upper_limit - head_eps}" />
     </joint>
     <link name="${name}_screen_link"/>
@@ -117,5 +93,5 @@
       <parent link="${name}_2_link" />
       <child link="${name}_screen_link" />
-        <origin xyz="0.0528 0.08 0.0" rpy="${-90.0 * deg_to_rad} 0 0" />
+      <origin xyz="0.0528 0.08 0.0" rpy="${-90.0 * deg_to_rad} 0 0" />
     </joint>
     <gazebo reference="${name}_1_link">
@@ -130,13 +106,12 @@
     </gazebo>
     <gazebo reference="${name}_1_joint">
-       <implicitSpringDamper>1</implicitSpringDamper>
+      <implicitSpringDamper>1</implicitSpringDamper>
     </gazebo>
     <gazebo reference="${name}_2_joint">
-       <implicitSpringDamper>1</implicitSpringDamper>
+      <implicitSpringDamper>1</implicitSpringDamper>
     </gazebo>
     <!-- Head camera:Intel D435 -->
     <xacro:sensor_d435 parent="${name}_2_link" name="${name}_front_camera" topics_ns="${name}_front_camera" use_nominal_extrinsics="${use_sim_time}">
-       <origin xyz="0.03815 0.14750 0.0"
-                rpy="${-90.0 * deg_to_rad} 0.0 0.0"/>
+      <origin xyz="-0.0415999999999995 0.1555 0" rpy="1.5707963267949 0 3.14159265358979" />
     </xacro:sensor_d435>
   </xacro:macro>

Commit message: Invert head 2 joint direction

File: tiago_pro_description/urdf/head/head.urdf.xacro (robot description, xacro)
@@ -105,5 +105,5 @@
       <origin xyz="0.04597 0 0.10075"
       rpy="1.5708 0 0" />
-      <axis xyz="0 0 1" />
+      <axis xyz="0 0 -1" />
       <limit lower="${head_2_lower_limit * deg_to_rad}" upper="${head_2_upper_limit * deg_to_rad}" effort="2.77" velocity="${head_max_vel}" />
       <dynamics damping="${head_damping}" friction="${head_friction}"/>

Commit message: added frames for sellion and eyes

File: tiago_pro_description/urdf/head/head.urdf.xacro (robot description, xacro)
@@ -141,3 +141,22 @@
     </xacro:sensor_d435>
   </xacro:macro>
+  <!-- EYE FRAMES -->
+  <link name="sellion_link"/>
+  <joint name="sellion_joint" type="fixed">
+    <origin xyz="0.04 0.09205 0" rpy="${-90 * deg_to_rad} 0 0"/>
+    <child link="sellion_link" />
+    <parent link="head_2_link"/>
+  </joint>
+  <link name="eye_right_link"/>
+  <joint name="eye_right_joint" type="fixed">
+    <origin xyz="0.0 -0.1 0" rpy="0 0 0"/>
+    <child link="eye_right_link" />
+    <parent link="sellion_link"/>
+  </joint>
+  <link name="eye_left_link"/>
+  <joint name="eye_left_joint" type="fixed">
+    <origin xyz="0 0.1 0" rpy="0 0 0"/>
+    <child link="eye_left_link" />
+    <parent link="sellion_link"/>
+  </joint>
 </robot>
