Commit message: Modifying inertia of torso

File: tiago_pro_description/urdf/torso/torso.urdf.xacro (robot description, xacro)
@@ -82,9 +82,9 @@
     <!-- Lift torso -->
     <link name="${name}_lift_link">
-      <inertial>
-        <origin xyz="-0.11911204633044 -0.000151023929951286 -0.0721028051446563" rpy="0 0 0" />
+    <inertial>
+      <origin xyz="0 0 0" rpy="0 0 0" />
         <mass value="3.24266045177967" />
         <inertia ixx="0.0295369723560087" ixy="-7.85101789883696E-07" ixz="-8.58576921315497E-05" iyy="0.0170989395656347" iyz="-8.17944373020342E-06" izz="0.0290055792681799" />
-      </inertial>
+    </inertial>
       <visual>
         <origin xyz="0 0 0" rpy="0 0 0" />

Commit message: Put back safety controller for the torso + change motions

File: tiago_pro_description/urdf/torso/torso.urdf.xacro (robot description, xacro)
@@ -127,8 +127,8 @@
       <child link="${name}_lift_link" />
       <axis xyz="0 0 1" />
-      <limit effort="2000" lower="0" upper="0.33" velocity="${torso_max_vel}" />
+      <limit effort="2000" lower="0" upper="0.35" velocity="${torso_max_vel}" />
       <calibration rising="0.0" />
       <dynamics damping="1000" />
-      <safety_controller k_position="20" k_velocity="20" soft_lower_limit="0.0" soft_upper_limit="0.33" />
+      <safety_controller k_position="20" k_velocity="20" soft_lower_limit="${0.0 + torso_eps}" soft_upper_limit="${0.35 - torso_eps}" />
     </joint>
     <gazebo reference="${name}_lift_joint">

Commit message: Remove safety-eps form torso and update boxing motion

File: tiago_pro_description/urdf/torso/torso.urdf.xacro (robot description, xacro)
@@ -15,5 +15,5 @@
   <!--Constant parameters-->
   <xacro:property name="torso_max_vel" value="0.035" />
-  <xacro:property name="torso_eps" value="0.02" />
+  <xacro:property name="torso_eps" value="0.00" />
   <xacro:macro name="tiago_pro_torso" params="name parent has_tray">
     <!-- Connection with the base -->

Commit message: Scale sligthly the visual of the base_link of the torso to remove visualization bug + add visual for the head_link

File: tiago_pro_description/urdf/torso/torso.urdf.xacro (robot description, xacro)
@@ -29,7 +29,5 @@
           <mesh filename="package://tiago_pro_description/meshes/torso/base_link.stl" />
         </geometry>
-        <material name="">
-          <color rgba="0.298039215686275 0.298039215686275 0.298039215686275 1" />
-        </material>
+        <material name="pal/DarkGrey"/>
       </visual>
       <collision>
@@ -82,9 +80,9 @@
     <!-- Lift torso -->
     <link name="${name}_lift_link">
-    <inertial>
-      <origin xyz="0 0 0" rpy="0 0 0" />
-        <mass value="3.24266045177967" />
-        <inertia ixx="0.0295369723560087" ixy="-7.85101789883696E-07" ixz="-8.58576921315497E-05" iyy="0.0170989395656347" iyz="-8.17944373020342E-06" izz="0.0290055792681799" />
-    </inertial>
+      <inertial>
+        <origin xyz="0 0 0" rpy="0 0 0" />
+          <mass value="3.24266045177967" />
+          <inertia ixx="0.0295369723560087" ixy="-7.85101789883696E-07" ixz="-8.58576921315497E-05" iyy="0.0170989395656347" iyz="-8.17944373020342E-06" izz="0.0290055792681799" />
+      </inertial>
       <visual>
         <origin xyz="0 0 0" rpy="0 0 0" />
@@ -129,4 +127,19 @@
         <inertia ixx="0.000439179732174765" ixy="5.76286393008048E-20" ixz="1.09094748941927E-18" iyy="0.000498456551929403" iyz="-1.60059406264224E-19" izz="0.000881920896131913" />
       </inertial>
+      <visual>
+        <origin xyz="0 0 0.01085" rpy="0 0 0" />
+        <geometry>
+          <box size="0.11 0.092 0.0217" />
+        </geometry>
+        <material name="">
+          <color rgba="0.298039215686275 0.298039215686275 0.298039215686275 1" />
+        </material>
+      </visual>
+      <collision>
+        <origin xyz="0 0 0.01085" rpy="0 0 0" />
+        <geometry>
+          <box size="0.11 0.092 0.0217" />
+        </geometry>
+      </collision>
     </link>
     <joint name="${name}_head_joint" type="fixed">
@@ -136,7 +149,4 @@
       <axis xyz="0 0 0" />
     </joint>
-    <gazebo reference="${name}_head_link">
-      <material>Gazebo/DarkGrey</material>
-    </gazebo>
     <!-- Torso arm left link-->
     <link name="${name}_arm_left_link"/>
@@ -147,7 +157,4 @@
       <axis xyz="0 0 0" />
     </joint>
-    <gazebo reference="${name}_arm_left_link">
-      <material>Gazebo/DarkGrey</material>
-    </gazebo>
     <!-- Torso arm right link -->
     <link name="${name}_arm_right_link"/>
@@ -158,7 +165,4 @@
       <axis xyz="0 0 0" />
     </joint>
-    <gazebo reference="${name}_arm_right_link">
-      <material>Gazebo/DarkGrey</material>
-    </gazebo>
   </xacro:macro>
 </robot>

Commit message: Fix naming + change collision toroso_fixed

File: tiago_pro_description/urdf/torso/torso.urdf.xacro (robot description, xacro)
@@ -27,5 +27,5 @@
         <origin xyz="0 0 0" rpy="0 0 0" />
         <geometry>
-          <mesh filename="package://tiago_pro_description/meshes/torso/base_link.stl" />
+          <mesh filename="package://tiago_pro_description/meshes/torso/torso_fixed.stl" />
         </geometry>
         <material name="pal/DarkGrey"/>
@@ -34,5 +34,5 @@
         <origin xyz="0 0 0" rpy="0 0 0" />
         <geometry>
-          <mesh filename="package://tiago_pro_description/meshes/torso/base_link_collision.stl" />
+          <mesh filename="package://tiago_pro_description/meshes/torso/torso_fixed_collision.stl" />
         </geometry>
       </collision>
@@ -49,9 +49,4 @@
     <!-- Fixed column -->
     <link name="${name}_fixed_column_link">
-      <inertial>
-        <origin rpy="0 0 0" xyz="0 0 0" />
-        <mass value="0.01" />
-        <inertia ixx="0.000001" ixy="0" ixz="0" iyy="0.000001" iyz="0" izz="0.000001" />
-      </inertial>
       <visual>
         <origin rpy="0 0 0" xyz="0 0 0.275" />
@@ -61,11 +56,4 @@
         <material name="pal/DarkGrey"/>
       </visual>
-      <collision>
-        <origin rpy="0 0 0" xyz="0 0 0.275" />
-        <geometry>
-          <box size="0.23 0.253 0.45"/>
-        </geometry>
-        <material name="pal/DarkGrey"/>
-      </collision>
     </link>
     <joint name="${name}_fixed_column_joint" type="fixed">
