Commit message: Split ros2_control hardware into three RobotControl components

File: tiago_pro_description/ros2_control/ros2_control.urdf.xacro (robot description, xacro)
@@ -13,62 +13,11 @@
  -->
 <robot xmlns:xacro="http://ros.org/wiki/xacro" name="tiago_pro">
-  <xacro:macro name="tiago_pro_ros2_control" params="use_sim_time:=^|false">
-    <xacro:arg name="arm_type_left" default="tiago-pro"/>
-    <xacro:arg name="arm_type_right" default="tiago-pro"/>
-    <xacro:arg name="end_effector_left" default="pal-pro-pripper"/>
-    <xacro:arg name="end_effector_right" default="pal-pro-gripper"/>
-    <xacro:arg name="ft_sensor_left" default="no-ft-sensor"/>
-    <xacro:arg name="ft_sensor_right" default="no-ft-sensor"/>
-    <xacro:arg name="description_calibration_dir" default="$(find tiago_pro_description)/urdf/calibration" />
-    <!-- TODO-->
-    <xacro:property name="arm_type_left" value="$(arg arm_type_left)" />
-    <xacro:property name="arm_type_right" value="$(arg arm_type_right)" />
-    <xacro:property name="end_effector_left" value="$(arg end_effector_left)" />
-    <xacro:property name="end_effector_right" value="$(arg end_effector_right)" />
-    <xacro:property name="has_ft_sensor_left" value="${ft_sensor_left != 'no-ft-sensor'}" />
-    <xacro:property name="has_ft_sensor_right" value="${ft_sensor_right != 'no-ft-sensor'}" />
-    <xacro:property name="has_arm_left" value="${arm_type_left != 'no-arm'}" />
-    <xacro:property name="has_arm_right" value="${arm_type_right != 'no-arm'}" />
-    <xacro:include filename="$(find omni_base_description)/urdf/sensors/sensors.ros2_control.xacro" />
-    <xacro:include filename="$(find omni_base_description)/urdf/wheels/wheel.ros2_control.xacro" />
-    <xacro:include filename="$(find tiago_pro_description)/urdf/torso/torso.ros2_control.xacro" />
-    <xacro:include filename="$(find tiago_pro_description)/urdf/head/head.ros2_control.xacro" />
-    <xacro:include filename="$(find pal_sea_arm_description)/urdf/arm/arm.ros2_control.xacro" />
-    <xacro:if value="${end_effector_left == 'pal-pro-gripper' or end_effector_right == 'pal-pro-gripper'}">
-      <xacro:include filename="$(find pal_pro_gripper_description)/urdf/pal_pro_gripper.ros2_control.xacro" />
-    </xacro:if>
-    <!-- calibration offsets -->
-    <xacro:include filename="$(arg description_calibration_dir)/calibration_constants.urdf.xacro" />
-    <!-- Init the ROS 2 control gazebo interface -->
-    <xacro:if value="${use_sim_time}">
-      <gazebo>
-        <plugin filename="libgazebo_ros2_control.so" name="gazebo_ros2_control">
-          <parameters>$(find tiago_pro_description)/ros2_control/gazebo_controller_manager_cfg.yaml</parameters>
-        </plugin>
-      </gazebo>
-    </xacro:if>
-    <ros2_control name="ros2_control_tiago_pro_system" type="system">
-      <hardware>
-        <xacro:if value="$(arg use_sim_time)">
-          <plugin>gazebo_ros2_control/GazeboSystem</plugin>
-        </xacro:if>
-        <xacro:unless value="$(arg use_sim_time)">
-          <plugin>robot_control/RobotControl</plugin>
-        </xacro:unless>
-      </hardware>
-      <!-- wheels -->
-      <xacro:ros2_control_wheel side="front_right" />
-      <xacro:ros2_control_wheel side="front_left" />
-      <xacro:ros2_control_wheel side="rear_right" />
-      <xacro:ros2_control_wheel side="rear_left" />
-      <!-- IMU -->
-      <xacro:if value="$(arg use_sim_time)">
-        <xacro:ros2_control_imu name="base_imu_sensor"/>
-      </xacro:if>
-      <!-- torso -->
-      <xacro:ros2_control_torso name="torso_lift" reduction="1.0" />
-      <!-- head -->
-      <xacro:ros2_control_head name="head_1" reduction="1.0" offset_value="${head_1_joint_offset}" />
-      <xacro:ros2_control_head name="head_2" reduction="1.0" offset_value="${head_2_joint_offset}" />
+  <xacro:macro name="ros2_control_wheels">
+    <xacro:ros2_control_wheel side="front_right" />
+    <xacro:ros2_control_wheel side="front_left" />
+    <xacro:ros2_control_wheel side="rear_right" />
+    <xacro:ros2_control_wheel side="rear_left" />
+  </xacro:macro>
+  <xacro:macro name="ros2_control_arms">
       <!-- arm left -->
       <xacro:if value="${has_arm_left}">
@@ -106,5 +55,92 @@
         </xacro:if>
       </xacro:if>
-    </ros2_control>
+  </xacro:macro>
+  <xacro:macro name="tiago_pro_ros2_control" params="use_sim_time:=^|false">
+    <xacro:arg name="arm_type_left" default="tiago-pro"/>
+    <xacro:arg name="arm_type_right" default="tiago-pro"/>
+    <xacro:arg name="end_effector_left" default="pal-pro-pripper"/>
+    <xacro:arg name="end_effector_right" default="pal-pro-gripper"/>
+    <xacro:arg name="ft_sensor_left" default="no-ft-sensor"/>
+    <xacro:arg name="ft_sensor_right" default="no-ft-sensor"/>
+    <xacro:arg name="description_calibration_dir" default="$(find tiago_pro_description)/urdf/calibration" />
+    <!-- TODO-->
+    <xacro:property name="arm_type_left" value="$(arg arm_type_left)" />
+    <xacro:property name="arm_type_right" value="$(arg arm_type_right)" />
+    <xacro:property name="end_effector_left" value="$(arg end_effector_left)" />
+    <xacro:property name="end_effector_right" value="$(arg end_effector_right)" />
+    <xacro:property name="has_ft_sensor_left" value="${ft_sensor_left != 'no-ft-sensor'}" />
+    <xacro:property name="has_ft_sensor_right" value="${ft_sensor_right != 'no-ft-sensor'}" />
+    <xacro:property name="has_arm_left" value="${arm_type_left != 'no-arm'}" />
+    <xacro:property name="has_arm_right" value="${arm_type_right != 'no-arm'}" />
+    <xacro:include filename="$(find omni_base_description)/urdf/sensors/sensors.ros2_control.xacro" />
+    <xacro:include filename="$(find omni_base_description)/urdf/wheels/wheel.ros2_control.xacro" />
+    <xacro:include filename="$(find tiago_pro_description)/urdf/torso/torso.ros2_control.xacro" />
+    <xacro:include filename="$(find tiago_pro_description)/urdf/head/head.ros2_control.xacro" />
+    <xacro:include filename="$(find pal_sea_arm_description)/urdf/arm/arm.ros2_control.xacro" />
+    <xacro:if value="${end_effector_left == 'pal-pro-gripper' or end_effector_right == 'pal-pro-gripper'}">
+      <xacro:include filename="$(find pal_pro_gripper_description)/urdf/pal_pro_gripper.ros2_control.xacro" />
+    </xacro:if>
+    <!-- calibration offsets -->
+    <xacro:include filename="$(arg description_calibration_dir)/calibration_constants.urdf.xacro" />
+    <!-- Simulation -->
+    <xacro:if value="$(arg use_sim_time)">
+      <!-- Init the ROS 2 control gazebo interface -->
+      <gazebo>
+        <plugin filename="libgazebo_ros2_control.so" name="gazebo_ros2_control">
+          <parameters>$(find tiago_pro_description)/ros2_control/gazebo_controller_manager_cfg.yaml</parameters>
+        </plugin>
+      </gazebo>
+      <ros2_control name="ros2_control_gazebo_system" type="system">
+        <hardware>
+          <plugin>gazebo_ros2_control/GazeboSystem</plugin>
+        </hardware>
+        <!-- wheels -->
+        <xacro:ros2_control_wheels/>
+        <!-- IMU -->
+        <xacro:ros2_control_imu name="base_imu_sensor"/>
+        <!-- torso -->
+        <xacro:ros2_control_torso name="torso_lift" reduction="1.0" />
+        <!-- head -->
+        <xacro:ros2_control_head name="head_1" reduction="1.0" offset_value="${head_1_joint_offset}" />
+        <xacro:ros2_control_head name="head_2" reduction="1.0" offset_value="${head_2_joint_offset}" />
+        <!-- arms -->
+          <xacro:ros2_control_arms/>
+      </ros2_control>
+    </xacro:if>
+    <!-- Hardware -->
+    <xacro:unless value="$(arg use_sim_time)">
+      <!-- CAN system -->
+      <ros2_control name="ros2_control_tiago_pro_system_can" type="system">
+        <hardware>
+          <plugin>robot_control/RobotControl</plugin>
+          <param name="group">can</param>
+        </hardware>
+        <!-- wheels -->
+        <xacro:ros2_control_wheels />
+        <!-- IMU -->
+        <!-- <xacro:ros2_control_imu name="base_imu_sensor"/> -->
+        <!-- torso -->
+        <xacro:ros2_control_torso name="torso_lift" reduction="1.0" />
+      </ros2_control>
+      <!-- Dynamixels system -->
+      <ros2_control name="ros2_control_tiago_pro_system_dynamixel" type="system">
+        <hardware>
+          <plugin>robot_control/RobotControl</plugin>
+          <param name="group">dynamixel</param>
+        </hardware>
+        <!-- head -->
+        <xacro:ros2_control_head name="head_1" reduction="1.0" offset_value="${head_1_joint_offset}" />
+        <xacro:ros2_control_head name="head_2" reduction="1.0" offset_value="${head_2_joint_offset}" />
+      </ros2_control>
+      <!-- Ethercat system -->
+      <ros2_control name="ros2_control_tiago_pro_system_ethercat" type="system">
+        <hardware>
+          <plugin>robot_control/RobotControl</plugin>
+          <param name="group">ethercat</param>
+        </hardware>
+        <!-- arms -->
+        <xacro:ros2_control_arms/>
+      </ros2_control>
+    </xacro:unless>
   </xacro:macro>
 </robot>

Commit message: Update torso limits

File: tiago_pro_description/ros2_control/ros2_control.urdf.xacro (robot description, xacro)
@@ -123,5 +123,5 @@
       </ros2_control>
       <!-- Dynamixels system -->
-      <ros2_control name="ros2_control_tiago_pro_system_dynamixel" type="system" rw_rate="100">
+      <ros2_control name="ros2_control_tiago_pro_system_dynamixel" type="system" rw_rate="200">
         <hardware>
           <plugin>robot_control/RobotControl</plugin>

File: tiago_pro_description/urdf/torso/torso.urdf.xacro (robot description, xacro)
@@ -14,5 +14,5 @@
 <robot xmlns:xacro="http://ros.org/wiki/xacro">
   <!--Constant parameters-->
-  <xacro:property name="torso_max_vel" value="0.07" />
+  <xacro:property name="torso_max_vel" value="0.035" />
   <xacro:property name="torso_eps" value="0.02" />
   <xacro:macro name="tiago_pro_torso" params="name parent has_tray">
@@ -127,8 +127,8 @@
       <child link="${name}_lift_link" />
       <axis xyz="0 0 1" />
-      <limit effort="2000" lower="0" upper="0.35" velocity="${torso_max_vel}" />
+      <limit effort="2000" lower="0" upper="0.33" velocity="${torso_max_vel}" />
       <calibration rising="0.0" />
       <dynamics damping="1000" />
-      <safety_controller k_position="20" k_velocity="20" soft_lower_limit="0.0" soft_upper_limit="0.35" />
+      <safety_controller k_position="20" k_velocity="20" soft_lower_limit="0.0" soft_upper_limit="0.33" />
     </joint>
     <gazebo reference="${name}_lift_joint">

Commit message: Delete for now xela components

File: tiago_pro_description/ros2_control/ros2_control.urdf.xacro (robot description, xacro)
@@ -19,6 +19,6 @@
     <xacro:ros2_control_wheel side="rear_left" />
   </xacro:macro>
-  <xacro:macro name="allegro_ros2_control" params="side allegro_can pid_controllers xela_can">
-    <ros2_control name="ros2_control_allegro_hand_system_${side}" type="system" rw_rate="1000">
+  <xacro:macro name="allegro_ros2_control" params="side allegro_can pid_controllers">
+    <ros2_control name="ros2_control_allegro_hand_system_${side}" type="system" rw_rate="200">
       <hardware>
         <plugin>allegro_hand_system/AllegroHandSystem</plugin>
@@ -27,10 +27,4 @@
       </hardware>
       <xacro:ros2_control_allegro_hand name="gripper_${side}" pid_controllers="$(arg pid_controllers)" reduction="1.0" />
-    </ros2_control>
-    <ros2_control name="ros2_control_xela_sensor_${side}" type="sensor" rw_rate="1000">
-      <hardware>
-        <plugin>xela_uskin_sensor/XelaUskinSensor</plugin>
-        <param name="${can_device_name}">${xela_can}</param>
-      </hardware>
     </ros2_control>
   </xacro:macro>
@@ -164,8 +158,8 @@
       <xacro:arg name="pid_controllers" default="true"/>
       <xacro:if value="${end_effector_right == 'allegro-hand'}">
-        <xacro:allegro_ros2_control side="right" allegro_can="can0" pid_controllers="$(arg pid_controllers)" xela_can="can1"/>
+        <xacro:allegro_ros2_control side="right" allegro_can="can0" pid_controllers="$(arg pid_controllers)"/>
       </xacro:if>
       <xacro:if value="${end_effector_left == 'allegro-hand'}">
-        <xacro:allegro_ros2_control side="left" allegro_can="can2" pid_controllers="$(arg pid_controllers)" xela_can="can3"/>
+        <xacro:allegro_ros2_control side="left" allegro_can="can2" pid_controllers="$(arg pid_controllers)"/>
       </xacro:if>
     </xacro:unless>
