Commit message: remove deg_to_rad to make use of pal_urdf_utils package

File: tiago_pro_description/robots/tiago_pro.urdf.xacro (robot description, xacro)
@@ -14,4 +14,6 @@
 <robot  xmlns:xacro="http://ros.org/wiki/xacro" name="tiago_pro">
 <!-- Includes -->
+<xacro:include filename="$(find pal_urdf_utils)/urdf/deg_to_rad.xacro" />
+<xacro:include filename="$(find pal_urdf_utils)/urdf/materials.urdf.xacro" />
 <xacro:include filename="$(find tiago_pro_description)/gazebo/gazebo.urdf.xacro" />
 <xacro:include filename="$(find tiago_pro_description)/urdf/torso/torso_dual.urdf.xacro" />

File: tiago_pro_description/urdf/head/head.urdf.xacro (robot description, xacro)
@@ -14,5 +14,4 @@
 <robot xmlns:xacro="http://ros.org/wiki/xacro">
   <!--File includes-->
-  <xacro:include filename="$(find tiago_pro_description)/urdf/deg_to_rad.xacro" />
   <xacro:include filename="$(find tiago_pro_description)/urdf/head/head.transmission.xacro" />
   <xacro:include filename="$(find realsense2_description)/urdf/_d435.urdf.xacro" />
@@ -52,7 +51,5 @@
           <mesh filename="package://tiago_pro_description/meshes/head/head_1_link.stl" scale="1 1 1"/>
         </geometry>
-        <material name="">
-          <color rgba="0.29804 0.29804 0.29804 1" />
-        </material>
+        <material name="pal/DarkGrey"/>
       </visual>
       <collision>
@@ -97,7 +94,5 @@
           <mesh filename="package://tiago_pro_description/meshes/head/head_2_link.stl" scale="1 1 1"/>
         </geometry>
-        <material name="">
-          <color rgba="0.29804 0.29804 0.29804 1" />
-        </material>
+        <material name="White"/>
       </visual>
       <collision>
@@ -129,8 +124,10 @@
     </joint>
     <gazebo reference="${name}_1_link">
+      <material>Gazebo/DarkGrey</material>
       <mu1>0.9</mu1>
       <mu2>0.9</mu2>
     </gazebo>
     <gazebo reference="${name}_2_link">
+      <material>Gazebo/White</material>
       <mu1>0.9</mu1>
       <mu2>0.9</mu2>

File: tiago_pro_description/urdf/torso/torso_dual.urdf.xacro (robot description, xacro)
@@ -9,5 +9,4 @@
 <robot xmlns:xacro="http://ros.org/wiki/xacro">
   <!--File includes-->
-  <xacro:include filename="$(find tiago_pro_description)/urdf/deg_to_rad.xacro" />
   <xacro:include filename="$(find tiago_pro_description)/urdf/torso/torso.transmission.xacro" />
   <!--Constant parameters-->
@@ -32,7 +31,5 @@
           filename="package://tiago_pro_description/meshes/torso/torso_fixed_link.stl" />
       </geometry>
-      <material name="">
-        <color rgba="0.29804 0.29804 0.29804 1" />
-      </material>
+      <material name="pal/DarkGrey"/>
     </visual>
     <collision>
@@ -41,5 +38,5 @@
         <box size="0.23 0.253 0.2"/>
       </geometry>
-      <material name="DarkGrey"/>
+      <material name="pal/DarkGrey"/>
     </collision>
     <collision>
@@ -48,5 +45,5 @@
         <box size="0.15 0.253 0.06"/>
       </geometry>
-      <material name="DarkGrey"/>
+      <material name="pal/DarkGrey"/>
     </collision>
     <collision>
@@ -55,7 +52,10 @@
         <box size="0.47 0.5 0.02"/>
       </geometry>
-      <material name="DarkGrey"/>
+      <material name="pal/DarkGrey"/>
     </collision>
   </link>
+  <gazebo reference="${name}_fixed_link">
+    <material>Gazebo/DarkGrey</material>
+  </gazebo>
   <joint name="${name}_fixed_joint" type="fixed">
     <origin rpy="0 0 0" xyz="-0.0245 0 0.215" />
@@ -78,5 +78,5 @@
         <box size="0.18 0.2 0.55"/>
       </geometry>
-      <material name="DarkGrey"/>
+      <material name="pal/DarkGrey"/>
     </visual>
     <collision>
@@ -85,5 +85,5 @@
         <box size="0.23 0.253 0.45"/>
       </geometry>
-      <material name="DarkGrey"/>
+      <material name="pal/DarkGrey"/>
     </collision>
   </link>
@@ -121,9 +121,5 @@
           filename="package://tiago_pro_description/meshes/torso/torso_lift_link.stl" />
       </geometry>
-      <material
-        name="">
-        <color
-          rgba="0.752941176470588 0.752941176470588 0.752941176470588 1" />
-      </material>
+      <material name="White"/>
     </visual>
     <collision>

Commit message: Change arm_ft_ to wrist_ft to match TIAGo

File: tiago_pro_description/robots/tiago_pro.urdf.xacro (robot description, xacro)
@@ -57,9 +57,9 @@
 <xacro:property name="has_end_effector_left"
   value="${end_effector_left not in ['false', 'False', 'no-ee']}" />
-<xacro:property name="end_effector_left_link" value="${'arm_left_ft_tool_link' if has_ft_sensor_left else 'arm_left_tool_link'}" />
+<xacro:property name="end_effector_left_link" value="${'wrist_left_ft_tool_link' if has_ft_sensor_left else 'arm_left_tool_link'}" />
 <xacro:property name="end_effector_left_name" value="gripper_left" />
 <xacro:property name="has_end_effector_right"
   value="${end_effector_right not in ['false', 'False', 'no-ee']}" />
-<xacro:property name="end_effector_right_link" value="${'arm_right_ft_tool_link' if has_ft_sensor_right else 'arm_right_tool_link'}" />
+<xacro:property name="end_effector_right_link" value="${'wrist_right_ft_tool_link' if has_ft_sensor_right else 'arm_right_tool_link'}" />
 <xacro:property name="end_effector_right_name" value="gripper_right" />
 <!-- Base -->
@@ -85,8 +85,8 @@
 <!-- FT sensors -->
 <xacro:if value="${has_ft_sensor_right}">
-    <xacro:ft_sensor name="arm_right" parent="arm_right_tool_link"/>
+    <xacro:ft_sensor name="wrist_right" parent="arm_right_tool_link"/>
 </xacro:if>
 <xacro:if value="${has_ft_sensor_left}">
-    <xacro:ft_sensor name="arm_left" parent="arm_left_tool_link"/>
+    <xacro:ft_sensor name="wrist_left" parent="arm_left_tool_link"/>
 </xacro:if>
 <!-- Grippers -->

Commit message: fix misaligned

File: tiago_pro_description/robots/tiago_pro.urdf.xacro (robot description, xacro)
@@ -39,10 +39,8 @@
 <xacro:property name="arm_model" value="tiago-pro" />
 <xacro:property name="description_calibration_dir"       value="${arg description_calibration_dir}"/>
-<xacro:if
-  value="${end_effector_left not in ['pal-pro-gripper', 'custom', 'no-ee']}">
+<xacro:if value="${end_effector_left not in ['pal-pro-gripper', 'custom', 'no-ee']}">
   <xacro:wrong_end_effector_left />
 </xacro:if>
-<xacro:if
-  value="${end_effector_right not in ['pal-pro-gripper', 'custom', 'no-ee']}">
+<xacro:if value="${end_effector_right not in ['pal-pro-gripper', 'custom', 'no-ee']}">
   <xacro:wrong_end_effector_right />
 </xacro:if>
@@ -53,12 +51,10 @@
   <xacro:wrong_ft_sensor_right />
 </xacro:if>
-<xacro:if
-  value="${laser_model not in ['no-laser', 'sick-551', 'sick-561', 'sick-571', 'hokuyo', 'ydlidar-tg30', 'ydlidar-tg15']}">
+<xacro:if value="${laser_model not in ['no-laser', 'sick-551', 'sick-561', 'sick-571', 'hokuyo', 'ydlidar-tg30', 'ydlidar-tg15']}">
   <xacro:wrong_laser_model />
 </xacro:if>
 <xacro:property name="has_ft_sensor_left"     value="${ft_sensor_left in ['rokubi']}"/>
 <xacro:property name="has_ft_sensor_right"    value="${ft_sensor_right in ['rokubi']}"/>
-<xacro:property name="has_end_effector_left"
-  value="${end_effector_left not in ['no-ee']}" />
+<xacro:property name="has_end_effector_left"  value="${end_effector_left not in ['no-ee']}" />
 <xacro:property name="end_effector_left_link" value="${'wrist_left_ft_tool_link' if has_ft_sensor_left else 'arm_left_tool_link'}" />
 <xacro:property name="end_effector_left_name" value="gripper_left" />

Commit message: Choose to spawn the arms or not in the urdf

File: tiago_pro_description/robots/tiago_pro.urdf.xacro (robot description, xacro)
@@ -25,4 +25,6 @@
 <!-- Parameters -->
 <xacro:arg name="laser_model" default="hokuyo"/> <!-- no-laser, hokuyo, sick-551, sick-561, sick-571-->
+<xacro:arg name="arm_model_left" default="tiago-pro" /> <!-- tiago-pro, no-arm -->
+<xacro:arg name="arm_model_right" default="tiago-pro" /> <!-- tiago-pro, no-arm -->
 <xacro:arg name="end_effector_left" default="pal-pro-gripper" /> <!-- pal-pro-gripper custom-->
 <xacro:arg name="end_effector_right" default="pal-pro-gripper" /> <!-- pal-pro-gripper, custom-->
@@ -33,4 +35,6 @@
 <xacro:arg name="extrinsic_calibration_dir" default="$(find tiago_pro_description)/urdf"/>
 <xacro:property name="laser_model" value="$(arg laser_model)" />
+<xacro:property name="arm_model_left" value="$(arg arm_model_left)" />
+<xacro:property name="arm_model_right" value="$(arg arm_model_right)" />
 <xacro:property name="end_effector_left" value="$(arg end_effector_left)" />
 <xacro:property name="end_effector_right" value="$(arg end_effector_right)" />
@@ -39,8 +43,14 @@
 <xacro:property name="arm_model" value="tiago-pro" />
 <xacro:property name="description_calibration_dir"       value="${arg description_calibration_dir}"/>
-<xacro:if value="${end_effector_left not in ['pal-pro-gripper', 'custom', 'no-ee']}">
+<xacro:if value="${arm_model_left not in ['tiago-pro', 'no-arm']}">
+  <xacro:wrong_arm_model_left />
+</xacro:if>
+<xacro:if value="${arm_model_right not in ['tiago-pro', 'no-arm']}">
+  <xacro:wrong_arm_model_right />
+</xacro:if>
+<xacro:if value="${end_effector_left not in ['pal-pro-gripper', 'custom', 'no-end-effector']}">
   <xacro:wrong_end_effector_left />
 </xacro:if>
-<xacro:if value="${end_effector_right not in ['pal-pro-gripper', 'custom', 'no-ee']}">
+<xacro:if value="${end_effector_right not in ['pal-pro-gripper', 'custom', 'no-end-effector']}">
   <xacro:wrong_end_effector_right />
 </xacro:if>
@@ -51,13 +61,15 @@
   <xacro:wrong_ft_sensor_right />
 </xacro:if>
-<xacro:if value="${laser_model not in ['no-laser', 'sick-551', 'sick-561', 'sick-571', 'hokuyo', 'ydlidar-tg30', 'ydlidar-tg15']}">
+<xacro:if value="${laser_model not in ['no-laser', 'sick-551', 'sick-561', 'sick-571', 'hokuyo']}">
   <xacro:wrong_laser_model />
 </xacro:if>
-<xacro:property name="has_ft_sensor_left"     value="${ft_sensor_left in ['rokubi']}"/>
-<xacro:property name="has_ft_sensor_right"    value="${ft_sensor_right in ['rokubi']}"/>
-<xacro:property name="has_end_effector_left"  value="${end_effector_left not in ['no-ee']}" />
+<xacro:property name="has_arm_left"    value="${arm_model_left not in ['no-arm']}"/>
+<xacro:property name="has_ft_sensor_left"     value="${ft_sensor_left not in ['no-ft-sensor']}"/>
+<xacro:property name="has_end_effector_left"  value="${end_effector_left not in ['no-end-effector']}" />
 <xacro:property name="end_effector_left_link" value="${'wrist_left_ft_tool_link' if has_ft_sensor_left else 'arm_left_tool_link'}" />
 <xacro:property name="end_effector_left_name" value="gripper_left" />
-<xacro:property name="has_end_effector_right"  value="${end_effector_right not in ['no-ee']}" />
+<xacro:property name="has_arm_right"    value="${arm_model_right not in ['no-arm']}"/>
+<xacro:property name="has_ft_sensor_right"    value="${ft_sensor_right not in ['no-ft-sensor']}"/>
+<xacro:property name="has_end_effector_right"  value="${end_effector_right not in ['no-end-effector']}" />
 <xacro:property name="end_effector_right_link" value="${'wrist_right_ft_tool_link' if has_ft_sensor_right else 'arm_right_tool_link'}" />
 <xacro:property name="end_effector_right_name" value="gripper_right" />
@@ -75,22 +87,26 @@
 <!-- Arms -->
 <xacro:include filename="$(arg description_calibration_dir)/calibration_constants.urdf.xacro" />
-<xacro:pal_sea_arm name="arm_left" parent="torso_lift_link"  arm_model="${arm_model}" reflect="1" arm_1_offset="${arm_left_1_joint_offset}" arm_2_offset="${arm_left_2_joint_offset}" arm_3_offset="${arm_left_3_joint_offset}" arm_4_offset="${arm_left_4_joint_offset}" arm_5_offset="${arm_left_5_joint_offset}" arm_6_offset="${arm_left_6_joint_offset}" arm_7_offset="${arm_left_7_joint_offset}">
-  <origin xyz="$(arg arm_x) $(arg arm_y) $(arg arm_z)"
-          rpy="$(arg arm_roll) $(arg arm_pitch) $(arg arm_yaw)"/>
-</xacro:pal_sea_arm>
-<xacro:pal_sea_arm name="arm_right" parent="torso_lift_link"  arm_model="${arm_model}" reflect="1" arm_1_offset="${arm_right_1_joint_offset}" arm_2_offset="${arm_right_2_joint_offset}" arm_3_offset="${arm_right_3_joint_offset}" arm_4_offset="${arm_right_4_joint_offset}" arm_5_offset="${arm_right_5_joint_offset}" arm_6_offset="${arm_right_6_joint_offset}" arm_7_offset="${arm_right_7_joint_offset}">
-  <origin xyz="$(arg arm_x) ${-1.0*$(arg arm_y)} $(arg arm_z)"
-	  rpy="$(arg arm_roll) ${-1.0*$(arg arm_pitch)} ${-3.14159 -$(arg arm_yaw)}"/>
-</xacro:pal_sea_arm>
-<!-- FT sensors -->
-<xacro:if value="${has_ft_sensor_right}">
+<xacro:if value="${has_arm_left}">
+  <xacro:pal_sea_arm name="arm_left" parent="torso_lift_link"  arm_model="${arm_model_left}" reflect="1" arm_1_offset="${arm_left_1_joint_offset}" arm_2_offset="${arm_left_2_joint_offset}" arm_3_offset="${arm_left_3_joint_offset}" arm_4_offset="${arm_left_4_joint_offset}" arm_5_offset="${arm_left_5_joint_offset}" arm_6_offset="${arm_left_6_joint_offset}" arm_7_offset="${arm_left_7_joint_offset}">
+    <origin xyz="$(arg arm_x) $(arg arm_y) $(arg arm_z)"
+            rpy="$(arg arm_roll) $(arg arm_pitch) $(arg arm_yaw)"/>
+  </xacro:pal_sea_arm>
+  <!-- FT sensors -->
+  <xacro:if value="${has_ft_sensor_left}">
+      <xacro:ft_sensor name="wrist_left" parent="arm_left_tool_link"/>
+  </xacro:if>
+  <xacro:pal_sea_arm_end_effector name="gripper_left" parent="${end_effector_left_link}" type="${end_effector_left}" has_end_effector="${has_end_effector_left}" reflect="-1" is_dual="true"/>
+</xacro:if>
+<xacro:if value="${has_arm_right}">
+  <xacro:pal_sea_arm name="arm_right" parent="torso_lift_link"  arm_model="${arm_model_right}" reflect="1" arm_1_offset="${arm_right_1_joint_offset}" arm_2_offset="${arm_right_2_joint_offset}" arm_3_offset="${arm_right_3_joint_offset}" arm_4_offset="${arm_right_4_joint_offset}" arm_5_offset="${arm_right_5_joint_offset}" arm_6_offset="${arm_right_6_joint_offset}" arm_7_offset="${arm_right_7_joint_offset}">
+    <origin xyz="$(arg arm_x) ${-1.0*$(arg arm_y)} $(arg arm_z)"
+      rpy="$(arg arm_roll) ${-1.0*$(arg arm_pitch)} ${-3.14159 -$(arg arm_yaw)}"/>
+  </xacro:pal_sea_arm>
+  <!-- FT sensors -->
+  <xacro:if value="${has_ft_sensor_right}">
     <xacro:ft_sensor name="wrist_right" parent="arm_right_tool_link"/>
+  </xacro:if>
+  <xacro:pal_sea_arm_end_effector name="gripper_right" parent="${end_effector_right_link}" type="${end_effector_right}" has_end_effector="${has_end_effector_right}" reflect="1" is_dual="true"/>
 </xacro:if>
-<xacro:if value="${has_ft_sensor_left}">
-    <xacro:ft_sensor name="wrist_left" parent="arm_left_tool_link"/>
-</xacro:if>
-<!-- Grippers -->
-<xacro:pal_sea_arm_end_effector name="gripper_left" parent="${end_effector_left_link}" type="${end_effector_left}" has_end_effector="${has_end_effector_left}" reflect="-1" is_dual="true"/>
-<xacro:pal_sea_arm_end_effector name="gripper_right" parent="${end_effector_right_link}" type="${end_effector_right}" has_end_effector="${has_end_effector_right}" reflect="1" is_dual="true"/>
 <!-- ROS 2 Control -->
 <xacro:include filename="$(find tiago_pro_description)/ros2_control/ros2_control.urdf.xacro" />

File: tiago_pro_description/ros2_control/ros2_control.urdf.xacro (robot description, xacro)
@@ -15,5 +15,6 @@
        name="tiago_pro" >
   <xacro:macro name="tiago_pro_ros2_control" params="use_sim:=^|false">
-    <xacro:arg name="arm_model" default="tiago-pro"/>
+    <xacro:arg name="arm_model_left" default="tiago-pro"/>
+    <xacro:arg name="arm_model_right" default="tiago-pro"/>
     <xacro:arg name="end_effector_left" default="pal-pro-pripper"/>
     <xacro:arg name="end_effector_right" default="pal-pro-gripper"/>
@@ -21,8 +22,12 @@
     <xacro:arg name="ft_sensor_right" default="no-ft-sensor"/>
     <xacro:arg name="description_calibration_dir" default="$(find tiago_pro_description)/urdf/calibration" /> <!-- TODO-->
+    <xacro:property name="arm_model_left" value="$(arg arm_model_left)" />
+    <xacro:property name="arm_model_right" value="$(arg arm_model_right)" />
     <xacro:property name="end_effector_left" value="$(arg end_effector_left)" />
     <xacro:property name="end_effector_right" value="$(arg end_effector_right)" />
     <xacro:property name="has_ft_sensor_left" value="${ft_sensor_left != 'no-ft-sensor'}" />
     <xacro:property name="has_ft_sensor_right" value="${ft_sensor_right != 'no-ft-sensor'}" />
+    <xacro:property name="has_arm_left" value="${arm_model_left != 'no-arm'}" />
+    <xacro:property name="has_arm_right" value="${arm_model_right != 'no-arm'}" />
     <xacro:include filename="$(find omni_base_description)/urdf/sensors/sensors.ros2_control.xacro" />
     <xacro:include filename="$(find omni_base_description)/urdf/wheels/wheel.ros2_control.xacro" />
@@ -59,35 +64,37 @@
       <xacro:ros2_control_head name="head_2" reduction="1.0" offset_value="${head_2_joint_offset}" />
       <!-- arm left -->
-      <xacro:ros2_control_arm name="arm_left_1" reduction="1.0" offset_value="${arm_left_1_joint_offset}" />
-      <xacro:ros2_control_arm name="arm_left_2" reduction="1.0" offset_value="${arm_left_2_joint_offset}" />
-      <xacro:ros2_control_arm name="arm_left_3" reduction="1.0" offset_value="${arm_left_3_joint_offset}" />
-      <xacro:ros2_control_arm name="arm_left_4" reduction="1.0" offset_value="${arm_left_4_joint_offset}" />
-      <xacro:ros2_control_arm name="arm_left_5" reduction="1.0" offset_value="${arm_left_5_joint_offset}" />
-      <xacro:ros2_control_arm name="arm_left_6" reduction="1.0" offset_value="${arm_left_6_joint_offset}" />
-      <xacro:ros2_control_arm name="arm_left_7" reduction="1.0" offset_value="${arm_left_7_joint_offset}" />
+      <xacro:if value="${has_arm_left}">
+        <xacro:ros2_control_arm name="arm_left_1" reduction="1.0" offset_value="${arm_left_1_joint_offset}" />
+        <xacro:ros2_control_arm name="arm_left_2" reduction="1.0" offset_value="${arm_left_2_joint_offset}" />
+        <xacro:ros2_control_arm name="arm_left_3" reduction="1.0" offset_value="${arm_left_3_joint_offset}" />
+        <xacro:ros2_control_arm name="arm_left_4" reduction="1.0" offset_value="${arm_left_4_joint_offset}" />
+        <xacro:ros2_control_arm name="arm_left_5" reduction="1.0" offset_value="${arm_left_5_joint_offset}" />
+        <xacro:ros2_control_arm name="arm_left_6" reduction="1.0" offset_value="${arm_left_6_joint_offset}" />
+        <xacro:ros2_control_arm name="arm_left_7" reduction="1.0" offset_value="${arm_left_7_joint_offset}" />
+        <xacro:if value="${has_ft_sensor_left}">
+          <xacro:include filename="$(find pal_sea_arm_description)/urdf/sensors/sensors.ros2_control.xacro"/>
+          <xacro:ros2_control_force_torque_sensor name="wrist_left_ft_sensor"/>
+        </xacro:if>
+        <xacro:if value="${end_effector_left == 'pal-pro-gripper'}">
+          <xacro:ros2_control_pal_pro_gripper name="gripper_left" reduction="1.0" />
+        </xacro:if>
+      </xacro:if>
       <!-- arm right -->
-      <xacro:ros2_control_arm name="arm_right_1" reduction="1.0" offset_value="${arm_right_1_joint_offset}" />
-      <xacro:ros2_control_arm name="arm_right_2" reduction="1.0" offset_value="${arm_right_2_joint_offset}" />
-      <xacro:ros2_control_arm name="arm_right_3" reduction="1.0" offset_value="${arm_right_3_joint_offset}" />
-      <xacro:ros2_control_arm name="arm_right_4" reduction="1.0" offset_value="${arm_right_4_joint_offset}" />
-      <xacro:ros2_control_arm name="arm_right_5" reduction="1.0" offset_value="${arm_right_5_joint_offset}" />
-      <xacro:ros2_control_arm name="arm_right_6" reduction="1.0" offset_value="${arm_right_6_joint_offset}" />
-      <xacro:ros2_control_arm name="arm_right_7" reduction="1.0" offset_value="${arm_right_7_joint_offset}" />
-      <xacro:if value="${end_effector_left == 'pal-pro-gripper'}">
-        <!-- pal-pro-gripper -->
-        <xacro:ros2_control_pal_pro_gripper name="gripper_left" reduction="1.0" />
-      </xacro:if>
-      <xacro:if value="${end_effector_right == 'pal-pro-gripper'}">
-        <!-- pal-pro-gripper -->
-        <xacro:ros2_control_pal_pro_gripper name="gripper_right" reduction="1.0" />
-      </xacro:if>
-      <!-- Force Torque sensor -->
-      <xacro:if value="${has_ft_sensor_left}">
-        <xacro:include filename="$(find pal_sea_arm_description)/urdf/sensors/sensors.ros2_control.xacro"/>
-        <xacro:ros2_control_force_torque_sensor name="wrist_left_ft_sensor"/>
-      </xacro:if>
-      <xacro:if value="${has_ft_sensor_right}">
-        <xacro:include filename="$(find pal_sea_arm_description)/urdf/sensors/sensors.ros2_control.xacro"/>
-        <xacro:ros2_control_force_torque_sensor name="wrist_right_ft_sensor"/>s
+      <xacro:if value="${has_arm_right}">
+        <xacro:ros2_control_arm name="arm_right_1" reduction="1.0" offset_value="${arm_right_1_joint_offset}" />
+        <xacro:ros2_control_arm name="arm_right_2" reduction="1.0" offset_value="${arm_right_2_joint_offset}" />
+        <xacro:ros2_control_arm name="arm_right_3" reduction="1.0" offset_value="${arm_right_3_joint_offset}" />
+        <xacro:ros2_control_arm name="arm_right_4" reduction="1.0" offset_value="${arm_right_4_joint_offset}" />
+        <xacro:ros2_control_arm name="arm_right_5" reduction="1.0" offset_value="${arm_right_5_joint_offset}" />
+        <xacro:ros2_control_arm name="arm_right_6" reduction="1.0" offset_value="${arm_right_6_joint_offset}" />
+        <xacro:ros2_control_arm name="arm_right_7" reduction="1.0" offset_value="${arm_right_7_joint_offset}" />
+        <xacro:if value="${has_ft_sensor_right}">
+          <xacro:include filename="$(find pal_sea_arm_description)/urdf/sensors/sensors.ros2_control.xacro"/>
+          <xacro:ros2_control_force_torque_sensor name="wrist_right_ft_sensor"/>s
+        </xacro:if>
+        <xacro:if value="${end_effector_right == 'pal-pro-gripper'}">
+          <!-- pal-pro-gripper -->
+          <xacro:ros2_control_pal_pro_gripper name="gripper_right" reduction="1.0" />
+        </xacro:if>
       </xacro:if>
     </ros2_control>
