Commit message: Applying autoformater

File: tiago_pro_description/robots/tiago_pro.urdf.xacro (robot description, xacro)
@@ -12,103 +12,108 @@
   limitations under the License.
 -->
-<robot  xmlns:xacro="http://ros.org/wiki/xacro" name="tiago_pro">
-<!-- Includes -->
-<xacro:include filename="$(find pal_urdf_utils)/urdf/deg_to_rad.urdf.xacro" />
-<xacro:include filename="$(find pal_urdf_utils)/urdf/materials.urdf.xacro" />
-<xacro:include filename="$(find tiago_pro_description)/gazebo/gazebo.urdf.xacro" />
-<xacro:include filename="$(find tiago_pro_description)/urdf/torso/torso_dual.urdf.xacro" />
-<xacro:include filename="$(find tiago_pro_description)/urdf/head/head.urdf.xacro" />
-<xacro:include filename="$(find omni_base_description)/urdf/base/base_sensors.urdf.xacro" />
-<xacro:include filename="$(find pal_sea_arm_description)/urdf/arm/arm.urdf.xacro" />
-<xacro:include filename="$(find pal_sea_arm_description)/urdf/end_effector/end_effector.urdf.xacro" />
-<xacro:include filename="$(find pal_sea_arm_description)/urdf/sensors/ft_sensor.urdf.xacro" />
-<!-- Parameters -->
-<xacro:arg name="laser_model" default="hokuyo"/> <!-- no-laser, hokuyo, sick-551, sick-561, sick-571-->
-<xacro:arg name="arm_model_left" default="tiago-pro" /> <!-- tiago-pro, no-arm -->
-<xacro:arg name="arm_model_right" default="tiago-pro" /> <!-- tiago-pro, no-arm -->
-<xacro:arg name="end_effector_left" default="pal-pro-gripper" /> <!-- pal-pro-gripper custom-->
-<xacro:arg name="end_effector_right" default="pal-pro-gripper" /> <!-- pal-pro-gripper, custom-->
-<xacro:arg name="ft_sensor_left" default="no-ft-sensor" /> <!-- no-ft-sensor, rokubi -->
-<xacro:arg name="ft_sensor_right" default="no-ft-sensor" /> <!-- no-ft-sensor, rokubi -->
-<xacro:arg name="use_sim" default="false"/>
-<xacro:arg name="description_calibration_dir" default="$(find tiago_pro_description)/urdf"/>
-<xacro:arg name="extrinsic_calibration_dir" default="$(find tiago_pro_description)/urdf"/>
-<xacro:property name="laser_model" value="$(arg laser_model)" />
-<xacro:property name="arm_model_left" value="$(arg arm_model_left)" />
-<xacro:property name="arm_model_right" value="$(arg arm_model_right)" />
-<xacro:property name="end_effector_left" value="$(arg end_effector_left)" />
-<xacro:property name="end_effector_right" value="$(arg end_effector_right)" />
-<xacro:property name="ft_sensor_left" value="$(arg ft_sensor_left)" />
-<xacro:property name="ft_sensor_right" value="$(arg ft_sensor_right)" />
-<xacro:property name="arm_model" value="tiago-pro" />
-<xacro:property name="description_calibration_dir"       value="${arg description_calibration_dir}"/>
-<xacro:if value="${arm_model_left not in ['tiago-pro', 'no-arm']}">
-  <xacro:wrong_arm_model_left />
-</xacro:if>
-<xacro:if value="${arm_model_right not in ['tiago-pro', 'no-arm']}">
-  <xacro:wrong_arm_model_right />
-</xacro:if>
-<xacro:if value="${end_effector_left not in ['pal-pro-gripper', 'custom', 'no-end-effector']}">
-  <xacro:wrong_end_effector_left />
-</xacro:if>
-<xacro:if value="${end_effector_right not in ['pal-pro-gripper', 'custom', 'no-end-effector']}">
-  <xacro:wrong_end_effector_right />
-</xacro:if>
-<xacro:if value="${ft_sensor_left not in ['no-ft-sensor', 'rokubi']}">
-  <xacro:wrong_ft_sensor_left />
-</xacro:if>
-<xacro:if value="${ft_sensor_right not in ['no-ft-sensor', 'rokubi']}">
-  <xacro:wrong_ft_sensor_right />
-</xacro:if>
-<xacro:if value="${laser_model not in ['no-laser', 'sick-571']}">
-  <xacro:wrong_laser_model />
-</xacro:if>
-<xacro:property name="has_arm_left"    value="${arm_model_left not in ['no-arm']}"/>
-<xacro:property name="has_ft_sensor_left"     value="${ft_sensor_left not in ['no-ft-sensor']}"/>
-<xacro:property name="has_end_effector_left"  value="${end_effector_left not in ['no-end-effector']}" />
-<xacro:property name="end_effector_left_link" value="${'wrist_left_ft_tool_link' if has_ft_sensor_left else 'arm_left_tool_link'}" />
-<xacro:property name="end_effector_left_name" value="gripper_left" />
-<xacro:property name="has_arm_right"    value="${arm_model_right not in ['no-arm']}"/>
-<xacro:property name="has_ft_sensor_right"    value="${ft_sensor_right not in ['no-ft-sensor']}"/>
-<xacro:property name="has_end_effector_right"  value="${end_effector_right not in ['no-end-effector']}" />
-<xacro:property name="end_effector_right_link" value="${'wrist_right_ft_tool_link' if has_ft_sensor_right else 'arm_right_tool_link'}" />
-<xacro:property name="end_effector_right_name" value="gripper_right" />
-<!-- Base -->
-<xacro:base_sensors name="base" front_laser_model="$(arg laser_model)" rear_laser_model="$(arg laser_model)"/>
-<!-- Torso. TODO:change for custom torso -->
-<xacro:tiago_pro_torso name="torso" parent="base_link"/>
-<xacro:tiago_pro_head name="head" parent="torso_lift_link"/>
-<xacro:arg name="arm_x" default="0.08976" />
-<xacro:arg name="arm_y" default="0.15918" />
-<xacro:arg name="arm_z" default="-0.092008" />
-<xacro:arg name="arm_roll" default="-2.0679" />
-<xacro:arg name="arm_pitch" default="0.0" />
-<xacro:arg name="arm_yaw" default="-1.2217" />
-<!-- Arms -->
-<xacro:include filename="$(arg description_calibration_dir)/calibration_constants.urdf.xacro" />
-<xacro:if value="${has_arm_left}">
-  <xacro:pal_sea_arm name="arm_left" parent="torso_lift_link"  arm_model="${arm_model_left}" reflect="1" arm_1_offset="${arm_left_1_joint_offset}" arm_2_offset="${arm_left_2_joint_offset}" arm_3_offset="${arm_left_3_joint_offset}" arm_4_offset="${arm_left_4_joint_offset}" arm_5_offset="${arm_left_5_joint_offset}" arm_6_offset="${arm_left_6_joint_offset}" arm_7_offset="${arm_left_7_joint_offset}">
-    <origin xyz="$(arg arm_x) $(arg arm_y) $(arg arm_z)"
-            rpy="$(arg arm_roll) $(arg arm_pitch) $(arg arm_yaw)"/>
-  </xacro:pal_sea_arm>
-  <!-- FT sensors -->
-  <xacro:if value="${has_ft_sensor_left}">
+<robot xmlns:xacro="http://ros.org/wiki/xacro" name="tiago_pro">
+  <!-- Includes -->
+  <xacro:include filename="$(find pal_urdf_utils)/urdf/deg_to_rad.urdf.xacro" />
+  <xacro:include filename="$(find pal_urdf_utils)/urdf/materials.urdf.xacro" />
+  <xacro:include filename="$(find tiago_pro_description)/gazebo/gazebo.urdf.xacro" />
+  <xacro:include filename="$(find tiago_pro_description)/urdf/torso/torso_dual.urdf.xacro" />
+  <xacro:include filename="$(find tiago_pro_description)/urdf/head/head.urdf.xacro" />
+  <xacro:include filename="$(find omni_base_description)/urdf/base/base_sensors.urdf.xacro" />
+  <xacro:include filename="$(find pal_sea_arm_description)/urdf/arm/arm.urdf.xacro" />
+  <xacro:include filename="$(find pal_sea_arm_description)/urdf/end_effector/end_effector.urdf.xacro" />
+  <xacro:include filename="$(find pal_sea_arm_description)/urdf/sensors/ft_sensor.urdf.xacro" />
+  <!-- Parameters -->
+  <xacro:arg name="laser_model" default="hokuyo"/>
+  <!-- no-laser, hokuyo, sick-551, sick-561, sick-571-->
+  <xacro:arg name="arm_model_left" default="tiago-pro" />
+  <!-- tiago-pro, no-arm -->
+  <xacro:arg name="arm_model_right" default="tiago-pro" />
+  <!-- tiago-pro, no-arm -->
+  <xacro:arg name="end_effector_left" default="pal-pro-gripper" />
+  <!-- pal-pro-gripper custom-->
+  <xacro:arg name="end_effector_right" default="pal-pro-gripper" />
+  <!-- pal-pro-gripper, custom-->
+  <xacro:arg name="ft_sensor_left" default="no-ft-sensor" />
+  <!-- no-ft-sensor, rokubi -->
+  <xacro:arg name="ft_sensor_right" default="no-ft-sensor" />
+  <!-- no-ft-sensor, rokubi -->
+  <xacro:arg name="use_sim" default="false"/>
+  <xacro:arg name="description_calibration_dir" default="$(find tiago_pro_description)/urdf"/>
+  <xacro:arg name="extrinsic_calibration_dir" default="$(find tiago_pro_description)/urdf"/>
+  <xacro:property name="laser_model" value="$(arg laser_model)" />
+  <xacro:property name="arm_model_left" value="$(arg arm_model_left)" />
+  <xacro:property name="arm_model_right" value="$(arg arm_model_right)" />
+  <xacro:property name="end_effector_left" value="$(arg end_effector_left)" />
+  <xacro:property name="end_effector_right" value="$(arg end_effector_right)" />
+  <xacro:property name="ft_sensor_left" value="$(arg ft_sensor_left)" />
+  <xacro:property name="ft_sensor_right" value="$(arg ft_sensor_right)" />
+  <xacro:property name="arm_model" value="tiago-pro" />
+  <xacro:property name="description_calibration_dir" value="${arg description_calibration_dir}"/>
+  <xacro:if value="${arm_model_left not in ['tiago-pro', 'no-arm']}">
+    <xacro:wrong_arm_model_left />
+  </xacro:if>
+  <xacro:if value="${arm_model_right not in ['tiago-pro', 'no-arm']}">
+    <xacro:wrong_arm_model_right />
+  </xacro:if>
+  <xacro:if value="${end_effector_left not in ['pal-pro-gripper', 'custom', 'no-end-effector']}">
+    <xacro:wrong_end_effector_left />
+  </xacro:if>
+  <xacro:if value="${end_effector_right not in ['pal-pro-gripper', 'custom', 'no-end-effector']}">
+    <xacro:wrong_end_effector_right />
+  </xacro:if>
+  <xacro:if value="${ft_sensor_left not in ['no-ft-sensor', 'rokubi']}">
+    <xacro:wrong_ft_sensor_left />
+  </xacro:if>
+  <xacro:if value="${ft_sensor_right not in ['no-ft-sensor', 'rokubi']}">
+    <xacro:wrong_ft_sensor_right />
+  </xacro:if>
+  <xacro:if value="${laser_model not in ['no-laser', 'sick-571']}">
+    <xacro:wrong_laser_model />
+  </xacro:if>
+  <xacro:property name="has_arm_left" value="${arm_model_left not in ['no-arm']}"/>
+  <xacro:property name="has_ft_sensor_left" value="${ft_sensor_left not in ['no-ft-sensor']}"/>
+  <xacro:property name="has_end_effector_left" value="${end_effector_left not in ['no-end-effector']}" />
+  <xacro:property name="end_effector_left_link" value="${'wrist_left_ft_tool_link' if has_ft_sensor_left else 'arm_left_tool_link'}" />
+  <xacro:property name="end_effector_left_name" value="gripper_left" />
+  <xacro:property name="has_arm_right" value="${arm_model_right not in ['no-arm']}"/>
+  <xacro:property name="has_ft_sensor_right" value="${ft_sensor_right not in ['no-ft-sensor']}"/>
+  <xacro:property name="has_end_effector_right" value="${end_effector_right not in ['no-end-effector']}" />
+  <xacro:property name="end_effector_right_link" value="${'wrist_right_ft_tool_link' if has_ft_sensor_right else 'arm_right_tool_link'}" />
+  <xacro:property name="end_effector_right_name" value="gripper_right" />
+  <!-- Base -->
+  <xacro:base_sensors name="base" front_laser_model="$(arg laser_model)" rear_laser_model="$(arg laser_model)"/>
+  <!-- Torso. TODO:change for custom torso -->
+  <xacro:tiago_pro_torso name="torso" parent="base_link"/>
+  <xacro:tiago_pro_head name="head" parent="torso_lift_link"/>
+  <xacro:arg name="arm_x" default="0.08976" />
+  <xacro:arg name="arm_y" default="0.15918" />
+  <xacro:arg name="arm_z" default="-0.092008" />
+  <xacro:arg name="arm_roll" default="-2.0679" />
+  <xacro:arg name="arm_pitch" default="0.0" />
+  <xacro:arg name="arm_yaw" default="-1.2217" />
+  <!-- Arms -->
+  <xacro:include filename="$(arg description_calibration_dir)/calibration_constants.urdf.xacro" />
+  <xacro:if value="${has_arm_left}">
+    <xacro:pal_sea_arm name="arm_left" parent="torso_lift_link" arm_model="${arm_model_left}" reflect="1" arm_1_offset="${arm_left_1_joint_offset}" arm_2_offset="${arm_left_2_joint_offset}" arm_3_offset="${arm_left_3_joint_offset}" arm_4_offset="${arm_left_4_joint_offset}" arm_5_offset="${arm_left_5_joint_offset}" arm_6_offset="${arm_left_6_joint_offset}" arm_7_offset="${arm_left_7_joint_offset}">
+      <origin xyz="$(arg arm_x) $(arg arm_y) $(arg arm_z)" rpy="$(arg arm_roll) $(arg arm_pitch) $(arg arm_yaw)"/>
+    </xacro:pal_sea_arm>
+    <!-- FT sensors -->
+    <xacro:if value="${has_ft_sensor_left}">
       <xacro:ft_sensor name="wrist_left" parent="arm_left_tool_link"/>
+    </xacro:if>
+    <xacro:pal_sea_arm_end_effector name="gripper_left" parent="${end_effector_left_link}" type="${end_effector_left}" has_end_effector="${has_end_effector_left}" reflect="-1" is_dual="true"/>
   </xacro:if>
-  <xacro:pal_sea_arm_end_effector name="gripper_left" parent="${end_effector_left_link}" type="${end_effector_left}" has_end_effector="${has_end_effector_left}" reflect="-1" is_dual="true"/>
-</xacro:if>
-<xacro:if value="${has_arm_right}">
-  <xacro:pal_sea_arm name="arm_right" parent="torso_lift_link"  arm_model="${arm_model_right}" reflect="1" arm_1_offset="${arm_right_1_joint_offset}" arm_2_offset="${arm_right_2_joint_offset}" arm_3_offset="${arm_right_3_joint_offset}" arm_4_offset="${arm_right_4_joint_offset}" arm_5_offset="${arm_right_5_joint_offset}" arm_6_offset="${arm_right_6_joint_offset}" arm_7_offset="${arm_right_7_joint_offset}">
-    <origin xyz="$(arg arm_x) ${-1.0*$(arg arm_y)} $(arg arm_z)"
-      rpy="$(arg arm_roll) ${-1.0*$(arg arm_pitch)} ${-3.14159 -$(arg arm_yaw)}"/>
-  </xacro:pal_sea_arm>
-  <!-- FT sensors -->
-  <xacro:if value="${has_ft_sensor_right}">
-    <xacro:ft_sensor name="wrist_right" parent="arm_right_tool_link"/>
+  <xacro:if value="${has_arm_right}">
+    <xacro:pal_sea_arm name="arm_right" parent="torso_lift_link" arm_model="${arm_model_right}" reflect="1" arm_1_offset="${arm_right_1_joint_offset}" arm_2_offset="${arm_right_2_joint_offset}" arm_3_offset="${arm_right_3_joint_offset}" arm_4_offset="${arm_right_4_joint_offset}" arm_5_offset="${arm_right_5_joint_offset}" arm_6_offset="${arm_right_6_joint_offset}" arm_7_offset="${arm_right_7_joint_offset}">
+      <origin xyz="$(arg arm_x) ${-1.0*$(arg arm_y)} $(arg arm_z)" rpy="$(arg arm_roll) ${-1.0*$(arg arm_pitch)} ${-3.14159 -$(arg arm_yaw)}"/>
+    </xacro:pal_sea_arm>
+    <!-- FT sensors -->
+    <xacro:if value="${has_ft_sensor_right}">
+      <xacro:ft_sensor name="wrist_right" parent="arm_right_tool_link"/>
+    </xacro:if>
+    <xacro:pal_sea_arm_end_effector name="gripper_right" parent="${end_effector_right_link}" type="${end_effector_right}" has_end_effector="${has_end_effector_right}" reflect="1" is_dual="true"/>
   </xacro:if>
-  <xacro:pal_sea_arm_end_effector name="gripper_right" parent="${end_effector_right_link}" type="${end_effector_right}" has_end_effector="${has_end_effector_right}" reflect="1" is_dual="true"/>
-</xacro:if>
-<!-- ROS 2 Control -->
-<xacro:include filename="$(find tiago_pro_description)/ros2_control/ros2_control.urdf.xacro" />
-<xacro:tiago_pro_ros2_control use_sim="$(arg use_sim)" />
+  <!-- ROS 2 Control -->
+  <xacro:include filename="$(find tiago_pro_description)/ros2_control/ros2_control.urdf.xacro" />
+  <xacro:tiago_pro_ros2_control use_sim="$(arg use_sim)" />
 </robot>
