Commit message: Robot urdf reestructured

File: tiago_pro_description/robots/tiago_pro.urdf.xacro (robot description, xacro)
@@ -13,14 +13,4 @@
 -->
 <robot xmlns:xacro="http://ros.org/wiki/xacro" name="tiago_pro">
-  <!-- INCLUDES -->
-  <xacro:include filename="$(find pal_urdf_utils)/urdf/deg_to_rad.urdf.xacro" />
-  <xacro:include filename="$(find pal_urdf_utils)/urdf/materials.urdf.xacro" />
-  <xacro:include filename="$(find tiago_pro_description)/gazebo/gazebo.urdf.xacro" />
-  <xacro:include filename="$(find tiago_pro_description)/urdf/torso/torso_dual.urdf.xacro" />
-  <xacro:include filename="$(find tiago_pro_description)/urdf/head/head.urdf.xacro" />
-  <xacro:include filename="$(find omni_base_description)/urdf/base/base_sensors.urdf.xacro" />
-  <xacro:include filename="$(find pal_sea_arm_description)/urdf/arm/arm.urdf.xacro" />
-  <xacro:include filename="$(find pal_sea_arm_description)/urdf/end_effector/end_effector.urdf.xacro" />
-  <xacro:include filename="$(find pal_sea_arm_description)/urdf/sensors/ft_sensor.urdf.xacro" />
   <!-- ARGUMENTS -->
   <!-- no-laser, sick-571-->
@@ -41,4 +31,10 @@
   <xacro:arg name="description_calibration_dir" default="$(find tiago_pro_description)/urdf"/>
   <xacro:arg name="extrinsic_calibration_dir" default="$(find tiago_pro_description)/urdf"/>
+  <xacro:arg name="arm_x" default="0.08976" />
+  <xacro:arg name="arm_y" default="0.15918" />
+  <xacro:arg name="arm_z" default="-0.092008" />
+  <xacro:arg name="arm_roll" default="-2.0679" />
+  <xacro:arg name="arm_pitch" default="0.0" />
+  <xacro:arg name="arm_yaw" default="-1.2217" />
   <!-- PROPERTIES -->
   <xacro:property name="laser_model" value="$(arg laser_model)" />
@@ -51,4 +47,15 @@
   <xacro:property name="arm_model" value="tiago-pro" />
   <xacro:property name="description_calibration_dir" value="${arg description_calibration_dir}"/>
+  <xacro:property name="has_arm_left" value="${arm_model_left not in ['no-arm']}"/>
+  <xacro:property name="has_ft_sensor_left" value="${ft_sensor_left not in ['no-ft-sensor']}"/>
+  <xacro:property name="has_end_effector_left" value="${end_effector_left not in ['no-end-effector']}" />
+  <xacro:property name="end_effector_left_link" value="${'wrist_left_ft_tool_link' if has_ft_sensor_left else 'arm_left_tool_link'}" />
+  <xacro:property name="end_effector_left_name" value="gripper_left" />
+  <xacro:property name="has_arm_right" value="${arm_model_right not in ['no-arm']}"/>
+  <xacro:property name="has_ft_sensor_right" value="${ft_sensor_right not in ['no-ft-sensor']}"/>
+  <xacro:property name="has_end_effector_right" value="${end_effector_right not in ['no-end-effector']}" />
+  <xacro:property name="end_effector_right_link" value="${'wrist_right_ft_tool_link' if has_ft_sensor_right else 'arm_right_tool_link'}" />
+  <xacro:property name="end_effector_right_name" value="gripper_right" />
+  <!-- Properties check -->
   <xacro:if value="${arm_model_left not in ['tiago-pro', 'no-arm']}">
     <xacro:wrong_arm_model_left />
@@ -72,14 +79,33 @@
     <xacro:wrong_laser_model />
   </xacro:if>
-  <xacro:property name="has_arm_left" value="${arm_model_left not in ['no-arm']}"/>
-  <xacro:property name="has_ft_sensor_left" value="${ft_sensor_left not in ['no-ft-sensor']}"/>
-  <xacro:property name="has_end_effector_left" value="${end_effector_left not in ['no-end-effector']}" />
-  <xacro:property name="end_effector_left_link" value="${'wrist_left_ft_tool_link' if has_ft_sensor_left else 'arm_left_tool_link'}" />
-  <xacro:property name="end_effector_left_name" value="gripper_left" />
-  <xacro:property name="has_arm_right" value="${arm_model_right not in ['no-arm']}"/>
-  <xacro:property name="has_ft_sensor_right" value="${ft_sensor_right not in ['no-ft-sensor']}"/>
-  <xacro:property name="has_end_effector_right" value="${end_effector_right not in ['no-end-effector']}" />
-  <xacro:property name="end_effector_right_link" value="${'wrist_right_ft_tool_link' if has_ft_sensor_right else 'arm_right_tool_link'}" />
-  <xacro:property name="end_effector_right_name" value="gripper_right" />
+  <!-- INCLUDES -->
+  <!-- Tools -->
+  <xacro:include filename="$(find pal_urdf_utils)/urdf/deg_to_rad.urdf.xacro" />
+  <!-- Base -->
+  <xacro:include filename="$(find omni_base_description)/urdf/base/base_sensors.urdf.xacro" />
+  <!-- Torso -->
+  <xacro:include filename="$(find tiago_pro_description)/urdf/torso/torso_dual.urdf.xacro" />
+  <!-- Arm -->
+  <xacro:if value="${has_arm_right or has_arm_left}">
+    <xacro:include filename="$(arg description_calibration_dir)/calibration_constants.urdf.xacro" />
+    <xacro:include filename="$(find pal_sea_arm_description)/urdf/arm/arm.urdf.xacro" />
+  </xacro:if>
+  <!-- End effector -->
+  <xacro:if value="${(has_arm_right or has_arm_left) and (has_end_effector_right or has_end_effector_left)}">
+    <xacro:include filename="$(find pal_sea_arm_description)/urdf/end_effector/end_effector.urdf.xacro" />
+  </xacro:if>
+  <!-- Force Torque sensor -->
+  <xacro:if value="${has_ft_sensor_right or has_ft_sensor_left}">
+    <xacro:include filename="$(find pal_sea_arm_description)/urdf/sensors/ft_sensor.urdf.xacro" />
+    <xacro:include filename="$(find pal_sea_arm_description)/urdf/sensors/ft_sensor.gazebo.xacro" />
+  </xacro:if>
+  <!-- Head -->
+  <xacro:include filename="$(find tiago_pro_description)/urdf/head/head.urdf.xacro" />
+  <!-- Materials for visualization -->
+  <xacro:include filename="$(find pal_urdf_utils)/urdf/materials.urdf.xacro" />
+  <!-- Generic simulator_gazebo plugins -->
+  <xacro:include filename="$(find tiago_pro_description)/gazebo/gazebo.urdf.xacro" />
+  <!-- ROS 2 Control -->
+  <xacro:include filename="$(find tiago_pro_description)/ros2_control/ros2_control.urdf.xacro" />
   <!-- ROBOT DEFINITION -->
   <!-- Base -->
@@ -87,35 +113,37 @@
   <!-- Torso. TODO:change for custom torso -->
   <xacro:tiago_pro_torso name="torso" parent="base_link"/>
+  <!-- Head -->
   <xacro:tiago_pro_head name="head" parent="torso_lift_link"/>
-  <xacro:arg name="arm_x" default="0.08976" />
-  <xacro:arg name="arm_y" default="0.15918" />
-  <xacro:arg name="arm_z" default="-0.092008" />
-  <xacro:arg name="arm_roll" default="-2.0679" />
-  <xacro:arg name="arm_pitch" default="0.0" />
-  <xacro:arg name="arm_yaw" default="-1.2217" />
-  <!-- Arms -->
-  <xacro:include filename="$(arg description_calibration_dir)/calibration_constants.urdf.xacro" />
+  <!-- Left arm -->
   <xacro:if value="${has_arm_left}">
+    <!-- Arm -->
     <xacro:pal_sea_arm name="arm_left" parent="torso_lift_link" arm_model="${arm_model_left}" reflect="1" arm_1_offset="${arm_left_1_joint_offset}" arm_2_offset="${arm_left_2_joint_offset}" arm_3_offset="${arm_left_3_joint_offset}" arm_4_offset="${arm_left_4_joint_offset}" arm_5_offset="${arm_left_5_joint_offset}" arm_6_offset="${arm_left_6_joint_offset}" arm_7_offset="${arm_left_7_joint_offset}">
       <origin xyz="$(arg arm_x) $(arg arm_y) $(arg arm_z)" rpy="$(arg arm_roll) $(arg arm_pitch) $(arg arm_yaw)"/>
     </xacro:pal_sea_arm>
+    <!-- End effector -->
+    <xacro:if value="${has_end_effector_left}">
+      <xacro:pal_sea_arm_end_effector name="gripper_left" parent="${end_effector_left_link}" type="${end_effector_left}" has_end_effector="${has_end_effector_left}" reflect="-1" is_dual="true"/>
+    </xacro:if>
     <!-- FT sensors -->
     <xacro:if value="${has_ft_sensor_left}">
       <xacro:ft_sensor name="wrist_left" parent="arm_left_tool_link"/>
     </xacro:if>
-    <xacro:pal_sea_arm_end_effector name="gripper_left" parent="${end_effector_left_link}" type="${end_effector_left}" has_end_effector="${has_end_effector_left}" reflect="-1" is_dual="true"/>
   </xacro:if>
+  <!-- Right arm -->
   <xacro:if value="${has_arm_right}">
+    <!-- Arm -->
     <xacro:pal_sea_arm name="arm_right" parent="torso_lift_link" arm_model="${arm_model_right}" reflect="1" arm_1_offset="${arm_right_1_joint_offset}" arm_2_offset="${arm_right_2_joint_offset}" arm_3_offset="${arm_right_3_joint_offset}" arm_4_offset="${arm_right_4_joint_offset}" arm_5_offset="${arm_right_5_joint_offset}" arm_6_offset="${arm_right_6_joint_offset}" arm_7_offset="${arm_right_7_joint_offset}">
       <origin xyz="$(arg arm_x) ${-1.0*$(arg arm_y)} $(arg arm_z)" rpy="$(arg arm_roll) ${-1.0*$(arg arm_pitch)} ${-3.14159 -$(arg arm_yaw)}"/>
     </xacro:pal_sea_arm>
+    <!-- End effector -->
+    <xacro:if value="${has_end_effector_right}">
+      <xacro:pal_sea_arm_end_effector name="gripper_right" parent="${end_effector_right_link}" type="${end_effector_right}" has_end_effector="${has_end_effector_right}" reflect="1" is_dual="true"/>
+    </xacro:if>
     <!-- FT sensors -->
     <xacro:if value="${has_ft_sensor_right}">
       <xacro:ft_sensor name="wrist_right" parent="arm_right_tool_link"/>
     </xacro:if>
-    <xacro:pal_sea_arm_end_effector name="gripper_right" parent="${end_effector_right_link}" type="${end_effector_right}" has_end_effector="${has_end_effector_right}" reflect="1" is_dual="true"/>
   </xacro:if>
   <!-- ROS 2 Control -->
-  <xacro:include filename="$(find tiago_pro_description)/ros2_control/ros2_control.urdf.xacro" />
   <xacro:tiago_pro_ros2_control use_sim="$(arg use_sim)" />
 </robot>

Commit message: Changed arm_model to arm_type in the URDF

File: tiago_pro_description/robots/tiago_pro.urdf.xacro (robot description, xacro)
@@ -17,7 +17,7 @@
   <xacro:arg name="laser_model" default="sick-571"/>
   <!-- tiago-pro, no-arm -->
-  <xacro:arg name="arm_model_left" default="tiago-pro" />
+  <xacro:arg name="arm_type_left" default="tiago-pro" />
   <!-- tiago-pro, no-arm -->
-  <xacro:arg name="arm_model_right" default="tiago-pro" />
+  <xacro:arg name="arm_type_right" default="tiago-pro" />
   <!-- pal-pro-gripper custom-->
   <xacro:arg name="end_effector_left" default="pal-pro-gripper" />
@@ -40,19 +40,19 @@
   <!-- PROPERTIES -->
   <xacro:property name="laser_model" value="$(arg laser_model)" />
-  <xacro:property name="arm_model_left" value="$(arg arm_model_left)" />
-  <xacro:property name="arm_model_right" value="$(arg arm_model_right)" />
+  <xacro:property name="arm_type_left" value="$(arg arm_type_left)" />
+  <xacro:property name="arm_type_right" value="$(arg arm_type_right)" />
   <xacro:property name="end_effector_left" value="$(arg end_effector_left)" />
   <xacro:property name="end_effector_right" value="$(arg end_effector_right)" />
   <xacro:property name="ft_sensor_left" value="$(arg ft_sensor_left)" />
   <xacro:property name="ft_sensor_right" value="$(arg ft_sensor_right)" />
-  <xacro:property name="arm_model" value="tiago-pro" />
+  <xacro:property name="arm_type" value="tiago-pro" />
   <xacro:property name="description_calibration_dir" value="${arg description_calibration_dir}"/>
   <xacro:property name="is_public_sim" value="$(arg is_public_sim)" />
-  <xacro:property name="has_arm_left" value="${arm_model_left not in ['no-arm']}"/>
+  <xacro:property name="has_arm_left" value="${arm_type_left not in ['no-arm']}"/>
   <xacro:property name="has_ft_sensor_left" value="${ft_sensor_left not in ['no-ft-sensor']}"/>
   <xacro:property name="has_end_effector_left" value="${end_effector_left not in ['no-end-effector']}" />
   <xacro:property name="end_effector_left_link" value="${'wrist_left_ft_tool_link' if has_ft_sensor_left else 'arm_left_tool_link'}" />
   <xacro:property name="end_effector_left_name" value="gripper_left" />
-  <xacro:property name="has_arm_right" value="${arm_model_right not in ['no-arm']}"/>
+  <xacro:property name="has_arm_right" value="${arm_type_right not in ['no-arm']}"/>
   <xacro:property name="has_ft_sensor_right" value="${ft_sensor_right not in ['no-ft-sensor']}"/>
   <xacro:property name="has_end_effector_right" value="${end_effector_right not in ['no-end-effector']}" />
@@ -60,9 +60,9 @@
   <xacro:property name="end_effector_right_name" value="gripper_right" />
   <!-- Properties check -->
-  <xacro:if value="${arm_model_left not in ['tiago-pro', 'no-arm']}">
-    <xacro:wrong_arm_model_left />
+  <xacro:if value="${arm_type_left not in ['tiago-pro', 'no-arm']}">
+    <xacro:wrong_arm_type_left />
   </xacro:if>
-  <xacro:if value="${arm_model_right not in ['tiago-pro', 'no-arm']}">
-    <xacro:wrong_arm_model_right />
+  <xacro:if value="${arm_type_right not in ['tiago-pro', 'no-arm']}">
+    <xacro:wrong_arm_type_right />
   </xacro:if>
   <xacro:if value="${end_effector_left not in ['pal-pro-gripper', 'custom', 'no-end-effector']}">
@@ -121,5 +121,5 @@
   <xacro:if value="${has_arm_left}">
     <!-- Arm -->
-    <xacro:pal_sea_arm name="arm_left" parent="torso_lift_link" arm_model="${arm_model_left}" reflect="1" arm_1_offset="${arm_left_1_joint_offset}" arm_2_offset="${arm_left_2_joint_offset}" arm_3_offset="${arm_left_3_joint_offset}" arm_4_offset="${arm_left_4_joint_offset}" arm_5_offset="${arm_left_5_joint_offset}" arm_6_offset="${arm_left_6_joint_offset}" arm_7_offset="${arm_left_7_joint_offset}">
+    <xacro:pal_sea_arm name="arm_left" parent="torso_lift_link" arm_type="${arm_type_left}" reflect="1" arm_1_offset="${arm_left_1_joint_offset}" arm_2_offset="${arm_left_2_joint_offset}" arm_3_offset="${arm_left_3_joint_offset}" arm_4_offset="${arm_left_4_joint_offset}" arm_5_offset="${arm_left_5_joint_offset}" arm_6_offset="${arm_left_6_joint_offset}" arm_7_offset="${arm_left_7_joint_offset}">
       <origin xyz="$(arg arm_x) $(arg arm_y) $(arg arm_z)" rpy="$(arg arm_roll) $(arg arm_pitch) $(arg arm_yaw)"/>
     </xacro:pal_sea_arm>
@@ -136,5 +136,5 @@
   <xacro:if value="${has_arm_right}">
     <!-- Arm -->
-    <xacro:pal_sea_arm name="arm_right" parent="torso_lift_link" arm_model="${arm_model_right}" reflect="1" arm_1_offset="${arm_right_1_joint_offset}" arm_2_offset="${arm_right_2_joint_offset}" arm_3_offset="${arm_right_3_joint_offset}" arm_4_offset="${arm_right_4_joint_offset}" arm_5_offset="${arm_right_5_joint_offset}" arm_6_offset="${arm_right_6_joint_offset}" arm_7_offset="${arm_right_7_joint_offset}">
+    <xacro:pal_sea_arm name="arm_right" parent="torso_lift_link" arm_type="${arm_type_right}" reflect="1" arm_1_offset="${arm_right_1_joint_offset}" arm_2_offset="${arm_right_2_joint_offset}" arm_3_offset="${arm_right_3_joint_offset}" arm_4_offset="${arm_right_4_joint_offset}" arm_5_offset="${arm_right_5_joint_offset}" arm_6_offset="${arm_right_6_joint_offset}" arm_7_offset="${arm_right_7_joint_offset}">
       <origin xyz="$(arg arm_x) ${-1.0*$(arg arm_y)} $(arg arm_z)" rpy="$(arg arm_roll) ${-1.0*$(arg arm_pitch)} ${-3.14159 -$(arg arm_yaw)}"/>
     </xacro:pal_sea_arm>

File: tiago_pro_description/ros2_control/ros2_control.urdf.xacro (robot description, xacro)
@@ -12,22 +12,22 @@
   limitations under the License.
  -->
-<robot xmlns:xacro="http://ros.org/wiki/xacro"
-       name="tiago_pro" >
+<robot xmlns:xacro="http://ros.org/wiki/xacro" name="tiago_pro">
   <xacro:macro name="tiago_pro_ros2_control" params="use_sim:=^|false">
-    <xacro:arg name="arm_model_left" default="tiago-pro"/>
-    <xacro:arg name="arm_model_right" default="tiago-pro"/>
+    <xacro:arg name="arm_type_left" default="tiago-pro"/>
+    <xacro:arg name="arm_type_right" default="tiago-pro"/>
     <xacro:arg name="end_effector_left" default="pal-pro-pripper"/>
     <xacro:arg name="end_effector_right" default="pal-pro-gripper"/>
     <xacro:arg name="ft_sensor_left" default="no-ft-sensor"/>
     <xacro:arg name="ft_sensor_right" default="no-ft-sensor"/>
-    <xacro:arg name="description_calibration_dir" default="$(find tiago_pro_description)/urdf/calibration" /> <!-- TODO-->
-    <xacro:property name="arm_model_left" value="$(arg arm_model_left)" />
-    <xacro:property name="arm_model_right" value="$(arg arm_model_right)" />
+    <xacro:arg name="description_calibration_dir" default="$(find tiago_pro_description)/urdf/calibration" />
+    <!-- TODO-->
+    <xacro:property name="arm_type_left" value="$(arg arm_type_left)" />
+    <xacro:property name="arm_type_right" value="$(arg arm_type_right)" />
     <xacro:property name="end_effector_left" value="$(arg end_effector_left)" />
     <xacro:property name="end_effector_right" value="$(arg end_effector_right)" />
     <xacro:property name="has_ft_sensor_left" value="${ft_sensor_left != 'no-ft-sensor'}" />
     <xacro:property name="has_ft_sensor_right" value="${ft_sensor_right != 'no-ft-sensor'}" />
-    <xacro:property name="has_arm_left" value="${arm_model_left != 'no-arm'}" />
-    <xacro:property name="has_arm_right" value="${arm_model_right != 'no-arm'}" />
+    <xacro:property name="has_arm_left" value="${arm_type_left != 'no-arm'}" />
+    <xacro:property name="has_arm_right" value="${arm_type_right != 'no-arm'}" />
     <xacro:include filename="$(find omni_base_description)/urdf/sensors/sensors.ros2_control.xacro" />
     <xacro:include filename="$(find omni_base_description)/urdf/wheels/wheel.ros2_control.xacro" />
@@ -36,5 +36,5 @@
     <xacro:include filename="$(find pal_sea_arm_description)/urdf/arm/arm.ros2_control.xacro" />
     <xacro:if value="${end_effector_left == 'pal-pro-gripper' or end_effector_right == 'pal-pro-gripper'}">
-        <xacro:include filename="$(find pal_pro_gripper_description)/urdf/pal_pro_gripper.ros2_control.xacro" />
+      <xacro:include filename="$(find pal_pro_gripper_description)/urdf/pal_pro_gripper.ros2_control.xacro" />
     </xacro:if>
     <!-- calibration offsets -->
@@ -91,5 +91,5 @@
         <xacro:if value="${has_ft_sensor_right}">
           <xacro:include filename="$(find pal_sea_arm_description)/urdf/sensors/sensors.ros2_control.xacro"/>
-          <xacro:ros2_control_force_torque_sensor name="wrist_right_ft_sensor"/>
+          <xacro:ros2_control_force_torque_sensor name="wrist_right_ft_sensor"/>s
         </xacro:if>
         <xacro:if value="${end_effector_right == 'pal-pro-gripper'}">

Commit message: Added calibrated tf realsense for the real robot

File: tiago_pro_description/robots/tiago_pro.urdf.xacro (robot description, xacro)
@@ -39,4 +39,5 @@
   <xacro:arg name="arm_yaw" default="-1.2217" />
   <!-- PROPERTIES -->
+  <xacro:property name="use_sim" value="$(arg use_sim)" />
   <xacro:property name="laser_model" value="$(arg laser_model)" />
   <xacro:property name="arm_type_left" value="$(arg arm_type_left)" />

File: tiago_pro_description/urdf/head/head.urdf.xacro (robot description, xacro)
@@ -136,5 +136,5 @@
     </gazebo>
     <!-- Head camera:Intel D435 -->
-    <xacro:sensor_d435 parent="${name}_2_link" name="${name}_d435_camera" topics_ns="${name}_d435_camera" use_nominal_extrinsics="true">
+    <xacro:sensor_d435 parent="${name}_2_link" name="${name}_d435_camera" topics_ns="${name}_d435_camera" use_nominal_extrinsics="${use_sim}">
        <origin xyz="0.03815 0.14750 0.0"
                 rpy="${-90.0 * deg_to_rad} 0.0 0.0"/>

Commit message: Add is missing is_multiple xacro arg

File: tiago_pro_description/robots/tiago_pro.urdf.xacro (robot description, xacro)
@@ -30,4 +30,5 @@
   <xacro:arg name="use_sim" default="false"/>
   <xacro:arg name="is_public_sim" default="false"/>
+  <xacro:arg name="is_multiple" default="false"/>
   <xacro:arg name="description_calibration_dir" default="$(find tiago_pro_description)/urdf"/>
   <xacro:arg name="extrinsic_calibration_dir" default="$(find tiago_pro_description)/urdf"/>
@@ -40,4 +41,5 @@
   <!-- PROPERTIES -->
   <xacro:property name="use_sim" value="$(arg use_sim)" />
+  <xacro:property name="is_multiple" value="$(arg is_multiple)" />
   <xacro:property name="laser_model" value="$(arg laser_model)" />
   <xacro:property name="arm_type_left" value="$(arg arm_type_left)" />

Commit message: Change occurences of sim_time to use_sim_time

File: tiago_pro_description/robots/tiago_pro.urdf.xacro (robot description, xacro)
@@ -28,5 +28,5 @@
   <!-- no-ft-sensor, rokubi -->
   <xacro:arg name="ft_sensor_right" default="no-ft-sensor" />
-  <xacro:arg name="use_sim" default="false"/>
+  <xacro:arg name="use_sim_time" default="false"/>
   <xacro:arg name="is_public_sim" default="false"/>
   <xacro:arg name="is_multiple" default="false"/>
@@ -40,5 +40,5 @@
   <xacro:arg name="arm_yaw" default="-1.2217" />
   <!-- PROPERTIES -->
-  <xacro:property name="use_sim" value="$(arg use_sim)" />
+  <xacro:property name="use_sim_time" value="$(arg use_sim_time)" />
   <xacro:property name="is_multiple" value="$(arg is_multiple)" />
   <xacro:property name="laser_model" value="$(arg laser_model)" />
@@ -150,4 +150,4 @@
   </xacro:if>
   <!-- ROS 2 Control -->
-  <xacro:tiago_pro_ros2_control use_sim="$(arg use_sim)" />
+  <xacro:tiago_pro_ros2_control use_sim_time="$(arg use_sim_time)" />
 </robot>

File: tiago_pro_description/ros2_control/ros2_control.urdf.xacro (robot description, xacro)
@@ -13,5 +13,5 @@
  -->
 <robot xmlns:xacro="http://ros.org/wiki/xacro" name="tiago_pro">
-  <xacro:macro name="tiago_pro_ros2_control" params="use_sim:=^|false">
+  <xacro:macro name="tiago_pro_ros2_control" params="use_sim_time:=^|false">
     <xacro:arg name="arm_type_left" default="tiago-pro"/>
     <xacro:arg name="arm_type_right" default="tiago-pro"/>
@@ -50,8 +50,8 @@
     <ros2_control name="ros2_control_tiago_pro_system" type="system">
       <hardware>
-        <xacro:if value="$(arg use_sim)">
+        <xacro:if value="$(arg use_sim_time)">
           <plugin>gazebo_ros2_control/GazeboSystem</plugin>
         </xacro:if>
-        <xacro:unless value="$(arg use_sim)">
+        <xacro:unless value="$(arg use_sim_time)">
           <plugin>robot_control/RobotControl</plugin>
         </xacro:unless>
@@ -63,5 +63,5 @@
       <xacro:ros2_control_wheel side="rear_left" />
       <!-- IMU -->
-      <xacro:if value="$(arg use_sim)">
+      <xacro:if value="$(arg use_sim_time)">
         <xacro:ros2_control_imu name="base_imu_sensor"/>
       </xacro:if>

Commit message: Support for new old arm naming

File: tiago_pro_description/robots/tiago_pro.urdf.xacro (robot description, xacro)
@@ -49,5 +49,4 @@
   <xacro:property name="ft_sensor_left" value="$(arg ft_sensor_left)" />
   <xacro:property name="ft_sensor_right" value="$(arg ft_sensor_right)" />
-  <xacro:property name="arm_type" value="tiago-pro" />
   <xacro:property name="description_calibration_dir" value="${arg description_calibration_dir}"/>
   <xacro:property name="is_public_sim" value="$(arg is_public_sim)" />
@@ -63,8 +62,8 @@
   <xacro:property name="end_effector_right_name" value="gripper_right" />
   <!-- Properties check -->
-  <xacro:if value="${arm_type_left not in ['tiago-pro', 'no-arm']}">
+  <xacro:if value="${arm_type_left not in ['tiago-pro-prototype', 'tiago-pro', 'no-arm']}">
     <xacro:wrong_arm_type_left />
   </xacro:if>
-  <xacro:if value="${arm_type_right not in ['tiago-pro', 'no-arm']}">
+  <xacro:if value="${arm_type_right not in ['tiago-pro-prototype', 'tiago-pro', 'no-arm']}">
     <xacro:wrong_arm_type_right />
   </xacro:if>
