Commit message: Support for removable tray

File: tiago_pro_description/robots/tiago_pro.urdf.xacro (robot description, xacro)
@@ -28,4 +28,6 @@
   <!-- no-ft-sensor, rokubi -->
   <xacro:arg name="ft_sensor_right" default="no-ft-sensor" />
+  <!-- False, True -->
+  <xacro:arg name="has_laptop_tray" default="False" />
   <xacro:arg name="use_sim_time" default="false"/>
   <xacro:arg name="is_public_sim" default="false"/>
@@ -49,4 +51,5 @@
   <xacro:property name="ft_sensor_left" value="$(arg ft_sensor_left)" />
   <xacro:property name="ft_sensor_right" value="$(arg ft_sensor_right)" />
+  <xacro:property name="has_laptop_tray" value="$(arg has_laptop_tray)" />
   <xacro:property name="description_calibration_dir" value="${arg description_calibration_dir}"/>
   <xacro:property name="is_public_sim" value="$(arg is_public_sim)" />
@@ -114,6 +117,6 @@
   <!-- Base -->
   <xacro:base_sensors name="base" front_laser_model="$(arg laser_model)" rear_laser_model="$(arg laser_model)"/>
-  <!-- Torso. TODO:change for custom torso -->
-  <xacro:tiago_pro_torso name="torso" parent="base_link"/>
+  <!-- Torso -->
+  <xacro:tiago_pro_torso name="torso" parent="base_link" has_tray="${has_laptop_tray}"/>
   <!-- Head -->
   <xacro:tiago_pro_head name="head" parent="torso_lift_link"/>

File: tiago_pro_description/urdf/torso/torso.urdf.xacro (robot description, xacro)
@@ -16,5 +16,5 @@
   <xacro:property name="torso_max_vel" value="0.07" />
   <xacro:property name="torso_eps" value="0.02" />
-  <xacro:macro name="tiago_pro_torso" params="name parent">
+  <xacro:macro name="tiago_pro_torso" params="name parent has_tray">
     <!-- Connection with the base -->
     <link name="${name}_base_link">
@@ -96,13 +96,15 @@
         </material>
       </visual>
-      <visual>
-        <origin xyz="-0.226436438571948 3.12797385809451E-05 0.00524038105676683" rpy="0 0 -1.5707963267949" />
-        <geometry>
-          <mesh filename="package://tiago_pro_description/meshes/torso/laptop_tray.stl" />
-        </geometry>
-        <material name="">
-          <color rgba="0.894117647058823 0.913725490196078 0.929411764705882 1" />
-        </material>
-      </visual>
+      <xacro:if value="${has_tray}">
+        <visual>
+          <origin xyz="-0.226436438571948 3.12797385809451E-05 0.00524038105676683" rpy="0 0 -1.5707963267949" />
+          <geometry>
+            <mesh filename="package://tiago_pro_description/meshes/torso/laptop_tray.stl" />
+          </geometry>
+          <material name="">
+            <color rgba="0.894117647058823 0.913725490196078 0.929411764705882 1" />
+          </material>
+        </visual>
+      </xacro:if>
       <collision>
         <origin xyz="0 0 0" rpy="0 0 0" />
@@ -111,10 +113,12 @@
         </geometry>
       </collision>
-      <collision>
-        <origin xyz="-0.226436438571948 3.12797385809451E-05 0.00524038105676683" rpy="0 0 -1.5707963267949" />
-        <geometry>
-          <mesh filename="package://tiago_pro_description/meshes/torso/laptop_tray_collision.stl" />
-        </geometry>
-      </collision>
+      <xacro:if value="${has_tray}">
+        <collision>
+          <origin xyz="-0.226436438571948 3.12797385809451E-05 0.00524038105676683" rpy="0 0 -1.5707963267949" />
+          <geometry>
+            <mesh filename="package://tiago_pro_description/meshes/torso/laptop_tray_collision.stl" />
+          </geometry>
+        </collision>
+      </xacro:if>
     </link>
     <joint name="${name}_lift_joint" type="prismatic">

Commit message: Added wrist_model and tool_changer args

File: tiago_pro_description/robots/tiago_pro.urdf.xacro (robot description, xacro)
@@ -20,4 +20,12 @@
   <!-- tiago-pro, no-arm -->
   <xacro:arg name="arm_type_right" default="tiago-pro" />
+  <!-- straight-wrist, spherical-wrist -->
+  <xacro:arg name="wrist_model_left" default="straight-wrist" />
+  <!-- straight-wrist, spherical-wrist -->
+  <xacro:arg name="wrist_model_right" default="straight-wrist" />
+  <!-- False, True -->
+  <xacro:arg name="tool_changer_right" default="True" />
+  <!-- False, True -->
+  <xacro:arg name="tool_changer_left" default="True" />
   <!-- pal-pro-gripper custom-->
   <xacro:arg name="end_effector_left" default="pal-pro-gripper" />
@@ -47,4 +55,8 @@
   <xacro:property name="arm_type_left" value="$(arg arm_type_left)" />
   <xacro:property name="arm_type_right" value="$(arg arm_type_right)" />
+  <xacro:property name="tool_changer_left" value="$(arg tool_changer_left)" />
+  <xacro:property name="tool_changer_right" value="$(arg tool_changer_right)" />
+  <xacro:property name="wrist_model_left" value="$(arg wrist_model_left)" />
+  <xacro:property name="wrist_model_right" value="$(arg wrist_model_right)" />
   <xacro:property name="end_effector_left" value="$(arg end_effector_left)" />
   <xacro:property name="end_effector_right" value="$(arg end_effector_right)" />
@@ -52,4 +64,5 @@
   <xacro:property name="ft_sensor_right" value="$(arg ft_sensor_right)" />
   <xacro:property name="has_laptop_tray" value="$(arg has_laptop_tray)" />
+  <xacro:property name="tool_changer" value="$(arg tool_changer)" />
   <xacro:property name="description_calibration_dir" value="${arg description_calibration_dir}"/>
   <xacro:property name="is_public_sim" value="$(arg is_public_sim)" />
@@ -124,10 +137,10 @@
   <xacro:if value="${has_arm_left}">
     <!-- Arm -->
-    <xacro:pal_sea_arm name="arm_left" parent="torso_lift_link" arm_type="${arm_type_left}" reflect="1" arm_1_offset="${arm_left_1_joint_offset}" arm_2_offset="${arm_left_2_joint_offset}" arm_3_offset="${arm_left_3_joint_offset}" arm_4_offset="${arm_left_4_joint_offset}" arm_5_offset="${arm_left_5_joint_offset}" arm_6_offset="${arm_left_6_joint_offset}" arm_7_offset="${arm_left_7_joint_offset}">
+    <xacro:pal_sea_arm name="arm_left" parent="torso_lift_link" arm_type="${arm_type_left}" wrist_model="${wrist_model_left}" reflect="1" arm_1_offset="${arm_left_1_joint_offset}" arm_2_offset="${arm_left_2_joint_offset}" arm_3_offset="${arm_left_3_joint_offset}" arm_4_offset="${arm_left_4_joint_offset}" arm_5_offset="${arm_left_5_joint_offset}" arm_6_offset="${arm_left_6_joint_offset}" arm_7_offset="${arm_left_7_joint_offset}">
       <origin xyz="$(arg arm_x) $(arg arm_y) $(arg arm_z)" rpy="$(arg arm_roll) $(arg arm_pitch) $(arg arm_yaw)"/>
     </xacro:pal_sea_arm>
     <!-- End effector -->
     <xacro:if value="${has_end_effector_left}">
-      <xacro:pal_sea_arm_end_effector name="gripper_left" parent="${end_effector_left_link}" type="${end_effector_left}" has_end_effector="${has_end_effector_left}" reflect="-1" is_dual="true"/>
+      <xacro:pal_sea_arm_end_effector name="gripper_left" parent="${end_effector_left_link}" type="${end_effector_left}" tool_changer="${tool_changer_left}" reflect="-1"/>
     </xacro:if>
     <!-- FT sensors -->
@@ -139,10 +152,10 @@
   <xacro:if value="${has_arm_right}">
     <!-- Arm -->
-    <xacro:pal_sea_arm name="arm_right" parent="torso_lift_link" arm_type="${arm_type_right}" reflect="1" arm_1_offset="${arm_right_1_joint_offset}" arm_2_offset="${arm_right_2_joint_offset}" arm_3_offset="${arm_right_3_joint_offset}" arm_4_offset="${arm_right_4_joint_offset}" arm_5_offset="${arm_right_5_joint_offset}" arm_6_offset="${arm_right_6_joint_offset}" arm_7_offset="${arm_right_7_joint_offset}">
+    <xacro:pal_sea_arm name="arm_right" parent="torso_lift_link" arm_type="${arm_type_right}" wrist_model="${wrist_model_right}" reflect="1" arm_1_offset="${arm_right_1_joint_offset}" arm_2_offset="${arm_right_2_joint_offset}" arm_3_offset="${arm_right_3_joint_offset}" arm_4_offset="${arm_right_4_joint_offset}" arm_5_offset="${arm_right_5_joint_offset}" arm_6_offset="${arm_right_6_joint_offset}" arm_7_offset="${arm_right_7_joint_offset}">
       <origin xyz="$(arg arm_x) ${-1.0*$(arg arm_y)} $(arg arm_z)" rpy="$(arg arm_roll) ${-1.0*$(arg arm_pitch)} ${-3.14159 -$(arg arm_yaw)}"/>
     </xacro:pal_sea_arm>
     <!-- End effector -->
     <xacro:if value="${has_end_effector_right}">
-      <xacro:pal_sea_arm_end_effector name="gripper_right" parent="${end_effector_right_link}" type="${end_effector_right}" has_end_effector="${has_end_effector_right}" reflect="1" is_dual="true"/>
+      <xacro:pal_sea_arm_end_effector name="gripper_right" parent="${end_effector_right_link}" type="${end_effector_right}" tool_changer="${tool_changer_right}" reflect="1"/>
     </xacro:if>
     <!-- FT sensors -->

File: tiago_pro_description/ros2_control/ros2_control.urdf.xacro (robot description, xacro)
@@ -20,39 +20,40 @@
   </xacro:macro>
   <xacro:macro name="ros2_control_arms">
-      <!-- arm left -->
-      <xacro:if value="${has_arm_left}">
-        <xacro:ros2_control_arm name="arm_left_1" reduction="1.0" offset_value="${arm_left_1_joint_offset}" />
-        <xacro:ros2_control_arm name="arm_left_2" reduction="1.0" offset_value="${arm_left_2_joint_offset}" />
-        <xacro:ros2_control_arm name="arm_left_3" reduction="1.0" offset_value="${arm_left_3_joint_offset}" />
-        <xacro:ros2_control_arm name="arm_left_4" reduction="1.0" offset_value="${arm_left_4_joint_offset}" />
-        <xacro:ros2_control_arm name="arm_left_5" reduction="1.0" offset_value="${arm_left_5_joint_offset}" />
-        <xacro:ros2_control_arm name="arm_left_6" reduction="1.0" offset_value="${arm_left_6_joint_offset}" />
-        <xacro:ros2_control_arm name="arm_left_7" reduction="1.0" offset_value="${arm_left_7_joint_offset}" />
-        <xacro:if value="${has_ft_sensor_left}">
-          <xacro:include filename="$(find pal_sea_arm_description)/urdf/sensors/sensors.ros2_control.xacro"/>
-          <xacro:ros2_control_force_torque_sensor name="wrist_left_ft_sensor"/>
-        </xacro:if>
-        <xacro:if value="${end_effector_left == 'pal-pro-gripper'}">
-          <xacro:ros2_control_pal_pro_gripper name="gripper_left" reduction="1.0" />
-        </xacro:if>
+    <!-- arm left -->
+    <xacro:if value="${has_arm_left}">
+      <xacro:ros2_control_arm name="arm_left_1" reduction="1.0" offset_value="${arm_left_1_joint_offset}" />
+      <xacro:ros2_control_arm name="arm_left_2" reduction="1.0" offset_value="${arm_left_2_joint_offset}" />
+      <xacro:ros2_control_arm name="arm_left_3" reduction="1.0" offset_value="${arm_left_3_joint_offset}" />
+      <xacro:ros2_control_arm name="arm_left_4" reduction="1.0" offset_value="${arm_left_4_joint_offset}" />
+      <xacro:ros2_control_arm name="arm_left_5" reduction="1.0" offset_value="${arm_left_5_joint_offset}" />
+      <xacro:ros2_control_arm name="arm_left_6" reduction="1.0" offset_value="${arm_left_6_joint_offset}" />
+      <xacro:ros2_control_arm name="arm_left_7" reduction="1.0" offset_value="${arm_left_7_joint_offset}" />
+      <xacro:if value="${has_ft_sensor_left}">
+        <xacro:include filename="$(find pal_sea_arm_description)/urdf/sensors/sensors.ros2_control.xacro"/>
+        <xacro:ros2_control_force_torque_sensor name="wrist_left_ft_sensor"/>
       </xacro:if>
-      <!-- arm right -->
-      <xacro:if value="${has_arm_right}">
-        <xacro:ros2_control_arm name="arm_right_1" reduction="1.0" offset_value="${arm_right_1_joint_offset}" />
-        <xacro:ros2_control_arm name="arm_right_2" reduction="1.0" offset_value="${arm_right_2_joint_offset}" />
-        <xacro:ros2_control_arm name="arm_right_3" reduction="1.0" offset_value="${arm_right_3_joint_offset}" />
-        <xacro:ros2_control_arm name="arm_right_4" reduction="1.0" offset_value="${arm_right_4_joint_offset}" />
-        <xacro:ros2_control_arm name="arm_right_5" reduction="1.0" offset_value="${arm_right_5_joint_offset}" />
-        <xacro:ros2_control_arm name="arm_right_6" reduction="1.0" offset_value="${arm_right_6_joint_offset}" />
-        <xacro:ros2_control_arm name="arm_right_7" reduction="1.0" offset_value="${arm_right_7_joint_offset}" />
-        <xacro:if value="${has_ft_sensor_right}">
-          <xacro:include filename="$(find pal_sea_arm_description)/urdf/sensors/sensors.ros2_control.xacro"/>
-          <xacro:ros2_control_force_torque_sensor name="wrist_right_ft_sensor"/>s
-        </xacro:if>
-        <xacro:if value="${end_effector_right == 'pal-pro-gripper'}">
-          <!-- pal-pro-gripper -->
-          <xacro:ros2_control_pal_pro_gripper name="gripper_right" reduction="1.0" />
-        </xacro:if>
+      <xacro:if value="${end_effector_left == 'pal-pro-gripper'}">
+        <xacro:ros2_control_pal_pro_gripper name="gripper_left" reduction="1.0" />
       </xacro:if>
+    </xacro:if>
+    <!-- arm right -->
+    <xacro:if value="${has_arm_right}">
+      <xacro:ros2_control_arm name="arm_right_1" reduction="1.0" offset_value="${arm_right_1_joint_offset}" />
+      <xacro:ros2_control_arm name="arm_right_2" reduction="1.0" offset_value="${arm_right_2_joint_offset}" />
+      <xacro:ros2_control_arm name="arm_right_3" reduction="1.0" offset_value="${arm_right_3_joint_offset}" />
+      <xacro:ros2_control_arm name="arm_right_4" reduction="1.0" offset_value="${arm_right_4_joint_offset}" />
+      <xacro:ros2_control_arm name="arm_right_5" reduction="1.0" offset_value="${arm_right_5_joint_offset}" />
+      <xacro:ros2_control_arm name="arm_right_6" reduction="1.0" offset_value="${arm_right_6_joint_offset}" />
+      <xacro:ros2_control_arm name="arm_right_7" reduction="1.0" offset_value="${arm_right_7_joint_offset}" />
+      <xacro:if value="${has_ft_sensor_right}">
+        <xacro:include filename="$(find pal_sea_arm_description)/urdf/sensors/sensors.ros2_control.xacro"/>
+        <xacro:ros2_control_force_torque_sensor name="wrist_right_ft_sensor"/>
+s
+      </xacro:if>
+      <xacro:if value="${end_effector_right == 'pal-pro-gripper'}">
+        <!-- pal-pro-gripper -->
+        <xacro:ros2_control_pal_pro_gripper name="gripper_right" reduction="1.0" />
+      </xacro:if>
+    </xacro:if>
   </xacro:macro>
   <xacro:macro name="tiago_pro_ros2_control" params="use_sim_time:=^|false">
@@ -79,5 +80,5 @@
     <xacro:include filename="$(find pal_sea_arm_description)/urdf/arm/arm.ros2_control.xacro" />
     <xacro:if value="${end_effector_left == 'pal-pro-gripper' or end_effector_right == 'pal-pro-gripper'}">
-      <xacro:include filename="$(find pal_pro_gripper_description)/urdf/pal_pro_gripper.ros2_control.xacro" />
+      <xacro:include filename="$(find pal_pro_gripper_description)/urdf/gripper.ros2_control.xacro" />
     </xacro:if>
     <!-- calibration offsets -->
@@ -105,5 +106,5 @@
         <xacro:ros2_control_head name="head_2" reduction="1.0" offset_value="${head_2_joint_offset}" />
         <!-- arms -->
-          <xacro:ros2_control_arms/>
+        <xacro:ros2_control_arms/>
       </ros2_control>
     </xacro:if>

Commit message: Support for multiple FT sensors at the same time

File: tiago_pro_description/robots/tiago_pro.urdf.xacro (robot description, xacro)
@@ -64,5 +64,4 @@
   <xacro:property name="ft_sensor_right" value="$(arg ft_sensor_right)" />
   <xacro:property name="has_laptop_tray" value="$(arg has_laptop_tray)" />
-  <xacro:property name="tool_changer" value="$(arg tool_changer)" />
   <xacro:property name="description_calibration_dir" value="${arg description_calibration_dir}"/>
   <xacro:property name="is_public_sim" value="$(arg is_public_sim)" />
@@ -90,12 +89,37 @@
     <xacro:wrong_end_effector_right />
   </xacro:if>
-  <xacro:if value="${ft_sensor_left not in ['no-ft-sensor', 'rokubi']}">
+  <xacro:if value="${ft_sensor_left not in ['no-ft-sensor', 'rokubi', 'ati']}">
     <xacro:wrong_ft_sensor_left />
   </xacro:if>
-  <xacro:if value="${ft_sensor_right not in ['no-ft-sensor', 'rokubi']}">
+  <xacro:if value="${ft_sensor_right not in ['no-ft-sensor', 'rokubi', 'ati']}">
     <xacro:wrong_ft_sensor_right />
   </xacro:if>
   <xacro:if value="${laser_model not in ['no-laser', 'sick-571']}">
     <xacro:wrong_laser_model />
+  </xacro:if>
+  <!-- Compatibility check within TC and ft sensors-->
+  <xacro:if value="${ft_sensor_right == 'rokubi' and wrist_model_right=='straight-wrist'}">
+    <xacro:error_ati_not_compatible_with_straight_wrist />
+  </xacro:if>
+  <xacro:if value="${ft_sensor_left == 'ati' and wrist_model_left=='straight-wrist'}">
+    <xacro:error_rokubi_not_compatible_with_spherical_wrist />
+  </xacro:if>
+  <xacro:if value="${ft_sensor_right == 'rokubi' and tool_changer_right}">
+    <xacro:error_rokubi_not_compatible_with_tc />
+  </xacro:if>
+  <xacro:if value="${ft_sensor_left == 'rokubi' and tool_changer_left}">
+    <xacro:error_rokubi_not_compatible_with_tc />
+  </xacro:if>
+  <xacro:if value="${not tool_changer_right and wrist_model_right=='spherical-wrist'}">
+    <xacro:error_spherical_wrist_always_comes_with_tc />
+  </xacro:if>
+  <xacro:if value="${not tool_changer_left and wrist_model_left=='spherical-wrist'}">
+    <xacro:error_spherical_wrist_always_comes_with_tc />
+  </xacro:if>
+  <xacro:if value="${not tool_changer_left and ft_sensor_left == 'ati'}">
+    <xacro:error_ati_always_comes_with_tc />
+  </xacro:if>
+  <xacro:if value="${not tool_changer_right and ft_sensor_right == 'ati'}">
+    <xacro:error_ati_always_comes_with_tc />
   </xacro:if>
   <!-- INCLUDES -->
@@ -118,6 +142,6 @@
   <!-- Force Torque sensor -->
   <xacro:if value="${has_ft_sensor_right or has_ft_sensor_left}">
-    <xacro:include filename="$(find pal_sea_arm_description)/urdf/sensors/ft_sensor.urdf.xacro" />
-    <xacro:include filename="$(find pal_sea_arm_description)/urdf/sensors/ft_sensor.gazebo.xacro" />
+    <xacro:include filename="$(find pal_sea_arm_description)/urdf/sensors/ft_sensor/ft_sensor.urdf.xacro" />
+    <xacro:include filename="$(find pal_sea_arm_description)/urdf/sensors/ft_sensor/ft_sensor.gazebo.xacro" />
   </xacro:if>
   <!-- Head -->
@@ -137,5 +161,5 @@
   <xacro:if value="${has_arm_left}">
     <!-- Arm -->
-    <xacro:pal_sea_arm name="arm_left" parent="torso_lift_link" arm_type="${arm_type_left}" wrist_model="${wrist_model_left}" reflect="1" arm_1_offset="${arm_left_1_joint_offset}" arm_2_offset="${arm_left_2_joint_offset}" arm_3_offset="${arm_left_3_joint_offset}" arm_4_offset="${arm_left_4_joint_offset}" arm_5_offset="${arm_left_5_joint_offset}" arm_6_offset="${arm_left_6_joint_offset}" arm_7_offset="${arm_left_7_joint_offset}">
+    <xacro:pal_sea_arm name="arm_left" parent="torso_lift_link" arm_type="${arm_type_left}" wrist_model="${wrist_model_left}" tool_changer="${tool_changer_left}" reflect="1" arm_1_offset="${arm_left_1_joint_offset}" arm_2_offset="${arm_left_2_joint_offset}" arm_3_offset="${arm_left_3_joint_offset}" arm_4_offset="${arm_left_4_joint_offset}" arm_5_offset="${arm_left_5_joint_offset}" arm_6_offset="${arm_left_6_joint_offset}" arm_7_offset="${arm_left_7_joint_offset}">
       <origin xyz="$(arg arm_x) $(arg arm_y) $(arg arm_z)" rpy="$(arg arm_roll) $(arg arm_pitch) $(arg arm_yaw)"/>
     </xacro:pal_sea_arm>
@@ -146,5 +170,5 @@
     <!-- FT sensors -->
     <xacro:if value="${has_ft_sensor_left}">
-      <xacro:ft_sensor name="wrist_left" parent="arm_left_tool_link"/>
+      <xacro:ft_sensor type="${ft_sensor_left}" name="wrist_left" parent="arm_left_tool_link"/>
     </xacro:if>
   </xacro:if>
@@ -152,5 +176,5 @@
   <xacro:if value="${has_arm_right}">
     <!-- Arm -->
-    <xacro:pal_sea_arm name="arm_right" parent="torso_lift_link" arm_type="${arm_type_right}" wrist_model="${wrist_model_right}" reflect="1" arm_1_offset="${arm_right_1_joint_offset}" arm_2_offset="${arm_right_2_joint_offset}" arm_3_offset="${arm_right_3_joint_offset}" arm_4_offset="${arm_right_4_joint_offset}" arm_5_offset="${arm_right_5_joint_offset}" arm_6_offset="${arm_right_6_joint_offset}" arm_7_offset="${arm_right_7_joint_offset}">
+    <xacro:pal_sea_arm name="arm_right" parent="torso_lift_link" arm_type="${arm_type_right}" wrist_model="${wrist_model_right}" tool_changer="${tool_changer_right}" reflect="1" arm_1_offset="${arm_right_1_joint_offset}" arm_2_offset="${arm_right_2_joint_offset}" arm_3_offset="${arm_right_3_joint_offset}" arm_4_offset="${arm_right_4_joint_offset}" arm_5_offset="${arm_right_5_joint_offset}" arm_6_offset="${arm_right_6_joint_offset}" arm_7_offset="${arm_right_7_joint_offset}">
       <origin xyz="$(arg arm_x) ${-1.0*$(arg arm_y)} $(arg arm_z)" rpy="$(arg arm_roll) ${-1.0*$(arg arm_pitch)} ${-3.14159 -$(arg arm_yaw)}"/>
     </xacro:pal_sea_arm>
@@ -161,5 +185,5 @@
     <!-- FT sensors -->
     <xacro:if value="${has_ft_sensor_right}">
-      <xacro:ft_sensor name="wrist_right" parent="arm_right_tool_link"/>
+      <xacro:ft_sensor type="${ft_sensor_right}" name="wrist_right" parent="arm_right_tool_link"/>
     </xacro:if>
   </xacro:if>

File: tiago_pro_description/ros2_control/ros2_control.urdf.xacro (robot description, xacro)
@@ -30,5 +30,5 @@
       <xacro:ros2_control_arm name="arm_left_7" reduction="1.0" offset_value="${arm_left_7_joint_offset}" />
       <xacro:if value="${has_ft_sensor_left}">
-        <xacro:include filename="$(find pal_sea_arm_description)/urdf/sensors/sensors.ros2_control.xacro"/>
+        <xacro:include filename="$(find pal_sea_arm_description)/urdf/sensors/ft_sensor/sensor.ros2_control.xacro"/>
         <xacro:ros2_control_force_torque_sensor name="wrist_left_ft_sensor"/>
       </xacro:if>
@@ -47,5 +47,5 @@
       <xacro:ros2_control_arm name="arm_right_7" reduction="1.0" offset_value="${arm_right_7_joint_offset}" />
       <xacro:if value="${has_ft_sensor_right}">
-        <xacro:include filename="$(find pal_sea_arm_description)/urdf/sensors/sensors.ros2_control.xacro"/>
+        <xacro:include filename="$(find pal_sea_arm_description)/urdf/sensors/ft_sensor/sensor.ros2_control.xacro"/>
         <xacro:ros2_control_force_torque_sensor name="wrist_right_ft_sensor"/>
 s
