Commit message: Fix head position

File: tiago_pro_description/robots/tiago_pro.urdf.xacro (robot description, xacro)
@@ -163,5 +163,5 @@
   <xacro:tiago_pro_torso name="torso" parent="base_link" has_tray="${has_laptop_tray}"/>
   <!-- Head -->
-  <xacro:tiago_pro_head name="head" parent="torso_lift_link"/>
+  <xacro:tiago_pro_head name="head" parent="torso_head_link"/>
   <!-- Left arm -->
   <xacro:if value="${has_arm_left}">

File: tiago_pro_description/urdf/head/head.urdf.xacro (robot description, xacro)
@@ -28,7 +28,14 @@
     <link name="${name}_1_link">
       <inertial>
-        <origin xyz="0.0016768 3.1033E-05 0.081737" rpy="0 0 0" />
-        <mass value="0.22677" />
-        <inertia ixx="0.00056619" ixy="3.0482E-07" ixz="6.7491E-05" iyy="0.00040222" iyz="-5.9322E-07" izz="0.00039176" />
+        <origin xyz="-0.0037459 -4.6685E-05 0.1055" rpy="0 0 0" />
+        <mass
+          value="0.15566" />
+        <inertia
+          ixx="0.0005208"
+          ixy="3.0453E-07"
+          ixz="-6.1005E-05"
+          iyy="0.00035021"
+          iyz="5.8627E-07"
+          izz="0.00033341" />
       </inertial>
       <visual>
@@ -49,5 +56,5 @@
     </link>
     <joint name="${name}_1_joint" type="revolute">
-      <origin xyz="0 0 0" rpy="0 0 3.14" />
+      <origin xyz="0 0 0" rpy="0 0 0" />
       <parent link="${parent}" />
       <child link="head_1_link" />
@@ -60,7 +67,16 @@
     <link name="${name}_2_link">
       <inertial>
-        <origin xyz="-0.0087157 0.11401 -0.00024206" rpy="0 0 0" />
-        <mass value="0.84465" />
-        <inertia ixx="0.006226" ixy="-0.00055126" ixz="-7.2157E-06" iyy="0.0050209" iyz="-1.0342E-05" izz="0.002495" />
+        <origin
+          xyz="-0.00875103486217405 0.114127350051331 -0.000389070804431699"
+          rpy="0 0 0" />
+        <mass
+          value="0.846359357446667" />
+        <inertia
+          ixx="0.00623850186261437"
+          ixy="-0.000550112126953165"
+          ixz="-9.403405403969E-06"
+          iyy="0.0050320204467172"
+          iyz="-5.68886635279132E-06"
+          izz="0.0024981099013485" />
       </inertial>
       <visual>
@@ -81,5 +97,5 @@
     </link>
     <joint name="head_2_joint" type="revolute">
-      <origin xyz="-0.0425 0 0.1011" rpy="1.5708 0 0" />
+      <origin xyz="0.0425 0 0.10585" rpy="1.5708 0 -3.1416" />
       <parent link="${name}_1_link" />
       <child link="${name}_2_link" />
@@ -113,5 +129,5 @@
     <!-- Head camera:Intel D435 -->
     <xacro:sensor_d435 parent="${name}_2_link" name="${name}_front_camera" topics_ns="${name}_front_camera" use_nominal_extrinsics="${use_sim_time}">
-      <origin xyz="-0.0415999999999995 0.1555 0" rpy="1.5707963267949 0 3.14159265358979" />
+      <origin xyz="-0.0416 0.1555 0" rpy="1.5708 0 3.1416" />
     </xacro:sensor_d435>
   </xacro:macro>

Commit message: Add camera model as parameter to check in head urdf

File: tiago_pro_description/robots/tiago_pro.urdf.xacro (robot description, xacro)
@@ -36,4 +36,6 @@
   <!-- no-ft-sensor, rokubi -->
   <xacro:arg name="ft_sensor_right" default="no-ft-sensor" />
+  <!-- realsense-d435 -->
+  <xacro:arg name="camera_model" default="realsense-d435" />
   <!-- False, True -->
   <xacro:arg name="has_laptop_tray" default="False" />
@@ -64,4 +66,5 @@
   <xacro:property name="ft_sensor_right" value="$(arg ft_sensor_right)" />
   <xacro:property name="has_laptop_tray" value="$(arg has_laptop_tray)" />
+  <xacro:property name="camera_model" value="$(arg camera_model)" />
   <xacro:property name="description_calibration_dir" value="${arg description_calibration_dir}"/>
   <xacro:property name="is_public_sim" value="$(arg is_public_sim)" />
@@ -163,5 +166,5 @@
   <xacro:tiago_pro_torso name="torso" parent="base_link" has_tray="${has_laptop_tray}"/>
   <!-- Head -->
-  <xacro:tiago_pro_head name="head" parent="torso_head_link"/>
+  <xacro:tiago_pro_head name="head" parent="torso_head_link" camera_model="$(arg camera_model)"/>
   <!-- Left arm -->
   <xacro:if value="${has_arm_left}">

Commit message: Remove has_tray argument

File: tiago_pro_description/robots/tiago_pro.urdf.xacro (robot description, xacro)
@@ -38,6 +38,4 @@
   <!-- realsense-d435 -->
   <xacro:arg name="camera_model" default="realsense-d435" />
-  <!-- False, True -->
-  <xacro:arg name="has_laptop_tray" default="False" />
   <xacro:arg name="use_sim_time" default="false"/>
   <xacro:arg name="is_public_sim" default="false"/>
@@ -65,5 +63,4 @@
   <xacro:property name="ft_sensor_left" value="$(arg ft_sensor_left)" />
   <xacro:property name="ft_sensor_right" value="$(arg ft_sensor_right)" />
-  <xacro:property name="has_laptop_tray" value="$(arg has_laptop_tray)" />
   <xacro:property name="camera_model" value="$(arg camera_model)" />
   <xacro:property name="description_calibration_dir" value="${arg description_calibration_dir}"/>
@@ -164,5 +161,5 @@
   <xacro:base_sensors name="base" front_laser_model="$(arg laser_model)" rear_laser_model="$(arg laser_model)"/>
   <!-- Torso -->
-  <xacro:tiago_pro_torso name="torso" parent="base_link" has_tray="${has_laptop_tray}"/>
+  <xacro:tiago_pro_torso name="torso" parent="base_link"/>
   <!-- Head -->
   <xacro:tiago_pro_head name="head" parent="torso_head_link" camera_model="$(arg camera_model)"/>

File: tiago_pro_description/urdf/torso/torso.urdf.xacro (robot description, xacro)
@@ -16,5 +16,5 @@
   <xacro:property name="torso_max_vel" value="0.035" />
   <xacro:property name="torso_eps" value="0.00" />
-  <xacro:macro name="tiago_pro_torso" params="name parent has_tray">
+  <xacro:macro name="tiago_pro_torso" params="name parent">
     <!-- Connection with the base -->
     <link name="${name}_base_link">
@@ -96,15 +96,4 @@
         </material>
       </visual>
-      <xacro:if value="${has_tray}">
-        <visual>
-          <origin xyz="-0.226436438571948 3.12797385809451E-05 0.00524038105676683" rpy="0 0 -1.5707963267949" />
-          <geometry>
-            <mesh filename="package://tiago_pro_description/meshes/torso/laptop_tray.stl" />
-          </geometry>
-          <material name="">
-            <color rgba="0.894117647058823 0.913725490196078 0.929411764705882 1" />
-          </material>
-        </visual>
-      </xacro:if>
       <collision>
         <origin xyz="0 0 0" rpy="0 0 0" />
@@ -113,12 +102,10 @@
         </geometry>
       </collision>
-      <xacro:if value="${has_tray}">
-        <collision>
-          <origin xyz="-0.226436438571948 3.12797385809451E-05 0.00524038105676683" rpy="0 0 -1.5707963267949" />
-          <geometry>
-            <mesh filename="package://tiago_pro_description/meshes/torso/laptop_tray_collision.stl" />
-          </geometry>
-        </collision>
-      </xacro:if>
+      <collision>
+        <origin xyz="-0.226436438571948 3.12797385809451E-05 0.00524038105676683" rpy="0 0 -1.5707963267949" />
+        <geometry>
+          <mesh filename="package://tiago_pro_description/meshes/torso/laptop_tray_collision.stl" />
+        </geometry>
+      </collision>
     </link>
     <joint name="${name}_lift_joint" type="prismatic">
@@ -153,26 +140,5 @@
     </gazebo>
     <!-- Torso arm left link-->
-    <link name="${name}_arm_left_link">
-      <inertial>
-        <origin xyz="0.0266347705878543 -1.34103746878278E-05 -0.0312554093037512" rpy="0 0 0" />
-        <mass value="0.230474445227561" />
-        <inertia ixx="0.000275825000057028" ixy="-2.98026741879157E-05" ixz="9.19765678097319E-05" iyy="0.000347873534928455" iyz="-2.2471230906564E-05" izz="0.00040318881619739" />
-      </inertial>
-      <visual>
-        <origin xyz="0 0 0" rpy="0 0 0" />
-        <geometry>
-          <mesh filename="package://tiago_pro_description/meshes/torso/arm_left_link.stl" />
-        </geometry>
-        <material name="">
-          <color rgba="0.250980392156863 0.250980392156863 0.250980392156863 1" />
-        </material>
-      </visual>
-      <collision>
-        <origin xyz="0 0 0" rpy="0 0 0" />
-        <geometry>
-          <mesh filename="package://tiago_pro_description/meshes/torso/arm_left_link_collision.stl" />
-        </geometry>
-      </collision>
-    </link>
+    <link name="${name}_arm_left_link"/>
     <joint name="${name}_arm_left_joint" type="fixed">
       <origin xyz="0.0898413194899453 0.159181203216899 -0.0920547375491735" rpy="-2.06788770984932 0 -1.22173047639603" />
@@ -185,26 +151,5 @@
     </gazebo>
     <!-- Torso arm right link -->
-    <link name="${name}_arm_right_link">
-      <inertial>
-        <origin xyz="-0.0266370901965068 -1.33503761214904E-05 -0.031255858525246" rpy="0 0 0" />
-        <mass value="0.230469561959048" />
-        <inertia ixx="0.000275821597759927" ixy="2.98126984098988E-05" ixz="-9.19722502498065E-05" iyy="0.000347870269485856" iyz="-2.24681274957806E-05" izz="0.000403186347482453" />
-      </inertial>
-      <visual>
-        <origin xyz="0 0 0" rpy="0 0 0" />
-        <geometry>
-          <mesh filename="package://tiago_pro_description/meshes/torso/arm_right_link.stl" />
-        </geometry>
-        <material name="">
-          <color rgba="0.250980392156863 0.250980392156863 0.250980392156863 1" />
-        </material>
-      </visual>
-      <collision>
-        <origin xyz="0 0 0" rpy="0 0 0" />
-        <geometry>
-          <mesh filename="package://tiago_pro_description/meshes/torso/arm_right_link_collision.stl" />
-        </geometry>
-      </collision>
-    </link>
+    <link name="${name}_arm_right_link"/>
     <joint name="${name}_arm_right_joint" type="fixed">
       <origin xyz="0.0898413194899453 -0.1591812032169 -0.0920547375491731" rpy="-2.06788770984932 0 -1.91986217719377" />

Commit message: Add allegro hand as a possible end effector

File: tiago_pro_description/robots/tiago_pro.urdf.xacro (robot description, xacro)
@@ -86,8 +86,8 @@
     <xacro:wrong_arm_type_right />
   </xacro:if>
-  <xacro:if value="${end_effector_left not in ['pal-pro-gripper', 'custom', 'no-end-effector']}">
+  <xacro:if value="${end_effector_left not in ['pal-pro-gripper', 'custom', 'no-end-effector', 'allegro-hand']}">
     <xacro:wrong_end_effector_left />
   </xacro:if>
-  <xacro:if value="${end_effector_right not in ['pal-pro-gripper', 'custom', 'no-end-effector']}">
+  <xacro:if value="${end_effector_right not in ['pal-pro-gripper', 'custom', 'no-end-effector', 'allegro-hand']}">
     <xacro:wrong_end_effector_right />
   </xacro:if>

File: tiago_pro_description/ros2_control/ros2_control.urdf.xacro (robot description, xacro)
@@ -18,4 +18,20 @@
     <xacro:ros2_control_wheel side="rear_right" />
     <xacro:ros2_control_wheel side="rear_left" />
+  </xacro:macro>
+  <xacro:macro name="allegro_ros2_control" params="side allegro_can pid_controllers xela_can">
+    <ros2_control name="ros2_control_allegro_hand_system_${side}" type="system" rw_rate="1000">
+      <hardware>
+        <plugin>allegro_hand_system/AllegroHandSystem</plugin>
+        <param name="${can_device_name}">${allegro_can}</param>
+        <param name="side">${side}</param>
+      </hardware>
+      <xacro:ros2_control_allegro_hand name="gripper_${side}" pid_controllers="$(arg pid_controllers)" reduction="1.0" />
+    </ros2_control>
+    <ros2_control name="ros2_control_xela_sensor_${side}" type="sensor" rw_rate="1000">
+      <hardware>
+        <plugin>xela_uskin_sensor/XelaUskinSensor</plugin>
+        <param name="${can_device_name}">${xela_can}</param>
+      </hardware>
+    </ros2_control>
   </xacro:macro>
   <xacro:macro name="ros2_control_arms">
@@ -73,4 +89,5 @@
     <xacro:property name="has_arm_left" value="${arm_type_left != 'no-arm'}" />
     <xacro:property name="has_arm_right" value="${arm_type_right != 'no-arm'}" />
+    <xacro:property name="can_device_name" value="can_device" />
     <xacro:include filename="$(find omni_base_description)/urdf/sensors/sensors.ros2_control.xacro" />
     <xacro:include filename="$(find omni_base_description)/urdf/wheels/wheel.ros2_control.xacro" />
@@ -80,4 +97,7 @@
     <xacro:if value="${end_effector_left == 'pal-pro-gripper' or end_effector_right == 'pal-pro-gripper'}">
       <xacro:include filename="$(find pal_pro_gripper_description)/urdf/gripper.ros2_control.xacro" />
+    </xacro:if>
+    <xacro:if value="${end_effector_left == 'allegro-hand' or end_effector_right == 'allegro-hand'}">
+      <xacro:include filename="$(find allegro_hand_description)/urdf/allegro_hand.ros2_control.xacro" />
     </xacro:if>
     <!-- calibration offsets -->
@@ -103,4 +123,11 @@
         <!-- arms -->
         <xacro:ros2_control_arms/>
+        <xacro:arg name="pid_controllers" default="false"/>
+        <xacro:if value="${end_effector_right == 'allegro-hand'}">
+          <xacro:ros2_control_allegro_hand name="gripper_right" pid_controllers="$(arg pid_controllers)" reduction="1.0" />
+        </xacro:if>
+        <xacro:if value="${end_effector_left == 'allegro-hand'}">
+          <xacro:ros2_control_allegro_hand name="gripper_left" pid_controllers="$(arg pid_controllers)" reduction="1.0" />
+        </xacro:if>
       </ros2_control>
     </xacro:if>
@@ -135,4 +162,11 @@
         <xacro:ros2_control_torso name="torso_lift" reduction="1.0" />
       </ros2_control>
+      <xacro:arg name="pid_controllers" default="true"/>
+      <xacro:if value="${end_effector_right == 'allegro-hand'}">
+        <xacro:allegro_ros2_control side="right" allegro_can="can0" pid_controllers="$(arg pid_controllers)" xela_can="can1"/>
+      </xacro:if>
+      <xacro:if value="${end_effector_left == 'allegro-hand'}">
+        <xacro:allegro_ros2_control side="left" allegro_can="can2" pid_controllers="$(arg pid_controllers)" xela_can="can3"/>
+      </xacro:if>
     </xacro:unless>
   </xacro:macro>

Commit message: Support for SEA in tiago_pro_description

File: tiago_pro_description/robots/tiago_pro.urdf.xacro (robot description, xacro)
@@ -38,4 +38,6 @@
   <!-- realsense-d435 -->
   <xacro:arg name="camera_model" default="realsense-d435" />
+  <!-- False, True -->
+  <xacro:arg name="torque_estimation" default="False" />
   <xacro:arg name="use_sim_time" default="false"/>
   <xacro:arg name="is_public_sim" default="false"/>
@@ -50,4 +52,5 @@
   <xacro:arg name="arm_yaw" default="-1.2217" />
   <!-- PROPERTIES -->
+  <xacro:property name="torque_estimation" value="$(arg torque_estimation)" />
   <xacro:property name="use_sim_time" value="$(arg use_sim_time)" />
   <xacro:property name="is_multiple" value="$(arg is_multiple)" />
@@ -167,5 +170,5 @@
   <xacro:if value="${has_arm_left}">
     <!-- Arm -->
-    <xacro:pal_sea_arm name="arm_left" parent="torso_lift_link" arm_type="${arm_type_left}" wrist_model="${wrist_model_left}" tool_changer="${tool_changer_left}" reflect="1"  joint_reflect="-1" arm_1_offset="${arm_left_1_joint_offset}" arm_2_offset="${arm_left_2_joint_offset}" arm_3_offset="${arm_left_3_joint_offset}" arm_4_offset="${arm_left_4_joint_offset}" arm_5_offset="${arm_left_5_joint_offset}" arm_6_offset="${arm_left_6_joint_offset}" arm_7_offset="${arm_left_7_joint_offset}">
+    <xacro:pal_sea_arm name="arm_left" parent="torso_lift_link" arm_type="${arm_type_left}" wrist_model="${wrist_model_left}" tool_changer="${tool_changer_left}" reflect="1" joint_reflect="-1" arm_1_offset="${arm_left_1_joint_offset}" arm_2_offset="${arm_left_2_joint_offset}" arm_3_offset="${arm_left_3_joint_offset}" arm_4_offset="${arm_left_4_joint_offset}" arm_5_offset="${arm_left_5_joint_offset}" arm_6_offset="${arm_left_6_joint_offset}" arm_7_offset="${arm_left_7_joint_offset}">
       <origin xyz="$(arg arm_x) $(arg arm_y) $(arg arm_z)" rpy="$(arg arm_roll) $(arg arm_pitch) $(arg arm_yaw)"/>
     </xacro:pal_sea_arm>
@@ -182,5 +185,5 @@
   <xacro:if value="${has_arm_right}">
     <!-- Arm -->
-    <xacro:pal_sea_arm name="arm_right" parent="torso_lift_link" arm_type="${arm_type_right}" wrist_model="${wrist_model_right}" tool_changer="${tool_changer_right}" reflect="1"  joint_reflect="1" arm_1_offset="${arm_right_1_joint_offset}" arm_2_offset="${arm_right_2_joint_offset}" arm_3_offset="${arm_right_3_joint_offset}" arm_4_offset="${arm_right_4_joint_offset}" arm_5_offset="${arm_right_5_joint_offset}" arm_6_offset="${arm_right_6_joint_offset}" arm_7_offset="${arm_right_7_joint_offset}">
+    <xacro:pal_sea_arm name="arm_right" parent="torso_lift_link" arm_type="${arm_type_right}" wrist_model="${wrist_model_right}" tool_changer="${tool_changer_right}" reflect="1" joint_reflect="1" arm_1_offset="${arm_right_1_joint_offset}" arm_2_offset="${arm_right_2_joint_offset}" arm_3_offset="${arm_right_3_joint_offset}" arm_4_offset="${arm_right_4_joint_offset}" arm_5_offset="${arm_right_5_joint_offset}" arm_6_offset="${arm_right_6_joint_offset}" arm_7_offset="${arm_right_7_joint_offset}">
       <origin xyz="$(arg arm_x) ${-1.0*$(arg arm_y)} $(arg arm_z)" rpy="$(arg arm_roll) ${-1.0*$(arg arm_pitch)} ${-3.14159 -$(arg arm_yaw)}"/>
     </xacro:pal_sea_arm>

File: tiago_pro_description/ros2_control/ros2_control.urdf.xacro (robot description, xacro)
@@ -22,11 +22,11 @@
     <!-- arm left -->
     <xacro:if value="${has_arm_left}">
-      <xacro:ros2_control_arm name="arm_left_1" reduction="1.0" offset_value="${arm_left_1_joint_offset}" />
-      <xacro:ros2_control_arm name="arm_left_2" reduction="1.0" offset_value="${arm_left_2_joint_offset}" />
-      <xacro:ros2_control_arm name="arm_left_3" reduction="1.0" offset_value="${arm_left_3_joint_offset}" />
-      <xacro:ros2_control_arm name="arm_left_4" reduction="1.0" offset_value="${arm_left_4_joint_offset}" />
-      <xacro:ros2_control_arm name="arm_left_5" reduction="1.0" offset_value="${arm_left_5_joint_offset}" />
-      <xacro:ros2_control_arm name="arm_left_6" reduction="1.0" offset_value="${arm_left_6_joint_offset}" />
-      <xacro:ros2_control_arm name="arm_left_7" reduction="1.0" offset_value="${arm_left_7_joint_offset}" />
+      <xacro:ros2_control_arm name="arm_left_1" reduction="121.0" offset_value="${arm_left_1_joint_offset}" use_sea_transmission="${torque_estimation}" />
+      <xacro:ros2_control_arm name="arm_left_2" reduction="121.0" offset_value="${arm_left_2_joint_offset}" use_sea_transmission="${torque_estimation}" />
+      <xacro:ros2_control_arm name="arm_left_3" reduction="101.0" offset_value="${arm_left_3_joint_offset}" use_sea_transmission="${torque_estimation}" />
+      <xacro:ros2_control_arm name="arm_left_4" reduction="101.0" offset_value="${arm_left_4_joint_offset}" use_sea_transmission="${torque_estimation}" />
+      <xacro:ros2_control_arm name="arm_left_5" reduction="101.0" offset_value="${arm_left_5_joint_offset}" use_sea_transmission="${torque_estimation}" />
+      <xacro:ros2_control_arm name="arm_left_6" reduction="101.0" offset_value="${arm_left_6_joint_offset}" use_sea_transmission="${torque_estimation}" />
+      <xacro:ros2_control_arm name="arm_left_7" reduction="101.0" offset_value="${arm_left_7_joint_offset}" use_sea_transmission="${torque_estimation}" />
       <xacro:if value="${has_ft_sensor_left}">
         <xacro:include filename="$(find pal_sea_arm_description)/urdf/sensors/ft_sensor/sensor.ros2_control.xacro"/>
@@ -39,11 +39,11 @@
     <!-- arm right -->
     <xacro:if value="${has_arm_right}">
-      <xacro:ros2_control_arm name="arm_right_1" reduction="1.0" offset_value="${arm_right_1_joint_offset}" />
-      <xacro:ros2_control_arm name="arm_right_2" reduction="1.0" offset_value="${arm_right_2_joint_offset}" />
-      <xacro:ros2_control_arm name="arm_right_3" reduction="1.0" offset_value="${arm_right_3_joint_offset}" />
-      <xacro:ros2_control_arm name="arm_right_4" reduction="1.0" offset_value="${arm_right_4_joint_offset}" />
-      <xacro:ros2_control_arm name="arm_right_5" reduction="1.0" offset_value="${arm_right_5_joint_offset}" />
-      <xacro:ros2_control_arm name="arm_right_6" reduction="1.0" offset_value="${arm_right_6_joint_offset}" />
-      <xacro:ros2_control_arm name="arm_right_7" reduction="1.0" offset_value="${arm_right_7_joint_offset}" />
+      <xacro:ros2_control_arm name="arm_right_1" reduction="121.0" offset_value="${arm_right_1_joint_offset}" use_sea_transmission="${torque_estimation}" />
+      <xacro:ros2_control_arm name="arm_right_2" reduction="121.0" offset_value="${arm_right_2_joint_offset}" use_sea_transmission="${torque_estimation}" />
+      <xacro:ros2_control_arm name="arm_right_3" reduction="101.0" offset_value="${arm_right_3_joint_offset}" use_sea_transmission="${torque_estimation}" />
+      <xacro:ros2_control_arm name="arm_right_4" reduction="101.0" offset_value="${arm_right_4_joint_offset}" use_sea_transmission="${torque_estimation}" />
+      <xacro:ros2_control_arm name="arm_right_5" reduction="101.0" offset_value="${arm_right_5_joint_offset}" use_sea_transmission="${torque_estimation}" />
+      <xacro:ros2_control_arm name="arm_right_6" reduction="101.0" offset_value="${arm_right_6_joint_offset}" use_sea_transmission="${torque_estimation}" />
+      <xacro:ros2_control_arm name="arm_right_7" reduction="101.0" offset_value="${arm_right_7_joint_offset}" use_sea_transmission="${torque_estimation}" />
       <xacro:if value="${has_ft_sensor_right}">
         <xacro:include filename="$(find pal_sea_arm_description)/urdf/sensors/ft_sensor/sensor.ros2_control.xacro"/>

Commit message: Uniform namespace

File: tiago_pro_description/robots/tiago_pro.urdf.xacro (robot description, xacro)
@@ -43,4 +43,5 @@
   <xacro:arg name="is_public_sim" default="false"/>
   <xacro:arg name="is_multiple" default="false"/>
+  <xacro:arg name="namespace" default=""/>
   <xacro:arg name="description_calibration_dir" default="$(find tiago_pro_description)/urdf"/>
   <xacro:arg name="extrinsic_calibration_dir" default="$(find tiago_pro_description)/urdf"/>
@@ -55,4 +56,5 @@
   <xacro:property name="use_sim_time" value="$(arg use_sim_time)" />
   <xacro:property name="is_multiple" value="$(arg is_multiple)" />
+  <xacro:property name="namespace" value="$(arg namespace)" />
   <xacro:property name="laser_model" value="$(arg laser_model)" />
   <xacro:property name="arm_type_left" value="$(arg arm_type_left)" />

Commit message: Added tip frame

File: tiago_pro_description/robots/tiago_pro.urdf.xacro (robot description, xacro)
@@ -201,3 +201,9 @@
   <!-- ROS 2 Control -->
   <xacro:tiago_pro_ros2_control use_sim_time="$(arg use_sim_time)" />
+  <link name="tip"/>
+  <joint name="tool0_to_tip" type="fixed">
+    <parent link="arm_right_tool_link"/>
+    <child link="tip"/>
+    <origin xyz="0 0 0.15" rpy="0 0 0"/>
+  </joint>
 </robot>
